File: hw/ZID_POD/ZID_POD.kicad_sch (KiCad schematic)
At the start: 2 parts

Commit message: POD start PCB
Parts:
- removed J?: Z80-Target, Package_DIP:DIP-40_W15.24mm, symbol AES_Library:Z80-Target-AES
- added J1: Z80-POD, AES_Library:CviLux_CF25401D0-05-NH_FFC-FPC-AES, symbol AES_Library:Z80-Pod-AES
- SKT1: renamed from J?; value ZID -> Z80 SOCKET PINS; footprint Connector_PinHeader_2.00mm:PinHeader_2x20_P2.00mm_Vertical -> Package_DIP:DIP-40_W15.24mm; PIN_NOTE BIDIRECTIONAL pins are OUT on Z80, IN on TARGET -> BIDIRECTIONAL pins are OUT on Z80, IN on DEBUGGER
Connections:
- net A0: now also J1.11 (A0)
- net A1: now also J1.10 (A1)
- net A10: now also J1.1 (A10)
- net A11: now also J1.40 (A11)
- net A12: now also J1.39 (A12)
- net A13: now also J1.38 (A13)
- net A14: now also J1.37 (A14)
- net A15: now also J1.36 (A15)
- net A2: now also J1.9 (A2)
- net A3: now also J1.8 (A3)
- net A4: now also J1.7 (A4)
- net A5: now also J1.6 (A5)
- net A6: now also J1.5 (A6)
- net A7: now also J1.4 (A7)
- net A8: now also J1.3 (A8)
- net A9: now also J1.2 (A9)
- net BACK-: now also J1.18 (~{BUSACK})
- net BREQ-: now also J1.16 (~{BUSREQ})
- net CLK: now also J1.35 (CLK)
- net D0: now also J1.27 (D0)
- net D1: now also J1.26 (D1)
- net D2: now also J1.29 (D2)
- net D3: now also J1.33 (D3)
- net D4: now also J1.34 (D4)
- net D5: now also J1.32 (D5)
- net D6: now also J1.31 (D6)
- net D7: now also J1.28 (D7)
- net GND: now also J1.12 (GND)
- net HALT-: now also J1.23 (~{HALT})
- net INT-: now also J1.25 (~{INT})
- net IORQ-: now also J1.21 (~{IORQ})
- net M1-: now also J1.14 (~{M1})
- net MREQ-: now also J1.22 (~{MREQ})
- net NMI-: now also J1.24 (~{NMI})
- net PWR: now also J1.30 (5V)
- net RD-: now also J1.20 (~{RD})
- net RFSH-: now also J1.13 (~{RFSH})
- net RST-: now also J1.15 (~{RESET})
- net WAIT-: now also J1.17 (~{WAIT})
- net WR-: now also J1.19 (~{WR})
