File: hw/ZID_POD/ZID_POD.kicad_pcb (KiCad board)
At the start: 2 copper layers, 2 parts, among them J1 Z80-POD

Commit message: POD-1 pcb
Parts:
- moved J1 31.5 mm to (116.7, 100.7), turned to 0 degrees
Routing:
- net /A11: track 0.00 -> 43.2 mm, vias 0 -> 1
- net /A12: track 0.00 -> 40.2 mm, vias 0 -> 1
- net /IORQ-: track 0.00 -> 37.6 mm, vias 0 -> 1
- net /A13: track 0.00 -> 37.1 mm, vias 0 -> 1
- net /MREQ-: track 0.00 -> 34.7 mm, vias 0 -> 2
- net /A14: track 0.00 -> 34.1 mm, vias 0 -> 1
- net /A15: track 0.00 -> 31.2 mm, vias 0 -> 1
- net /RD-: track 0.00 -> 31.2 mm, vias 0 -> 1
- net /HALT-: track 0.00 -> 31.0 mm, vias 0 -> 2
- net /WR-: track 0.00 -> 28.9 mm, vias 0 -> 1
- net /CLK: track 0.00 -> 28.4 mm, vias 0 -> 1
- net /BACK-: track 0.00 -> 27.3 mm, vias 0 -> 1
- net /NMI-: track 0.00 -> 27.2 mm, vias 0 -> 2
- net /INT-: track 0.00 -> 26.7 mm, vias 0 -> 2
- net /D1: track 0.00 -> 26.0 mm, vias 0 -> 2
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Other:
- board outline added: 52.8 x 19.3 mm
- board text added: "Copyright 2026, AESilky"
- board text added: "ZID CBL PIN-1"
