File: hw/ZID_MAIN/ZID_MAIN.kicad_sch (KiCad schematic)
At the start: 0 parts

Commit message: 8 output bits on RP. 10k PU for most. TVS.
Other:
- company: SilkyDESIGN -> SilkyDESIGN / CMOS1
Changed lines of the file:
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@@
 	(title_block
 		(title "Z80 In-Circuit Debugger (ZID)")
-		(date "2026-04-04")
+		(date "2026-04-05")
 		(rev "PR-1.0")
-		(company "SilkyDESIGN")
-		(comment 1 "Copyright 2026 AESilky")
+		(company "SilkyDESIGN / CMOS1")
+		(comment 1 "Copyright 2026 AESilky & SmM")
 	)
 	(sheet
