File: hw/ZID_MAIN/ZID_MAIN.kicad_sch (KiCad schematic)
At the start: 0 parts

Commit message: SCHM: Update CPLD pins and put all break units on board.
Parts:
- added C1, C2: 0.1u, Capacitor_SMD:C_0603_1608Metric_Pad1.08x0.95mm_HandSolder, symbol Device:C
- added C10, C11, C12, C13, C14, C15, C16, C17, C18, C19, C20, C21, C22, C23, C24, C25, C26, C27, C28, C29, C30, C31, C32, C33, C34, C35, C36, C37, C38, C39, C4, C40, C41, C42, C43, C44, C45, C46, C5, C6, C7, C8, C9: 0.1uF, Capacitor_SMD:C_0603_1608Metric, symbol Device:C_Small
- added C3: 100uF, Capacitor_SMD:C_1210_3225Metric_Pad1.33x2.70mm_HandSolder, symbol Device:C_Small
- added D1: BAT20J, Diode_SMD:D_SOD-323_HandSoldering, symbol AES_Library:AES-Schottky_Diode_PWR_Input
- added D2: SMAJ6.0A, Diode_SMD:D_SMA, symbol Diode:ESD5Zxx
- added D3, D4: PESD5V0L2U, Package_TO_SOT_SMD:SOT-323_SC-70, symbol Power_Protection:ESDA5V3L
- added H1, H2, H3, H4: MountingHole, MountingHole:MountingHole_3.2mm_M3, symbol Mechanical:MountingHole
- added J1: HDR 1x04 Socket, Connector_PinSocket_2.54mm:PinSocket_1x04_P2.54mm_Vertical, symbol Connector_Generic:Conn_01x04
- added J10: FFC/FPC-40 Socket, symbol Connector:Conn_01x40_Pin
- added J11: Conn_02x05_PINHDR_2.54mm, Connector_IDC:IDC-Header_2x05_P2.54mm_Vertical, symbol Connector_Generic:Conn_02x05_Odd_Even
- added J12: USB-C PWR ONLY, AES_Library:AES-USB_C-Molex-BdTopMnt-2171790001, symbol AES_Library:AES-USB-C-Amph_GSB1C46X
- added J2: Conn_02x03_Odd_Even, Connector_IDC:IDC-Header_2x03_P2.54mm_Vertical, symbol Connector_Generic:Conn_02x03_Odd_Even
- added J3: Conn_01x02_Pin_2.54mm, Connector_PinHeader_2.54mm:PinHeader_1x02_P2.54mm_Vertical, symbol Connector_Generic:Conn_01x02
- added J4: Conn_01x03, Connector_PinHeader_2.54mm:PinHeader_1x03_P2.54mm_Vertical, symbol Connector_Generic:Conn_01x03
- added J5, J6: Conn_01x08, Connector_PinHeader_2.54mm:PinHeader_1x08_P2.54mm_Vertical, symbol Connector_Generic:Conn_01x08
- added J7, J9: Conn_02x04_2.54mm, symbol Connector_Generic:Conn_02x04_Row_Letter_First
- added J8: Conn_02x04_2.54mm, symbol Connector_Generic:Conn_02x02_Row_Letter_First
- added JA1, JB1, JC1, JD1, JS1: SolderJumper_2_Open, symbol Jumper:SolderJumper_2_Open
- added JP1, JP3: Jumper_2_Small_Open_wsto-AES, Connector_PinHeader_2.00mm:PinHeader_1x03_P2.00mm_Vertical, symbol AES_Library:Jumper_2_Small_Open_wsto-AES
- added JP2: SolderJumper_2_Open, Jumper:SolderJumper-2_P1.3mm_Open_RoundedPad1.0x1.5mm, symbol Jumper:SolderJumper_2_Open
- added JP4, JP5, JP7: Jumper_2_Small_Bridged, Connector_PinHeader_2.00mm:PinHeader_1x02_P2.00mm_Vertical, symbol Jumper:Jumper_2_Small_Bridged
- added JP6: Jumper_2_Small_Open, Connector_PinHeader_2.00mm:PinHeader_1x02_P2.00mm_Vertical, symbol Jumper:Jumper_2_Small_Open
- added LED1, LED2, LED6: LED GREEN, LED_SMD:LED_0805_2012Metric, symbol Device:LED
- added LED10: LED BLUE, LED_SMD:LED_0805_2012Metric, symbol Device:LED
- added LED3, LED4, LED9: LED YELLOW, LED_SMD:LED_0805_2012Metric, symbol Device:LED
- added LED5, LED8: LED RED, LED_SMD:LED_0805_2012Metric, symbol Device:LED
- added LED7: LED ORANGE, LED_SMD:LED_0805_2012Metric, symbol Device:LED
- added M1: WS-RP2040-Zero, AES_Library:RP2040_WS-ZERO-AES, symbol AES_Library:RP2040_WS-AES
- added OP1, OP2, SBC1, SBC2, SBC3: AES-Option_A-B_2mm, Connector_PinHeader_2.00mm:PinHeader_1x03_P2.00mm_Vertical, symbol AES_Library:AES-Option_A-B_2mm
- added OP3: AES-Option_A-B, Connector_PinHeader_2.54mm:PinHeader_1x03_P2.54mm_Vertical, symbol AES_Library:AES-Option_A-B_2mm
- added R1: 18k, Resistor_SMD:R_0805_2012Metric, symbol Device:R_US
- added R10, R42: 0, Resistor_SMD:R_0805_2012Metric_Pad1.20x1.40mm_HandSolder, symbol Device:R_Small_US
- added R11, R13, R15, R17, R18: 820, Resistor_SMD:R_0805_2012Metric, symbol Device:R_Small_US
- added R12, R14, R16, R23, R24, R25, R31, R37, R8, R9: 10k, Resistor_SMD:R_0805_2012Metric, symbol Device:R_Small_US
- added R19, R20, R21, R22, R30, R33: 20k, Resistor_SMD:R_0805_2012Metric, symbol Device:R_Small_US
- added R2, R3: 6.8k, Resistor_SMD:R_0805_2012Metric, symbol Device:R_Small_US
- added R26, R27, R28, R4, R40, R41, R5, R6, R7: 4.7k, Resistor_SMD:R_0805_2012Metric, symbol Device:R_Small_US
- added R29, R32, R34, R36, R39: 1.2k, Resistor_SMD:R_0805_2012Metric, symbol Device:R_Small_US
- added R35, R38: 22, Resistor_SMD:R_0805_2012Metric, symbol Device:R_Small_US
- added RN1: 20k, Resistor_THT:R_Array_SIP9, symbol Device:R_Network08_US
- added SD1: SD-CARD Socket, AES_Library:AES-SDCard-GCT_MEM2075-00-140-01-A, symbol AES_Library:SD-Card-SPI-AES
- added SPARE1: ~, AES_Library:SPARE-and-SOIC-16-AES, symbol AES_Library:SPARE-16-AES
- added SW1: SW_Push, AES_Library:AES-SW_PUSH_SMD_1P1T_NO_6x6mm, symbol Switch:SW_Push
- added SW2: SW_DIP_x02, Button_Switch_THT:SW_DIP_SPSTx02_Piano_CTS_Series194-2MSTN_W7.62mm_P2.54mm, symbol Switch:SW_DIP_x02
- added TP1, TP10, TP11, TP12, TP13, TP14, TP15, TP16, TP17, TP18, TP19, TP2, TP20, TP21, TP22, TP23, TP24, TP25, TP26, TP27, TP3, TP4, TP5, TP6, TP9: TestPoint, Connector_PinHeader_2.54mm:PinHeader_1x01_P2.54mm_Vertical, symbol Connector:TestPoint
- added TP7: SYNC-CONN, Connector_PinHeader_2.54mm:PinHeader_1x01_P2.54mm_Vertical, symbol Connector:TestPoint_Alt
- added TP8: EXT-BRK(low actv), Connector_PinHeader_2.54mm:PinHeader_1x01_P2.54mm_Vertical, symbol Connector:TestPoint_Alt
- added U1: OSC-20MHz, AES_Library:OSC-8_14-AES, symbol AES_Library:OSC-8_14CAN-AES
- added U10: 74LVC2G04, Package_TO_SOT_SMD:SOT-23-6, symbol AES_Library:74LVC2G04-AES
- added U11: 74LVC125AS, Package_SO:SOIC-14_3.9x8.7mm_P1.27mm, symbol 74xx:74LVC125
- added U12: 74LVC273, Package_SO:SOIC-20W_7.5x12.8mm_P1.27mm, symbol AES_Library:74273-AES
- added U13, U2, U7: 74FCT2245, Package_SO:SOIC-20W_7.5x12.8mm_P1.27mm, symbol AES_Library:74245-AES
- added U14: AS7C1024B-10J, Package_SO:SOJ-32_10.16x20.955mm_P1.27mm, symbol Memory_RAM:AS7C1024B-xxJ
- added U15, U16, U18: 74FCT2245, Package_SO:SOIC-20W_7.5x12.8mm_P1.27mm, symbol AES_Library:74245_BA-AES
- added U17, U22: 74HCT166, Package_SO:SOIC-16_3.9x9.9mm_P1.27mm, symbol AES_Library:74166-AES
- added U19: ATF1508AS, Package_QFP:TQFP-100_14x14mm_P0.5mm, symbol AES_Library:ATF1508AS-AES
- added U20: 74FCT257T, Package_SO:SOIC-16W_7.5x10.3mm_P1.27mm, symbol 74xx:74LS257
- added U21: 74HCT161, Package_SO:SOIC-16_3.9x9.9mm_P1.27mm, symbol AES_Library:74161-AES
- added U23: 74AHCT00, Package_SO:SOIC-14_3.9x8.7mm_P1.27mm, symbol 74xx:74HCT00
- added U24: 74AHCT244, Package_SO:SOIC-20W_7.5x12.8mm_P1.27mm, symbol AES_Library:74244_OI-AES
- added U25, U26, U27, U28: ATF1504AS-44T, Package_QFP:TQFP-44_10x10mm_P0.8mm, symbol AES_Library:ATF1504AS-44T-AES
- added U3: 24LC32, Package_SO:SOIC-8_3.9x4.9mm_P1.27mm, symbol Memory_EEPROM:24LC32
- added U4: MIC2775, Package_TO_SOT_SMD:SOT-23-5, symbol AES_Library:MIC2775-AES
- added U5: SST39SF010, Package_DIP:DIP-32_W15.24mm_Socket_LongPads, symbol Memory_Flash:SST39SF010
- added U6: 74LVC245, Package_SO:SOIC-20W_7.5x12.8mm_P1.27mm, symbol AES_Library:74245-AES
- added U8: 74HCT14, symbol 74xx:74HC14
- added U9: Z80 C20MHz-PLCC, Package_LCC:PLCC-44, symbol AES_Library:Z84C0020V-AES
Connections:
- new net: JS1.2 (B), TP26.1, U8.13
- new net: LED4.1 (K), R17.1
- new net: LED4.2 (A), U12.16 (Q6)
- new net: OP2.3 (B), R24.2
- new net: U10.3, U12.6 (Q2)
- new net: LED7.2 (A), U23.6
- new net: TP27.1, U8.12
- new net: LED5.2 (A), R18.1
- new net: J3.2 (Pin_2), SW1.2, U4.4 (~{MR})
- new net: U17.13 (Qh), U22.1 (Ds)
- new net: R37.2, R38.1, TP8.1
- new net: LED1.1 (K), R11.1
- new net: OP1.2 (C), U20.10 (I1d)
- new net: LED2.1 (K), R13.1
- new net: LED2.2 (A), U12.12 (Q4)
- new net: JP4.1 (A), M1.23 (VBUS)
- new net: R10.2, SD1.10 (SHLD)
- new net: LED10.1 (K), R39.1
- new net: LED3.1 (K), R15.1
- new net: LED3.2 (A), U12.15 (Q5)
- new net: D1.1 (K), JP4.2 (B)
- new net: LED6.1 (K), R29.1
- new net: JP2.2 (B), R1.2, U3.1 (A0)
- new net: LED5.1 (K), U12.19 (Q7)
- new net: LED6.2 (A), U23.3
- new net: R38.2, U8.5
- new net: OP3.3 (B), U8.6, U8.9
- new net: LED9.1 (K), R36.1
- new net: JP5.2 (B), R14.2, U9.30 (~{RESET})
- new net: R35.1, TP7.1
- new net: J12.A4_B9 (VBUS), J12.B4_A9 (VBUS), JP7.1 (A)
- new net: J12.SH1 (SHIELD), J12.SH2 (SHIELD), J12.SH3 (SHIELD), J12.SH4 (SHIELD), R42.1
- new net: OP3.1 (A), U8.8
- new net: LED8.1 (K), R34.1
- new net: R23.2, U21.10 (CET), U21.3 (D0), U21.4 (D1), U21.5 (D2), U21.6 (D3), U21.9 (~{PE})
- new net: LED9.2 (A), U23.11
- new net: U10.1, U12.5 (Q1)
- new net: LED8.2 (A), U23.8
- new net: LED7.1 (K), R32.1
- new net: R35.2, U8.4
- new net: LED1.2 (A), U12.9 (Q3)
- new net +3.3V: C1.1, C2.2, C4.2, C5.2, C6.2, C7.2, J1.1 (Pin_1), J2.2 (Pin_2), M1.21 (3V3), R1.1, R12.1, R18.2, R2.2, R3.2, R4.2, R5.2, R6.2, R7.2, SD1.4 (VDD), U10.5 (VCC), U11.14 (VCC), U12.20 (VCC), U3.8 (VCC), U6.20 (VCC)
- new net +5V: C10.2, C11.2, C12.2, C13.2, C14.2, C15.2, C16.2, C17.2, C18.2, C19.2, C20.2, C21.2, C22.2, C23.2, C24.2, C25.2, C26.2, C27.2, C28.2, C29.2, C3.1, C30.2, C31.2, C32.2, C33.2, C34.2, C35.2, C36.2, C37.2, C38.2, C39.2, C40.2, C41.2, C42.2, C43.2, C44.2, C45.2, C46.2, C8.2, C9.2, D1.2 (A), D2.1 (K), J11.4 (Pin_4), J8.a1 (Pin_a1), J8.a2 (Pin_a2), J8.b1 (Pin_b1), J8.b2 (Pin_b2), J9.b4 (Pin_b4), JP7.2 (B), LED10.2 (A), R14.1, R16.2, R19.1, R20.1, R21.1, R22.1, R23.1, R24.1, R25.1, R26.1, R27.1, R28.1, R30.2, R31.2, R33.2, R37.1, R40.1, R41.1, R8.1, R9.1, RN1.1 (common), U1.1 (EN), U1.14 (PWR), U13.20 (VCC), U14.32 (VCC), U15.20 (VCC), U16.20 (VCC), U17.16 (VCC), U18.20 (VCC), U19.18 (VCCIO), U19.3 (VCCIO), U19.34 (VCCIO), U19.39 (VCCINT), U19.51 (VCCIO), U19.66 (VCCIO), U19.82 (VCCIO), U19.91 (VCCINT), U2.20 (VCC), U20.16 (VCC), U21.16 (VCC), U22.16 (VCC), U23.14 (VCC), U24.20 (VCC), U25.17 (VCCINT), U25.29 (VCCINT), U25.41 (VCCINT), U25.9 (VCCINT), U26.17 (VCCINT), U26.29 (VCCINT), U26.41 (VCCINT), U26.9 (VCCINT), U27.17 (VCCINT), U27.29 (VCCINT), U27.41 (VCCINT), U27.9 (VCCINT), U28.17 (VCCINT), U28.29 (VCCINT), U28.41 (VCCINT), U28.9 (VCCINT), U4.5 (VDD), U5.32 (VCC), U7.20 (VCC), U8.14 (VCC), U9.13 (V_{CC})
- new net ADDR_DOA: U25.3 (AMC4/IO), U26.6 (AMC1/IO)
- new net ADDR_DOB: U26.3 (AMC4/IO), U27.6 (AMC1/IO)
- new net ADDR_DOC: U27.3 (AMC4/IO), U28.6 (AMC1/IO)
- new net ADDR_DOD: TP11.1, U28.3 (AMC4/IO)
- new net AEN_CLK: U19.92 (AMC16/IO), U25.40 (IN/OE2/GCK2), U26.40 (IN/OE2/GCK2), U27.40 (IN/OE2/GCK2), U28.40 (IN/OE2/GCK2)
- new net AEN_CLR-: U19.94 (AMC13/IO), U25.39 (IN/GCLR), U26.39 (IN/GCLR), U27.39 (IN/GCLR), U28.39 (IN/GCLR)
- new net ATTN: U12.2 (Q0), U19.85 (H128/IO/GCK3)
- new net BA_CLK: U19.97 (AMC9/IO), U25.37 (IN/GCK1), U26.37 (IN/GCK1), U27.37 (IN/GCK1), U28.37 (IN/GCK1)
- new net BA_CLR-: U19.98 (AMC8/IO), U25.35 (D41/IO/GCK3), U26.35 (D41/IO/GCK3), U27.35 (D41/IO/GCK3), U28.35 (D41/IO/GCK3)
- new net BRD_RST-: SBC2.2 (C), U19.67 (GMC102/IO)
- new net BRK1_AEQ-: U19.64 (GMC99/IO), U25.43 (AMC14/IO)
- new net BRK2N_AEQ-: R40.2, U19.40 (EMC65/IO), U25.42 (AMC16/IO), U26.42 (AMC16/IO), U26.43 (AMC14/IO), U27.42 (AMC16/IO), U27.43 (AMC14/IO), U28.42 (AMC16/IO), U28.43 (AMC14/IO)
- new net BRKHW_DET-: R41.2, U19.23 (CMC37/IO), U25.44 (AMC11/IO), U25.5 (A3/IO/PD1), U26.44 (AMC11/IO), U26.5 (A3/IO/PD1), U27.44 (AMC11/IO), U27.5 (A3/IO/PD1), U28.44 (AMC11/IO), U28.5 (A3/IO/PD1)
- new net CLK: D3.1 (K), J10.6 (Pin_6), SBC1.2 (C), U19.87 (IN/GCK1), U9.7 (CLK)
- new net D7_B: U19.84 (HMC126/IO), U25.38 (IN/OE1), U25.6 (AMC1/IO)
- new net ENBL_DOA: U25.2 (AMC5/IO), U26.38 (IN/OE1)
- new net ENBL_DOB: U26.2 (AMC5/IO), U27.38 (IN/OE1)
- new net ENBL_DOC: U27.2 (AMC5/IO), U28.38 (IN/OE1)
- new net ENBL_DOD: TP10.1, U28.2 (AMC5/IO)
- new net EXTBRKRQ-: OP3.2 (C), U19.68 (GMC104/IO)
- new net FIXED_SEL: U19.83 (HMC125/IO), U20.1 (S)
- new net GND: C1.2, C10.1, C11.1, C12.1, C13.1, C14.1, C15.1, C16.1, C17.1, C18.1, C19.1, C2.1, C20.1, C21.1, C22.1, C23.1, C24.1, C25.1, C26.1, C27.1, C28.1, C29.1, C3.2, C30.1, C31.1, C32.1, C33.1, C34.1, C35.1, C36.1, C37.1, C38.1, C39.1, C4.1, C40.1, C41.1, C42.1, C43.1, C44.1, C45.1, C46.1, C5.1, C6.1, C7.1, C8.1, C9.1, D2.2 (A), D3.3 (A), D4.3 (A), J1.2 (Pin_2), J10.5 (Pin_5), J10.7 (Pin_7), J11.10 (Pin_10), J11.2 (Pin_2), J12.A1_B12 (GND), J12.B1_A12 (GND), J2.6 (Pin_6), J3.1 (Pin_1), J4.1 (Pin_1), J5.1 (Pin_1), J7.b1 (Pin_b1), J7.b2 (Pin_b2), J7.b3 (Pin_b3), J7.b4 (Pin_b4), J9.b1 (Pin_b1), J9.b2 (Pin_b2), J9.b3 (Pin_b3), JP2.1 (A), JS1.1 (A), M1.22 (GND), R10.1, R11.2, R13.2, R15.2, R17.2, R29.2, R32.2, R34.2, R36.2, R39.2, R42.2, SBC3.3 (B), SD1.6 (GND), SW1.1, SW2.1, SW2.2, TP9.1, U1.4 (G), U1.7 (G), U10.2 (GND), U11.1, U11.10, U11.13, U11.4, U11.7 (GND), U12.10 (GND), U13.10 (GND), U14.16 (GND), U15.1 (A>B), U15.10 (GND), U15.19 (~{OE}), U16.1 (A>B), U16.10 (GND), U16.19 (~{OE}), U17.1 (Ds), U17.6 (~{CE}), U17.8 (GND), U18.1 (A>B), U18.10 (GND), U18.19 (~{OE}), U19.11 (GND), U19.26 (GND), U19.38 (GND), U19.43 (GND), U19.59 (GND), U19.74 (GND), U19.86 (GND), U19.95 (GND), U2.10 (GND), U20.8 (GND), U21.8 (GND), U22.6 (~{CE}), U22.8 (GND), U23.7 (GND), U24.10 (GND), U24.19 (~{OEb}), U25.16 (GND), U25.24 (GND), U25.36 (GND), U25.4 (GND), U26.16 (GND), U26.24 (GND), U26.36 (GND), U26.4 (GND), U27.16 (GND), U27.24 (GND), U27.36 (GND), U27.4 (GND), U28.16 (GND), U28.24 (GND), U28.36 (GND), U28.4 (GND), U3.2 (A1), U3.3 (A2), U3.4 (GND), U3.7 (WP), U4.2 (GND), U5.1 (NC), U5.16 (GND), U5.30 (NC), U6.10 (GND), U7.10 (GND), U8.7 (GND), U9.33 (GND)
- new net GPI_A-: TP23.1, U26.33 (DMC57/IO)
- new net GPI_B-: TP24.1, TP25.1, U27.33 (DMC57/IO), U28.33 (DMC57/IO)
- new net GPO_A-: TP20.1, U26.34 (DMC62/IO)
- new net GPO_B-: TP21.1, TP22.1, U27.34 (DMC62/IO), U28.34 (DMC62/IO)
- new net I88: TP2.1, U19.88 (IN/OE1)
- new net IO10A: TP16.1, U25.10 (BMC25/IO)
- new net IO10B: TP17.1, U26.10 (BMC25/IO)
- new net IO10C: TP18.1, U27.10 (BMC25/IO)
- new net IO10D: TP19.1, U28.10 (BMC25/IO)
- new net IO77: TP5.1, U19.77 (HMC117/IO)
- new net IO78: TP4.1, U19.78 (HMC118/IO)
- new net IO8A: TP12.1, U25.8 (BMC30/IO)
- new net IO8B: TP13.1, U26.8 (BMC30/IO)
- new net IO8C: TP14.1, U27.8 (BMC30/IO)
- new net IO8D: TP15.1, U28.8 (BMC30/IO)
- new net IOECLK: M1.16 (GP15), U12.11 (Cp)
- new net JTCK: J11.1 (Pin_1), R26.2, U19.62 (F96/IO/JT.TCK), U25.26 (C48/IO/JT.TCK), U26.26 (C48/IO/JT.TCK), U27.26 (C48/IO/JT.TCK), U28.26 (C48/IO/JT.TCK)
- new net JTD1O2I: JA1.1 (A), U19.73 (G112/IO/JT.TDO), U25.1 (A8/IO/JT.TDI)
- new net JTD2O3I: JB1.1 (A), U25.32 (D56/IO/JT.TDO), U26.1 (A8/IO/JT.TDI)
- new net JTD3O4I: JC1.1 (A), U26.32 (D56/IO/JT.TDO), U27.1 (A8/IO/JT.TDI)
- new net JTD4O5I: JD1.1 (A), U27.32 (D56/IO/JT.TDO), U28.1 (A8/IO/JT.TDI)
- new net JTDI_CO: J11.9 (Pin_9), R28.2, U19.4 (B32/IO/JT.TDI)
- new net JTDO_CI: J11.3 (Pin_3), R25.2
- new net JTD_CBLI: JA1.2 (B), JB1.2 (B), JC1.2 (B), JD1.2 (B), U28.32 (D56/IO/JT.TDO)
- new net JTMS: J11.5 (Pin_5), R27.2, U19.15 (C48/IO/JT.TMS), U25.7 (B32/IO/JT.TMS), U26.7 (B32/IO/JT.TMS), U27.7 (B32/IO/JT.TMS), U28.7 (B32/IO/JT.TMS)
- new net LA0: U15.2 (A0), U25.11 (BMC24/IO), U26.11 (BMC24/IO), U27.11 (BMC24/IO), U28.11 (BMC24/IO)
- new net LA1: U15.3 (A1), U25.12 (BMC21/IO), U26.12 (BMC21/IO), U27.12 (BMC21/IO), U28.12 (BMC21/IO)
- new net LA10: U18.4 (A2), U25.23 (CMC41/IO), U26.23 (CMC41/IO), U27.23 (CMC41/IO), U28.23 (CMC41/IO)
- new net LA11: U18.5 (A3), U25.25 (CMC46/IO), U26.25 (CMC46/IO), U27.25 (CMC46/IO), U28.25 (CMC46/IO)
- new net LA12: U18.6 (A4), U25.27 (DMC49/IO), U26.27 (DMC49/IO), U27.27 (DMC49/IO), U28.27 (DMC49/IO)
- new net LA13: U18.7 (A5), U25.28 (DMC51/IO), U26.28 (DMC51/IO), U27.28 (DMC51/IO), U28.28 (DMC51/IO)
- new net LA14: U18.8 (A6), U25.30 (DMC52/IO), U26.30 (DMC52/IO), U27.30 (DMC52/IO), U28.30 (DMC52/IO)
- new net LA15: U18.9 (A7), U25.31 (DMC53/IO), U26.31 (DMC53/IO), U27.31 (DMC53/IO), U28.31 (DMC53/IO)
- new net LA2: U15.4 (A2), U25.13 (BMC20/IO), U26.13 (BMC20/IO), U27.13 (BMC20/IO), U28.13 (BMC20/IO)
- new net LA3: U15.5 (A3), U25.14 (BMC19/IO), U26.14 (BMC19/IO), U27.14 (BMC19/IO), U28.14 (BMC19/IO)
- new net LA4: U15.6 (A4), U25.15 (BMC17/IO), U26.15 (BMC17/IO), U27.15 (BMC17/IO), U28.15 (BMC17/IO)
- new net LA5: U15.7 (A5), U25.18 (CMC33/IO), U26.18 (CMC33/IO), U27.18 (CMC33/IO), U28.18 (CMC33/IO)
- new net LA6: U15.8 (A6), U25.19 (C35/IO/PD2), U26.19 (C35/IO/PD2), U27.19 (C35/IO/PD2), U28.19 (C35/IO/PD2)
- new net LA7: U15.9 (A7), U25.20 (CMC36/IO), U26.20 (CMC36/IO), U27.20 (CMC36/IO), U28.20 (CMC36/IO)
- new net LA8: U18.2 (A0), U25.21 (CMC37/IO), U26.21 (CMC37/IO), U27.21 (CMC37/IO), U28.21 (CMC37/IO)
- new net LA9: U18.3 (A1), U25.22 (CMC40/IO), U26.22 (CMC40/IO), U27.22 (CMC40/IO), U28.22 (CMC40/IO)
- new net LCL_IO: TP6.1, U19.33 (DMC54/IO)
- new net LRST-: U11.12, U19.71 (GMC109/IO), U23.10, U23.13, U23.2, U23.5
- new net MA0: M1.11 (GP10), U11.6
- new net MEMOP-: U19.60 (FMC93/IO), U21.2 (CP)
- new net MINT-: U10.6, U25.33 (DMC57/IO)
- new net MODINT-: J9.a4 (Pin_a4), JP6.1 (A), U25.34 (DMC62/IO)
- new net MOD_SEL-: U11.2, U19.96 (AMC11/IO), U6.19 (~{OE})
- new net MRD-: M1.12 (GP11), U11.8
- new net MRST-: M1.15 (GP14), U11.11, U12.1 (~{Mr})
- new net MSEL-: M1.13 (GP12), U11.3
- new net MWTRQ-: M1.14 (GP13), R12.2, U19.8 (BMC25/IO)
- new net PCRD_DIN: U19.21 (CMC40/IO), U22.13 (Qh)
- new net PCSAV_CLK: U17.7 (Clk), U19.69 (GMC105/IO), U22.7 (Clk)
- new net PU: OP1.1 (A), R31.1, U14.30 (CS2/CE2), U17.9 (~{Clr}), U20.13 (I1c), U20.3 (I1a), U20.6 (I1b), U22.9 (~{Clr})
- new net RAM_SEL-: U14.22 (~{CS1}/~{CE1}), U19.32 (DMC56/IO)
- new net RFMR-: OP1.3 (B), U19.35 (DMC53/IO)
- new net ROM_SEL: U19.27 (DMC64/IO), U8.1
- new net ROM_SEL-: U5.22 (CE), U8.2
- new net RRA0: U14.3 (A14), U19.29 (DMC61/IO), U5.29 (A14)
- new net RRA1: U14.31 (A15), U19.28 (DMC62/IO), U5.3 (A15)
- new net RRA2: U14.2 (A16), U19.30 (DMC59/IO), U5.2 (A16)
- new net RST-: JP3.2 (B), SBC2.3 (B), U4.1 (~{RST})
- new net SBCMODE-: R16.1, SBC3.2 (C), U19.24 (CMC35/IO)
- new net SBC_GPI0: U16.6 (A4), U19.55 (FMC86/IO)
- new net SBC_GPI1: U16.7 (A5), U19.56 (FMC88/IO)
- new net SBC_GPI2: U16.8 (A6), U19.22 (CMC38/IO)
- new net SBC_GPI3: R9.2, SW2.3, U19.20 (CMC41/IO)
- new net SBC_GPO0: U16.18 (B0), U19.17 (CMC45/IO)
- new net SBC_GPO1: U16.17 (B1), U19.16 (CMC46/IO)
- new net SBC_GPO2: U16.16 (B2), U19.46 (EMC73/IO)
- new net SBC_GPO3: U16.15 (B3), U19.47 (EMC75/IO)
- new net SBC_I0: J9.a1 (Pin_a1), U16.14 (B4)
- new net SBC_I1: J9.a2 (Pin_a2), U16.13 (B5)
- new net SBC_I2: J9.a3 (Pin_a3), U16.12 (B6)
- new net SBC_O0: J7.a1 (Pin_a1), U16.2 (A0)
- new net SBC_O1: J7.a2 (Pin_a2), U16.3 (A1)
- new net SBC_O2: J7.a3 (Pin_a3), U16.4 (A2)
- new net SBC_O3: J7.a4 (Pin_a4), U16.5 (A3)
- new net SCK_RX: J1.3 (Pin_3), M1.2 (GP1), R2.1, U3.6 (SCL)
- new net SDA_TX: J1.4 (Pin_4), M1.1 (GP0), R3.1, U3.5 (SDA)
- new net SOPNOW: U19.53 (FMC83/IO), U21.12 (Q2)
- new net SPICK: J2.3 (Pin_3), M1.17 (GP26), R5.1, SD1.5 (CLK)
- new net SPICS-: J4.2 (Pin_2), M1.20 (GP29), R6.1, SD1.2 (CS)
- new net SPICS2-: J2.5 (Pin_5), U10.4
- new net SPIMI: J2.1 (Pin_1), J4.3 (Pin_3), M1.19 (GP28), R7.1, SD1.7 (MISO)
- new net SPIMO: J2.4 (Pin_4), M1.18 (GP27), R4.1, SD1.3 (MOSI)
- new net SYNC: U19.37 (DMC49/IO), U8.3
- new net TA0: J10.30 (Pin_30), U2.11 (B7)
- new net TA1: J10.31 (Pin_31), U2.12 (B6)
- new net TA10: J10.40 (Pin_40), U7.13 (B5)
- new net TA11: J10.1 (Pin_1), U7.14 (B4)
- new net TA12: J10.2 (Pin_2), U7.15 (B3)
- new net TA13: J10.3 (Pin_3), U7.16 (B2)
- new net TA14: J10.4 (Pin_4), U7.17 (B1)
- new net TA15: J10.29 (Pin_29), U7.18 (B0)
- new net TA2: J10.32 (Pin_32), U2.13 (B5)
- new net TA3: J10.33 (Pin_33), U2.14 (B4)
- new net TA4: J10.34 (Pin_34), U2.15 (B3)
- new net TA5: J10.35 (Pin_35), U2.16 (B2)
- new net TA6: J10.36 (Pin_36), U2.17 (B1)
- new net TA7: J10.37 (Pin_37), U2.18 (B0)
- new net TA8: J10.38 (Pin_38), U7.11 (B7)
- new net TA9: J10.39 (Pin_39), U7.12 (B6)
- new net TBREQ-: J10.25 (Pin_25), R22.2, U24.13 (I1b)
- new net TBREQB-: U19.65 (GMC101/IO), U24.7 (O1b)
- new net TCLK: JP1.3 (C), SBC1.1 (A)
- new net TD0: J10.14 (Pin_14), J6.1 (Pin_1), U13.18 (B0)
- new net TD1: J10.15 (Pin_15), J6.2 (Pin_2), U13.17 (B1)
- new net TD2: J10.12 (Pin_12), J6.3 (Pin_3), U13.16 (B2)
- new net TD3: J10.8 (Pin_8), J6.4 (Pin_4), U13.15 (B3)
- new net TD4: J10.11 (Pin_11), J6.5 (Pin_5), U13.14 (B4)
- new net TD5: J10.9 (Pin_9), J6.6 (Pin_6), U13.13 (B5)
- new net TD6: J10.10 (Pin_10), J6.7 (Pin_7), U13.12 (B6)
- new net TD7: J10.13 (Pin_13), J6.8 (Pin_8), U13.11 (B7)
- new net TDBUSEN-: U13.19 (~{OE}), U19.81 (HMC123/IO)
- new net TDBUSIN-: U13.1 (A>B), U19.61 (FMC94/IO)
- new net TGTGO: U19.48 (EMC77/IO), U21.7 (CEP)
- new net TGTMODE-: U17.15 (~{LD}), U19.36 (DMC51/IO), U21.1 (~{MR}), U22.15 (~{LD}), U23.1
- new net TGTNOW: U19.54 (FMC85/IO), U21.15 (TC)
- new net TGTONLY-: R8.2, SW2.4, U19.76 (HMC115/IO)
- new net TINT-: J10.16 (Pin_16), JP6.2 (B), R19.2, U24.15 (I2b)
- new net TINTB-: U19.75 (HMC113/IO), U24.5 (O2b)
- new net TIORQ-: J10.20 (Pin_20), U20.12 (Zc), U24.6 (I2a)
- new net TM1-: J10.27 (Pin_27), U16.9 (A7)
- new net TMREQ-: J10.19 (Pin_19), U20.9 (Zd), U24.8 (I3a)
- new net TNMI-: J10.17 (Pin_17), R20.2, U24.11 (I0b)
- new net TNMIB-: U19.63 (GMC97/IO), U24.9 (O0b)
- new net TRD-: J10.21 (Pin_21), U20.7 (Zb), U24.4 (I1a)
- new net TRST-: D4.1 (K), J10.26 (Pin_26), JP3.3 (C), SBC2.1 (A)
- new net TWAIT-: J10.24 (Pin_24), R21.2, U23.12, U24.17 (I3b)
- new net TWAITB-: OP2.1 (A), U24.3 (O3b)
- new net TWAITRQ-: OP2.2 (C), U19.41 (E67/IO/PD2)
- new net TWR-: J10.22 (Pin_22), U20.4 (Za), U24.2 (I0a)
- new net V3D0: M1.3 (GP2), U12.3 (D0), U6.18 (B0)
- new net V3D1: M1.4 (GP3), U12.4 (D1), U6.17 (B1)
- new net V3D2: M1.5 (GP4), U12.7 (D2), U6.16 (B2)
- new net V3D3: M1.6 (GP5), U12.8 (D3), U6.15 (B3)
- new net V3D4: M1.7 (GP6), U12.13 (D4), U6.14 (B4)
- new net V3D5: M1.8 (GP7), U12.14 (D5), U6.13 (B5)
- new net V3D6: M1.9 (GP8), U12.17 (D6), U6.12 (B6)
- new net V3D7: M1.10 (GP9), U12.18 (D7), U6.11 (B7)
- new net ZA0: U11.5, U14.12 (A0), U15.18 (B0), U2.9 (A7), U22.14 (H), U5.12 (A0), U9.34 (A_{0})
- new net ZA1: U14.11 (A1), U15.17 (B1), U19.1 (A3/IO/PD1), U2.8 (A6), U22.12 (G), U5.11 (A1), U9.35 (A_{1})
- new net ZA10: RN1.4 (R3), U14.23 (A10), U17.11 (F), U18.16 (B2), U5.23 (A10), U7.7 (A5), U9.44 (A_{10})
- new net ZA11: RN1.3 (R2), U14.25 (A11), U17.10 (E), U18.15 (B3), U5.25 (A11), U7.6 (A4), U9.1 (A_{11})
- new net ZA12: RN1.2 (R1), U14.4 (A12), U17.5 (D), U18.14 (B4), U5.4 (A12), U7.5 (A3), U9.2 (A_{12})
- new net ZA13: RN1.6 (R5), U14.28 (A13), U17.4 (C), U18.13 (B5), U5.28 (A13), U7.4 (A2), U9.3 (A_{13})
- new net ZA14: RN1.8 (R7), U17.3 (B), U18.12 (B6), U19.10 (BMC22/IO), U7.3 (A1), U9.4 (A_{14})
- new net ZA15: RN1.9 (R8), U17.2 (A), U18.11 (B7), U19.9 (BMC24/IO), U7.2 (A0), U9.5 (A_{15})
- new net ZA2: U14.10 (A2), U15.16 (B2), U19.19 (CMC43/IO), U2.7 (A5), U22.11 (F), U5.10 (A2), U9.36 (A_{2})
- new net ZA3: U14.9 (A3), U15.15 (B3), U19.14 (BMC17/IO), U2.6 (A4), U22.10 (E), U5.9 (A3), U9.37 (A_{3})
- new net ZA4: U14.8 (A4), U15.14 (B4), U19.13 (BMC19/IO), U2.5 (A3), U22.5 (D), U5.8 (A4), U9.38 (A_{4})
- new net ZA5: U14.7 (A5), U15.13 (B5), U19.44 (EMC70/IO), U2.4 (A2), U22.4 (C), U5.7 (A5), U9.39 (A_{5})
- new net ZA6: U14.6 (A6), U15.12 (B6), U19.45 (EMC72/IO), U2.3 (A1), U22.3 (B), U5.6 (A6), U9.40 (A_{6})
- new net ZA7: U14.5 (A7), U15.11 (B7), U19.52 (FMC81/IO), U2.2 (A0), U22.2 (A), U5.5 (A7), U9.41 (A_{7})
- new net ZA8: RN1.7 (R6), U14.27 (A8), U17.14 (H), U18.18 (B0), U5.27 (A8), U7.9 (A7), U9.42 (A_{8})
- new net ZA9: RN1.5 (R4), U14.26 (A9), U17.12 (G), U18.17 (B1), U5.26 (A9), U7.8 (A6), U9.43 (A_{9})
- new net ZBACK: U20.15 (OE), U8.10
- new net ZBACK-: D3.2 (K), J10.23 (Pin_23), R30.1, U19.57 (FMC89/IO), U2.1 (A>B), U23.4, U24.1 (~{OEa}), U7.1 (A>B), U8.11, U9.27 (~{BUSACK})
- new net ZBREQ-: U19.70 (GMC107/IO), U9.29 (~{BUSREQ})
- new net ZD0: U13.2 (A0), U14.13 (I/O0), U19.6 (BMC29/IO), U5.13 (D0), U6.2 (A0), U9.16 (D_{0})
- new net ZD1: U13.3 (A1), U14.14 (I/O1), U19.93 (AMC14/IO), U5.14 (D1), U6.3 (A1), U9.17 (D_{1})
- new net ZD2: U13.4 (A2), U14.15 (I/O2), U19.100 (AMC5/IO), U5.15 (D2), U6.4 (A2), U9.14 (D_{2})
- new net ZD3: U13.5 (A3), U14.17 (I/O3), U19.99 (AMC6/IO), U5.17 (D3), U6.5 (A3), U9.9 (D_{3})
- new net ZD4: U13.6 (A4), U14.18 (I/O4), U19.50 (EMC80/IO), U5.18 (D4), U6.6 (A4), U9.8 (D_{4})
- new net ZD5: U13.7 (A5), U14.19 (I/O5), U19.49 (EMC78/IO), U5.19 (D5), U6.7 (A5), U9.10 (D_{5})
- new net ZD6: U13.8 (A6), U14.20 (I/O6), U19.5 (BMC30/IO), U5.20 (D6), U6.8 (A6), U9.11 (D_{6})
- new net ZD7: U13.9 (A7), U14.21 (I/O7), U19.7 (BMC27/IO), U5.21 (D7), U6.9 (A7), U9.15 (D_{7})
- new net ZHALT-: J10.18 (Pin_18), R33.1, U23.9, U9.20 (~{HALT})
- new net ZINT-: U19.80 (HMC121/IO), U9.18 (~{INT})
- new net ZIORQ-: J5.5 (Pin_5), U19.42 (EMC69/IO), U20.14 (I0c), U24.14 (O2a), U9.22 (~{IORQ})
- new net ZM1-: J5.3 (Pin_3), U16.11 (B7), U19.90 (IN/OE2/GCK2), U9.31 (~{M1})
- new net ZMREQ-: J5.4 (Pin_4), U19.89 (IN/GCLR), U20.11 (I0d), U24.12 (O3a), U9.21 (~{MREQ})
- new net ZNMI-: U19.58 (FMC91/IO), U9.19 (~{NMI})
- new net ZRD-: J5.6 (Pin_6), U11.9, U14.24 (~{OE}), U19.2 (AMC1/IO), U20.5 (I0b), U24.16 (O1a), U5.24 (OE), U6.1 (A>B), U9.23 (~{RD})
- new net ZRFSH-: D4.2 (K), J10.28 (Pin_28), J5.2 (Pin_2), U19.25 (CMC33/IO), U9.32 (~{RFSH})
- new net ZRST-: JP5.1 (A), U19.72 (GMC110/IO), U2.19 (~{OE}), U7.19 (~{OE})
- new net ZSPRSTRQ: TP3.1, U19.79 (HMC120/IO)
- new net ZWAIT-: J5.8 (Pin_8), U19.31 (DMC57/IO), U9.28 (~{WAIT})
- new net ZWR-: J5.7 (Pin_7), U14.29 (~{WE}), U19.12 (BMC21/IO), U20.2 (I0a), U24.18 (O0a), U5.31 (PGM), U9.26 (~{WR})
- new net _CLK: JP1.2 (B), SBC1.3 (B), TP1.1, U1.11 (O), U1.8 (O)
- no-connect marks 0 -> 19
Other:
- removed sheet Conn and Expand
- removed sheet Main Logic
- removed sheet hold
- note added: "3.3V Logic Section"
- note added: "Module provides 3.3V"
- note added: "{not Z80 pin}"

Commit message: SCHM: Updates per SM
Parts:
- U14: value AS7C1024B-10J -> AS7C1024B; symbol Memory_RAM:AS7C1024B-xxJ -> AES_Library:AS7C1024B_DIP32_SOP32-AES
- renumbered R41 to R40, R40 to R41
Other:
- moved on the sheet: R41, U14, U17, U22

Commit message: HW: Ready to lay out.
Parts:
- removed J10: FFC/FPC-40 Socket, symbol Connector:Conn_01x40_Pin
- removed R24: 10k, Resistor_SMD:R_0805_2012Metric, symbol Device:R_Small_US
- removed TP3: TestPoint, Connector_PinHeader_2.54mm:PinHeader_1x01_P2.54mm_Vertical, symbol Connector:TestPoint
- removed U24: 74AHCT244, Package_SO:SOIC-20W_7.5x12.8mm_P1.27mm, symbol AES_Library:74244_OI-AES
- added J10: FFC/FPC-40 Socket, AES_Library:CviLux_CF25401D0-05-NH_FFC-FPC-AES, symbol Connector_Generic:Conn_01x40
- added R23, R33, R38: 10k, Resistor_SMD:R_0805_2012Metric, symbol Device:R_Small_US
- added TP6: TestPoint, Connector_PinHeader_2.54mm:PinHeader_1x01_P2.54mm_Vertical, symbol Connector:TestPoint
- added U22: 74AHCT244, Package_SO:SOIC-20W_7.5x12.8mm_P1.27mm, symbol AES_Library:74244-AB-AES
- J7, J9: footprint (none) -> Connector_PinHeader_2.54mm:PinHeader_2x04_P2.54mm_Vertical
- J8: value Conn_02x04_2.54mm -> Conn_02x02_2.54mm; footprint (none) -> Connector_PinHeader_2.54mm:PinHeader_2x02_P2.54mm_Vertical
- JA1, JB1, JC1, JD1, JS1: footprint (none) -> Jumper:SolderJumper-2_P1.3mm_Open_TrianglePad1.0x1.5mm
- OP1: Function TGT-MREQ -> PASS-MREQ
- OP3: Function TGT-WAIT -> EXT-BRK; OP-A WAIT -> HIGH-T; OP-B NO WAIT -> LOW-T
- TP9: renamed from TP8; value EXT-BRK(low actv) -> EXT-BRK
- U8: footprint (none) -> Package_SO:SOIC-14_3.9x8.7mm_P1.27mm
- renumbered R23 to R24, R33 to R34, R34 to R35, R35 to R37, R37 to R40, R38 to R41, R40 to R42, R41 to R43, R42 to R44, TP4 to TP3, TP5 to TP4, TP6 to TP5, TP9 to TP8, U18 to U17, U19 to U18, U17 to U19, U22 to U23, U23 to U24
Connections:
- net ZSPRSTRQ is gone; now on net BRKPC_RD-: U18.79 (HMC120/IO)
- net +5V: now also R23.2, R33.2, R38.2, U22.20 (VCC)
- net CLK: now also J10.6 (Pin_6)
- net EXTBRKRQ-: now also R38.1
- net GND: now also J10.5 (Pin_5), J10.7 (Pin_7), U22.10 (GND), U22.19 (~{OEb})
- net PU: no longer OP1.1 (A)
- net TA0: now also J10.30 (Pin_30)
- net TA1: now also J10.31 (Pin_31)
- net TA10: now also J10.40 (Pin_40)
- net TA11: now also J10.1 (Pin_1)
- net TA12: now also J10.2 (Pin_2)
- net TA13: now also J10.3 (Pin_3)
- net TA14: now also J10.4 (Pin_4)
- net TA15: now also J10.29 (Pin_29)
- net TA2: now also J10.32 (Pin_32)
- net TA3: now also J10.33 (Pin_33)
- net TA4: now also J10.34 (Pin_34)
- net TA5: now also J10.35 (Pin_35)
- net TA6: now also J10.36 (Pin_36)
- net TA7: now also J10.37 (Pin_37)
- net TA8: now also J10.38 (Pin_38)
- net TA9: now also J10.39 (Pin_39)
- net TBREQ-: now also J10.25 (Pin_25), U22.13 (I1b)
- net TBREQB-: now also U22.7 (O1b)
- net TD0: now also J10.14 (Pin_14)
- net TD1: now also J10.15 (Pin_15)
- net TD2: now also J10.12 (Pin_12)
- net TD3: now also J10.8 (Pin_8)
- net TD4: now also J10.11 (Pin_11)
- net TD5: now also J10.9 (Pin_9)
- net TD6: now also J10.10 (Pin_10)
- net TD7: now also J10.13 (Pin_13)
- net TGTMODE-: no longer U19.15 (~{LD}), U23.15 (~{LD})
- net TINT-: now also J10.16 (Pin_16), U22.15 (I2b)
- net TINTB-: now also U22.5 (O2b)
- net TIORQ-: now also J10.20 (Pin_20), U22.14 (O2a)
- net TM1-: now also J10.27 (Pin_27)
- net TMREQ-: now also J10.19 (Pin_19), U22.12 (O3a)
- net TNMI-: now also J10.17 (Pin_17), U22.11 (I0b)
- net TNMIB-: now also U22.9 (O0b)
- net TRD-: now also J10.21 (Pin_21), U22.16 (O1a)
- net TRST-: now also J10.26 (Pin_26)
- net TWAIT-: now also J10.24 (Pin_24), U22.17 (I3b)
- net TWAITB-: now also U22.3 (O3b)
- net TWAITRQ-: now also R33.1
- net TWR-: now also J10.22 (Pin_22), U22.18 (O0a)
- net ZBACK-: now also J10.23 (Pin_23), U22.1 (~{OEa})
- net ZHALT-: now also J10.18 (Pin_18)
- net ZIORQ-: now also U22.6 (I2a)
- net ZMREQ-: now also U22.8 (I3a)
- net ZRD-: now also U22.4 (I1a)
- net ZRFSH-: now also J10.28 (Pin_28)
- net ZWR-: now also U22.2 (I0a)
- net at OP1.2 (C), U20.10 (I1d): now also R23.1
- net at U8.6, U8.9: now also OP3.1 (A); no longer OP3.3 (B)
- net at U8.8: now also OP3.3 (B); no longer OP3.1 (A)
- net PCSAV_CLK renamed BRKPC_RD-
- net BRKPC_RD-: no longer U18.69 (GMC105/IO)
- net SOPNOW: no longer names the net of U21.12 (Q2)
- net SOPNOW: no longer U18.53 (FMC83/IO)
- new net IO83: TP6.1, U18.53 (FMC83/IO)
- new net PC_LATCH-: U18.69 (GMC105/IO), U19.15 (~{LD}), U23.15 (~{LD})
- no-connect marks 19 -> 22
Other:
- moved on the sheet: JS1, OP1, OP2, OP3, R37, R40, R41, SPARE1, TP26, TP27, TP7, TP9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
