File: hw/ZID_MAIN/ZID_MAIN.kicad_sch (KiCad schematic)
At the start: 199 parts, among them J1 HDR 1x04 Socket, J10 FFC/FPC-40 Socket, J11 Conn_02x05_PINHDR_2.54mm, J12 USB-C PWR ONLY, J2 Conn_02x03_Odd_Even, J3 Conn_01x02_Pin_2.54mm, J4 Conn_01x03, J5 Conn_01x08, J6 Conn_01x08, J7 Conn_02x04_2.54mm, J8 Conn_02x02_2.54mm, J9 Conn_02x04_2.54mm, M1 WS-RP2040-Zero, SW1 SW_Push, SW2 SW_DIP_x02, U1 OSC-20MHz, U10 74LVC2G04, U11 74LVC125AS, U12 74LVC273, U13 74FCT2245, U14 AS7C1024B, U15 74FCT2245, U16 74FCT2245, U17 74FCT2245, U18 ATF1508AS, U19 74HCT166, U2 74FCT2245, U20 74FCT257T, U21 74HCT161, U22 74AHCT244, U23 74HCT166, U24 74AHCT00, U25 ATF1504AS-44T, U26 ATF1504AS-44T, U27 ATF1504AS-44T, U28 ATF1504AS-44T, U3 24LC32, U4 MIC2775, U5 SST39SF010, U6 74LVC245, U7 74FCT2245, U8 74HCT14, U9 Z80 C20MHz-PLCC

Commit message: PLD/SCHM: Move BRK Data & Don't-Care, GPIO, and TGT_GO count to 1504
Parts:
- removed J11: Conn_02x05_PINHDR_2.54mm, Connector_IDC:IDC-Header_2x05_P2.54mm_Vertical, symbol Connector_Generic:Conn_02x05_Odd_Even
- removed J2: Conn_02x03_Odd_Even, Connector_IDC:IDC-Header_2x03_P2.54mm_Vertical, symbol Connector_Generic:Conn_02x03_Odd_Even
- removed R24: 10k, Resistor_SMD:R_0805_2012Metric, symbol Device:R_Small_US
- removed U21: 74HCT161, Package_SO:SOIC-16_3.9x9.9mm_P1.27mm, symbol AES_Library:74161-AES
- added C16, C17, C18, C19: 0.1uF, Capacitor_SMD:C_0603_1608Metric, symbol Device:C_Small
- added J11, J12, J2: JST-PH-K B6B, Connector_JST:JST_PH_B6B-PH-K_1x06_P2.00mm_Vertical, symbol Connector_Generic:Conn_01x06
- added J13: Conn_02x05_PINHDR_2.54mm, Connector_IDC:IDC-Header_2x05_P2.54mm_Vertical, symbol Connector_Generic:Conn_02x05_Odd_Even
- added U24: ATF1504AS-44T, Package_QFP:TQFP-44_10x10mm_P0.8mm, symbol AES_Library:ATF1504AS-44T-AES
- renumbered C14 to C10, C15 to C11, C16 to C12, C17 to C13, C18 to C14, C19 to C15, C8 to C4, C4 to C47, C5 to C48, C6 to C49, C9 to C5, C7 to C50, C10 to C6, C11 to C7, C12 to C8, C13 to C9, J12 to J14, R31 to R24, R32 to R31, R33 to R32, R34 to R33, R35 to R34, R36 to R35, R37 to R36, R38 to R37, R39 to R38, R40 to R39, R41 to R40, R42 to R41, R43 to R42, R44 to R43, U22 to U21, U23 to U22, U24 to U23
Connections:
- net +3.3V: now also J2.1 (Pin_1)
- net +5V: now also C16.2, C17.2, C18.2, C19.2, J11.4 (Pin_4), J12.4 (Pin_4), J13.4 (Pin_4), U24.17 (VCCINT), U24.29 (VCCINT), U24.41 (VCCINT), U24.9 (VCCINT)
- net GND: now also C16.1, C17.1, C18.1, C19.1, J11.2 (Pin_2), J12.2 (Pin_2), J13.10 (Pin_10), J13.2 (Pin_2), J2.2 (Pin_2), U24.16 (GND), U24.24 (GND), U24.36 (GND), U24.4 (GND)
- net JTCK: now also J11.1 (Pin_1), J12.1 (Pin_1), J13.1 (Pin_1), U24.26 (C48/IO/JT.TCK)
- net JTD1O2I: now also U24.1 (A8/IO/JT.TDI); no longer JA1.1 (A), U25.1 (A8/IO/JT.TDI)
- net JTD2O3I: now also JA1.1 (A), U25.1 (A8/IO/JT.TDI), U24.32 (D56/IO/JT.TDO); no longer JB1.1 (A), U25.32 (D56/IO/JT.TDO), U26.1 (A8/IO/JT.TDI)
- net JTD3O4I: now also JB1.1 (A), U25.32 (D56/IO/JT.TDO), U26.1 (A8/IO/JT.TDI); no longer JC1.1 (A), U26.32 (D56/IO/JT.TDO), U27.1 (A8/IO/JT.TDI)
- net JTD4O5I: now also JC1.1 (A), U26.32 (D56/IO/JT.TDO), U27.1 (A8/IO/JT.TDI); no longer JD1.1 (A), U27.32 (D56/IO/JT.TDO), U28.1 (A8/IO/JT.TDI)
- net JTDI_CO: now also J11.6 (Pin_6), J12.6 (Pin_6), J13.9 (Pin_9)
- net JTDO_CI: now also J11.3 (Pin_3), J12.3 (Pin_3), J13.3 (Pin_3)
- net JTMS: now also J11.5 (Pin_5), J12.5 (Pin_5), J13.5 (Pin_5), U24.7 (B32/IO/JT.TMS)
- net LRST-: now also U24.39 (IN/GCLR)
- net SBC_GPI0: now also U24.35 (D41/IO/GCK3)
- net SBC_GPI1: now also U24.33 (DMC57/IO)
- net SBC_GPI2: now also U24.30 (DMC52/IO)
- net SBC_GPI3: now also U24.31 (DMC53/IO)
- net SBC_GPO0: now also U24.43 (AMC14/IO)
- net SBC_GPO1: now also U24.42 (AMC16/IO)
- net SBC_GPO2: now also U24.44 (AMC11/IO)
- net SBC_GPO3: now also U24.2 (AMC5/IO)
- net SPICK: now also J2.3 (Pin_3)
- net SPICS2-: now also J2.6 (Pin_6)
- net SPIMI: now also J2.4 (Pin_4)
- net SPIMO: now also J2.5 (Pin_5)
- net TGTMODE-: now also U24.27 (DMC49/IO)
- net ZA1: now also U24.15 (BMC17/IO)
- net ZA2: now also U24.14 (BMC19/IO)
- net ZA3: now also U24.13 (BMC20/IO)
- net ZA4: now also U24.12 (BMC21/IO)
- net ZD0: now also U24.21 (CMC37/IO)
- net ZD1: now also U24.20 (CMC36/IO)
- net ZD2: now also U24.22 (CMC40/IO)
- net ZD3: now also U24.25 (CMC46/IO)
- net ZD4: now also U24.23 (CMC41/IO)
- net ZD5: now also U24.6 (AMC1/IO)
- net ZD6: now also U24.3 (AMC4/IO)
- net ZD7: now also U24.5 (A3/IO/PD1)
- net ZRD-: now also U24.28 (DMC51/IO)
- net ZWR-: now also U24.10 (BMC25/IO)
- net MEMOP- renamed MEM_OP-
- net MEM_OP-: now also U24.37 (IN/GCK1)
- net TGTGO renamed TGT_GO
- net TGT_GO: now also U24.34 (DMC62/IO)
- net TGTNOW renamed TGT_NOW
- net TGT_NOW: now also U24.19 (C35/IO/PD2)
- new net BRK_DEQ: U24.8 (BMC30/IO)
- new net JTD5O6I: JD1.1 (A), U27.32 (D56/IO/JT.TDO), U28.1 (A8/IO/JT.TDI)
- new net SBC_IO: U24.18 (CMC33/IO)
- no-connect marks 22 -> 18
Other:
- moved on the sheet: C10, C11, C12, C13, C14, C15, C3, C4, C47, C48, C49, C5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

Commit message: PLD/SCHM: Update pins.
Parts:
- removed TP5: TestPoint, Connector_PinHeader_2.54mm:PinHeader_1x01_P2.54mm_Vertical, symbol Connector:TestPoint
- added TP6: TestPoint, Connector_PinHeader_2.54mm:PinHeader_1x01_P2.54mm_Vertical, symbol Connector:TestPoint
- OP2: value AES-Option_A-B_2mm -> pin header 1x03 0.1"; footprint Connector_PinHeader_2.00mm:PinHeader_1x03_P2.00mm_Vertical -> Connector_PinHeader_2.54mm:PinHeader_1x03_P2.54mm_Vertical
- OP3: value AES-Option_A-B -> pin header 1x03 0.1"
- SW1: footprint AES_Library:AES-SW_PUSH_SMD_1P1T_NO_6x6mm -> AES_Library:AES-SW_PUSH_SMD_1P1T_NO_45x45mm-CK
- U20: footprint Package_SO:SOIC-16W_7.5x10.3mm_P1.27mm -> Package_SO:SOIC-16_3.9x9.9mm_P1.27mm
- U9: footprint Package_LCC:PLCC-44 -> Package_LCC:PLCC-44_THT-Socket
- renumbered R32 to R30, R30 to R31, R31 to R32, R36 to R35, R35 to R36, R39 to R38, R40 to R39, R38 to R40, TP6 to TP5, TP9 to TP8, TP8 to TP9, U24 to U23, U23 to U24
Connections:
- net LCL_IO is gone; now on net SBC_IO: U18.33 (DMC54/IO)
- net BRK_DEQ: now also U18.46 (EMC73/IO)
- net SBC_GPO2: no longer U18.46 (EMC73/IO)
- net IOBD24: now reaches U23.11 (BMC24/IO)
- net IOBD24: now also TP6.1
- no-connect marks 18 -> 20

Commit message: PLD SCHM: Switch 74FCT2257 w 74FCT2244. Reassign 1508 pins.
Parts:
- removed U20: 74FCT257T, Package_SO:SOIC-16_3.9x9.9mm_P1.27mm, symbol 74xx:74LS257
- added JS1: SolderJumper_2_Open, Jumper:SolderJumper-2_P1.3mm_Open_TrianglePad1.0x1.5mm, symbol Jumper:SolderJumper_2_Open
- added R24: 10k, Resistor_SMD:R_0805_2012Metric, symbol Device:R_Small_US
- added TP10, TP12, TP3, TP33, TP34, TP4, TP5, TP8, TP9: TestPoint, Connector_PinHeader_2.54mm:PinHeader_1x01_P2.54mm_Vertical, symbol Connector:TestPoint
- added U20: 74FCT2244, symbol AES_Library:74244-AES
- renumbered JS1 to JS2, R24 to R25, R25 to R26, R26 to R27, R27 to R28, R28 to R29, R29 to R30, R30 to R31, R31 to R32, R32 to R33, R33 to R34, R34 to R35, R35 to R36, R36 to R37, R37 to R38, R38 to R39, R39 to R40, R40 to R41, R41 to R42, R42 to R43, R43 to R44, TP5 to TP11, TP6 to TP13, TP7 to TP14, TP8 to TP15, TP9 to TP16, TP10 to TP17, TP11 to TP18, TP12 to TP19, TP13 to TP20, TP14 to TP21, TP15 to TP22, TP16 to TP23, TP17 to TP24, TP18 to TP25, TP19 to TP26, TP20 to TP27, TP21 to TP28, TP22 to TP29, TP23 to TP30, TP24 to TP31, TP25 to TP32, TP26 to TP35, TP27 to TP36, TP3 to TP6, TP4 to TP7
Connections:
- net FIXED_SEL is gone; now on net ZRST-: U18.83 (HMC125/IO)
- net +5V: now also R23.1, R24.2, U20.20 (VCC); no longer R23.2
- net AEN_CLK: now also U18.57 (FMC89/IO); no longer U18.92 (AMC16/IO)
- net AEN_CLR-: now also U18.56 (FMC88/IO); no longer U18.94 (AMC13/IO)
- net BA_CLK: now also U18.55 (FMC86/IO); no longer U18.97 (AMC9/IO)
- net BA_CLR-: now also U18.58 (FMC91/IO); no longer U18.98 (AMC8/IO)
- net BRD_RST-: now also U18.36 (DMC51/IO); no longer U18.67 (GMC102/IO)
- net BRK1_AEQ-: now also U18.13 (BMC19/IO); no longer U18.64 (GMC99/IO)
- net BRKPC_RD-: now also U18.60 (FMC93/IO); no longer U18.79 (HMC120/IO)
- net BRK_DEQ: now also U18.14 (BMC17/IO); no longer U18.46 (EMC73/IO)
- net EXTBRKRQ-: now also U18.78 (HMC118/IO); no longer U18.68 (GMC104/IO)
- net GND: now also JS1.1 (A), U20.10 (GND)
- net MEM_OP-: now also U18.16 (CMC46/IO); no longer U18.60 (FMC93/IO)
- net MOD_SEL-: now also U18.19 (CMC43/IO); no longer U18.96 (AMC11/IO)
- net MWTRQ-: now also U18.24 (CMC35/IO); no longer U18.8 (BMC25/IO)
- net PCRD_DIN: now also U18.77 (HMC117/IO); no longer U18.21 (CMC40/IO)
- net PC_LATCH-: now also U18.20 (CMC41/IO); no longer U18.69 (GMC105/IO)
- net RAM_SEL-: now also U18.50 (EMC80/IO); no longer U18.32 (DMC56/IO)
- net RFMR-: now also U18.21 (CMC40/IO); no longer U18.35 (DMC53/IO)
- net ROM_SEL: now also U18.49 (EMC78/IO); no longer U18.27 (DMC64/IO)
- net RRA0: now also U18.47 (EMC75/IO); no longer U18.29 (DMC61/IO)
- net RRA1: now also U18.46 (EMC73/IO); no longer U18.28 (DMC62/IO)
- net RRA2: now also U18.48 (EMC77/IO); no longer U18.30 (DMC59/IO)
- net SBCMODE-: now also U18.22 (CMC38/IO); no longer U18.24 (CMC35/IO)
- net SBC_GPI0: no longer U18.55 (FMC86/IO)
- net SBC_GPI1: no longer U18.56 (FMC88/IO)
- net SBC_GPI2: no longer U18.22 (CMC38/IO)
- net SBC_GPI3: no longer U18.20 (CMC41/IO)
- net SBC_GPO0: no longer U18.17 (CMC45/IO)
- net SBC_GPO1: no longer U18.16 (CMC46/IO)
- net SBC_GPO3: no longer U18.47 (EMC75/IO)
- net SBC_IO: now also U18.45 (EMC72/IO); no longer U18.33 (DMC54/IO)
- net SYNC: now also U18.67 (GMC102/IO); no longer U18.37 (DMC49/IO)
- net TBREQB-: now also U18.33 (DMC54/IO); no longer U18.65 (GMC101/IO)
- net TDBUSEN-: now also U18.41 (E67/IO/PD2); no longer U18.81 (HMC123/IO)
- net TDBUSIN-: now also U18.17 (CMC45/IO); no longer U18.61 (FMC94/IO)
- net TGTMODE-: now also U18.84 (HMC126/IO); no longer U18.36 (DMC51/IO)
- net TGTONLY-: now also U18.31 (DMC57/IO); no longer U18.76 (HMC115/IO)
- net TGT_GO: now also U18.61 (FMC94/IO); no longer U18.48 (EMC77/IO)
- net TGT_NOW: now also U18.10 (BMC22/IO); no longer U18.54 (FMC85/IO)
- net TINTB-: now also U18.32 (DMC56/IO); no longer U18.75 (HMC113/IO)
- net TIORQ-: now also U20.16 (O1a), U20.7 (O1b)
- net TMREQ-: now also U20.18 (O0a), U20.9 (O0b)
- net TNMIB-: now also U18.35 (DMC53/IO); no longer U18.63 (GMC97/IO)
- net TRD-: now also U20.14 (O2a), U20.5 (O2b)
- net TWAITRQ-: now also U18.37 (DMC49/IO); no longer U18.41 (E67/IO/PD2)
- net TWR-: now also U20.12 (O3a), U20.3 (O3b)
- net ZA1: now also U18.2 (AMC1/IO); no longer U18.1 (A3/IO/PD1)
- net ZA14: now also U18.98 (AMC8/IO); no longer U18.10 (BMC22/IO)
- net ZA15: now also U18.94 (AMC13/IO); no longer U18.9 (BMC24/IO)
- net ZA2: now also U18.1 (A3/IO/PD1); no longer U18.19 (CMC43/IO)
- net ZA3: now also U18.100 (AMC5/IO); no longer U18.14 (BMC17/IO)
- net ZA4: now also U18.99 (AMC6/IO); no longer U18.13 (BMC19/IO)
- net ZA5: now also U18.64 (GMC99/IO); no longer U18.44 (EMC70/IO)
- net ZA6: now also U18.65 (GMC101/IO); no longer U18.45 (EMC72/IO)
- net ZA7: now also U18.75 (HMC113/IO); no longer U18.52 (FMC81/IO)
- net ZBACK-: now also U18.40 (EMC65/IO); no longer U18.57 (FMC89/IO), U8.11
- net ZBREQ-: now also U18.69 (GMC105/IO); no longer U18.70 (GMC107/IO)
- net ZD0: now also U18.5 (BMC30/IO); no longer U18.6 (BMC29/IO)
- net ZD1: now also U18.92 (AMC16/IO); no longer U18.93 (AMC14/IO)
- net ZD2: now also U18.93 (AMC14/IO); no longer U18.100 (AMC5/IO)
- net ZD3: now also U18.96 (AMC11/IO); no longer U18.99 (AMC6/IO)
- net ZD4: now also U18.8 (BMC25/IO); no longer U18.50 (EMC80/IO)
- net ZD5: now also U18.9 (BMC24/IO); no longer U18.49 (EMC78/IO)
- net ZD6: now also U18.7 (BMC27/IO); no longer U18.5 (BMC30/IO)
- net ZD7: now also U18.97 (AMC9/IO), U25.38 (IN/OE1), U25.6 (AMC1/IO); no longer U18.7 (BMC27/IO)
- net ZINT-: now also U18.68 (GMC104/IO); no longer U18.80 (HMC121/IO)
- net ZIORQ-: now also U18.63 (GMC97/IO), U20.4 (I1a); no longer U18.42 (EMC69/IO)
- net ZMREQ-: now also U18.23 (CMC37/IO), U20.2 (I0a); no longer U18.89 (IN/GCLR)
- net ZNMI-: now also U18.70 (GMC107/IO); no longer U18.58 (FMC91/IO)
- net ZRD-: now also U18.6 (BMC29/IO), U20.6 (I2a); no longer U18.2 (AMC1/IO)
- net ZRFSH-: now also U18.89 (IN/GCLR); no longer U18.25 (CMC33/IO)
- net ZRST-: no longer U18.72 (GMC110/IO)
- net ZWAIT-: now also U18.72 (GMC110/IO); no longer U18.31 (DMC57/IO)
- net ZWR-: now also U18.25 (CMC33/IO), U20.8 (I3a); no longer U18.12 (BMC21/IO)
- net at OP1.2 (C): now also R24.1, U20.11 (I0b); no longer R23.1
- net BRK2N_AEQ- renamed BRKN_AEQ-
- net BRKN_AEQ-: now also U18.12 (BMC21/IO); no longer U18.40 (EMC65/IO)
- net BRKHW_DET- renamed BRKHWDET-
- net BRKHWDET-: now also U18.76 (HMC115/IO); no longer U18.23 (CMC37/IO)
- removed net D7_B: U18.84 (HMC126/IO), U25.38 (IN/OE1), U25.6 (AMC1/IO)
- net I88 renamed IOE1
- net IO77 renamed IO62
- net IO62: now also U18.28 (DMC62/IO); no longer U18.77 (HMC117/IO)
- net IO78 renamed IO64
- net IO64: now also U18.27 (DMC64/IO); no longer U18.78 (HMC118/IO)
- net ZBACK: no longer names the net of U8.10
- net ZBACK: now also TP34.1
- new net: R23.2, U20.13 (I1b), U20.15 (I2b), U20.17 (I3b)
- new net: JS1.2 (B), TP33.1, U8.11
- new net IO120: TP5.1, U18.79 (HMC120/IO)
- new net IO121: TP4.1, U18.80 (HMC121/IO)
- new net IO123: TP3.1, U18.81 (HMC123/IO)
- new net IO59: TP9.1, U18.30 (DMC59/IO)
- new net IO61: TP8.1, U18.29 (DMC61/IO)
- new net IO81: TP12.1, U18.52 (FMC81/IO)
- new net IO85: TP10.1, U18.54 (FMC85/IO)
- new net TCBUSEN-: U18.42 (EMC69/IO), U20.1 (~{OEa})
- new net TCBUSFEN-: U18.44 (EMC70/IO), U20.19 (~{OEb})
Other:
- moved on the sheet: TP13, TP6, TP7, U8E

Commit message: PLD: Update pins. SCHM: PLD pins, TCTRL correction.
Parts:
- removed J7, J9: Conn_02x04_2.54mm, Connector_PinHeader_2.54mm:PinHeader_2x04_P2.54mm_Vertical, symbol Connector_Generic:Conn_02x04_Row_Letter_First
- removed J8: Conn_02x02_2.54mm, Connector_PinHeader_2.54mm:PinHeader_2x02_P2.54mm_Vertical, symbol Connector_Generic:Conn_02x02_Row_Letter_First
- removed R34: 20k, Resistor_SMD:R_0805_2012Metric, symbol Device:R_Small_US
- removed U10: 74LVC2G04, Package_TO_SOT_SMD:SOT-23-6, symbol AES_Library:74LVC2G04-AES
- removed unit 1 of U21
- added J7, J9: Conn 2x04 0.1" pin, Connector_PinHeader_2.54mm:PinHeader_2x04_P2.54mm_Vertical, symbol Connector_Generic:Conn_02x04_Odd_Even
- added J8: Conn 2x02 0.1" pin, Connector_PinHeader_2.54mm:PinHeader_2x02_P2.54mm_Vertical, symbol Connector_Generic:Conn_02x02_Odd_Even
- added TP33, TP34: TestPoint, Connector_PinHeader_2.54mm:PinHeader_1x01_P2.54mm_Vertical, symbol Connector:TestPoint
- added U10: 27WZ06, symbol AES_Library:NL27WZ06DFT2G-AES
- added unit 1 of U24
- C1, C2: value 0.1u -> 0.1uf; footprint Capacitor_SMD:C_0603_1608Metric_Pad1.08x0.95mm_HandSolder -> Capacitor_SMD:C_0603_1608Metric
- C3: footprint Capacitor_SMD:C_1210_3225Metric_Pad1.33x2.70mm_HandSolder -> Capacitor_SMD:C_0603_1608Metric
- J1: value HDR 1x04 Socket -> Conn 1x04 0.1" Socket
- J3: value Conn_01x02_Pin_2.54mm -> Conn 1x02 0.1" pin
- J4: value Conn_01x03 -> Conn 1x03 0.1" pin
- J5, J6: value Conn_01x08 -> Conn 1x08 0.1" pin
- R32: value 20k -> 10k
- SPARE1: footprint AES_Library:SPARE-and-SOIC-16-AES -> AES_Library:SPARE-16-SOT-5_6-AES
- U12: footprint Package_SO:SOIC-20W_7.5x12.8mm_P1.27mm -> Package_SO:SO-20_12.8x7.5mm_P1.27mm
- U13, U2, U7: footprint Package_SO:SOIC-20W_7.5x12.8mm_P1.27mm -> Package_SO:SSOP-20_3.9x8.7mm_P0.635mm; symbol AES_Library:74245-AES -> AES_Library:74FCT2245-AES
- U15, U17: footprint Package_SO:SOIC-20W_7.5x12.8mm_P1.27mm -> Package_SO:SSOP-20_3.9x8.7mm_P0.635mm; symbol AES_Library:74245_BA-AES -> AES_Library:74FCT2245-AES
- U16: footprint Package_SO:SOIC-20W_7.5x12.8mm_P1.27mm -> Package_SO:SSOP-20_3.9x8.7mm_P0.635mm
- U20: footprint (none) -> Package_SO:SSOP-20_3.9x8.7mm_P0.635mm; symbol AES_Library:74244-AES -> AES_Library:74FCT244-AES
- U23: renamed from U24; footprint Package_SO:SOIC-14_3.9x8.7mm_P1.27mm -> Package_SO:SO-14_3.9x8.65mm_P1.27mm
- U24: renamed from U21; value 74AHCT244 -> 74FCT2244; footprint Package_SO:SOIC-20W_7.5x12.8mm_P1.27mm -> Package_SO:SSOP-20_3.9x8.7mm_P0.635mm
- U24: renamed from U21; value 74AHCT244 -> 74FCT2244; footprint Package_SO:SOIC-20W_7.5x12.8mm_P1.27mm -> Package_SO:SSOP-20_3.9x8.7mm_P0.635mm; symbol AES_Library:74244-AB-AES -> AES_Library:74FCT2244-AB-AES
- U6: footprint Package_SO:SOIC-20W_7.5x12.8mm_P1.27mm -> Package_SO:SO-20_5.3x12.6mm_P1.27mm
- U8: value 74HCT14 -> 74AHCT14; footprint Package_SO:SOIC-14_3.9x8.7mm_P1.27mm -> Package_SO:SO-14_3.9x8.65mm_P1.27mm
- renumbered JS1 to JS6, JS2 to JS7, TP33 to TP42, TP34 to TP43, TP35 to TP44, TP36 to TP45, U22 to U21, U23 to U22
Connections:
- net +3.3V: now also R32.2, U10.5 (VCC)
- net +5V: now also J8.1 (Pin_1), J8.2 (Pin_2), J8.3 (Pin_3), J8.4 (Pin_4), J9.7 (Pin_7); no longer R32.2
- net GND: now also J7.1 (Pin_1), J7.3 (Pin_3), J7.5 (Pin_5), J7.7 (Pin_7), J9.1 (Pin_1), J9.3 (Pin_3), J9.5 (Pin_5), U10.2 (GND)
- net LA0: now also U15.18 (B0); no longer U15.2 (A0)
- net LA1: now also U15.17 (B1); no longer U15.3 (A1)
- net LA10: now also U17.16 (B2); no longer U17.4 (A2)
- net LA11: now also U17.15 (B3); no longer U17.5 (A3)
- net LA12: now also U17.14 (B4); no longer U17.6 (A4)
- net LA13: now also U17.13 (B5); no longer U17.7 (A5)
- net LA14: now also U17.12 (B6); no longer U17.8 (A6)
- net LA15: now also U17.11 (B7); no longer U17.9 (A7)
- net LA2: now also U15.16 (B2); no longer U15.4 (A2)
- net LA3: now also U15.15 (B3); no longer U15.5 (A3)
- net LA4: now also U15.14 (B4); no longer U15.6 (A4)
- net LA5: now also U15.13 (B5); no longer U15.7 (A5)
- net LA6: now also U15.12 (B6); no longer U15.8 (A6)
- net LA7: now also U15.11 (B7); no longer U15.9 (A7)
- net LA8: now also U17.18 (B0); no longer U17.2 (A0)
- net LA9: now also U17.17 (B1); no longer U17.3 (A1)
- net MODINT-: now also J9.8 (Pin_8), U10.6; no longer U25.34 (DMC62/IO)
- net SBC_I0: now also J9.2 (Pin_2)
- net SBC_I1: now also J9.4 (Pin_4)
- net SBC_I2: now also J9.6 (Pin_6)
- net SBC_O0: now also J7.2 (Pin_2)
- net SBC_O1: now also J7.4 (Pin_4)
- net SBC_O2: now also J7.6 (Pin_6)
- net SBC_O3: now also J7.8 (Pin_8)
- net SPICS2-: now also R32.1, U10.4
- net TIORQ-: now also U20.5 (Ob1), U24.4 (I1a); no longer U20.7 (O1b)
- net TMREQ-: now also U20.3 (Ob0), U24.2 (I0a); no longer U20.9 (O0b)
- net TRD-: now also U20.7 (Ob2), U24.6 (I2a); no longer U20.5 (O2b)
- net TWR-: now also U20.9 (Ob3), U24.8 (I3a); no longer U20.3 (O3b)
- net ZA0: now also U15.2 (A0); no longer U15.18 (B0)
- net ZA1: now also U15.3 (A1); no longer U15.17 (B1)
- net ZA10: now also U17.4 (A2); no longer U17.16 (B2)
- net ZA11: now also U17.5 (A3); no longer U17.15 (B3)
- net ZA12: now also U17.6 (A4); no longer U17.14 (B4)
- net ZA13: now also U17.7 (A5); no longer U17.13 (B5)
- net ZA14: now also U17.8 (A6); no longer U17.12 (B6)
- net ZA15: now also U17.9 (A7); no longer U17.11 (B7)
- net ZA2: now also U15.4 (A2); no longer U15.16 (B2)
- net ZA3: now also U15.5 (A3); no longer U15.15 (B3)
- net ZA4: now also U15.6 (A4); no longer U15.14 (B4)
- net ZA5: now also U15.7 (A5); no longer U15.13 (B5)
- net ZA6: now also U15.8 (A6); no longer U15.12 (B6)
- net ZA7: now also U15.9 (A7); no longer U15.11 (B7)
- net ZA8: now also U17.2 (A0); no longer U17.18 (B0)
- net ZA9: now also U17.3 (A1); no longer U17.17 (B1)
- net ZBACK-: now also U24.1 (~{OEa}); no longer R32.1
- net ZIORQ-: now also U24.16 (O1a)
- net ZMREQ-: now also U24.18 (O0a)
- net ZRD-: now also U22.40 (IN/OE2/GCK2), U24.14 (O2a); no longer U22.28 (DMC51/IO)
- net ZWR-: now also U22.38 (IN/OE1), U24.12 (O3a); no longer U22.10 (BMC25/IO)
- net at U12.6 (Q2): now also U10.3
- net at OP1.2 (C), R24.1: now also U20.17 (Ib0); no longer U20.11 (I0b)
- net at R23.2, U20.13 (Ib2), U20.15 (Ib1): now also U20.11 (Ib3); no longer U20.17 (I3b)
- net at U12.5 (Q1): now also U10.1
- net MINT-: no longer names the net of U25.33 (DMC57/IO)
- new net IOBD25: TP33.1, U22.10 (BMC25/IO)
- new net IOBD51: TP34.1, U22.28 (DMC51/IO)
- no-connect marks 20 -> 18
Other:
- moved on the sheet: J2, JP6, OP1, R19, R20, R21, R22, R24, U16
