File: hw/ZID_MAIN/ZID_MAIN.kicad_sch (KiCad schematic)
At the start: 216 parts, among them J1 Conn 1x04 0.1" Socket, J10 FFC/FPC-40 Socket, J11 JST-PH-K B6B, J12 JST-PH-K B6B, J13 Conn_02x05_PINHDR_2.54mm, J14 USB-C PWR ONLY, J2 JST-PH-K B6B, J3 Conn 1x02 0.1" pin, J4 Conn 1x03 0.1" pin, J5 Conn 1x08 0.1" pin, J6 Conn 1x08 0.1" pin, J7 Conn 2x04 0.1" pin, J8 Conn 2x02 0.1" pin, J9 Conn 2x04 0.1" pin, M1 WS-RP2040-Zero, SW1 SW_Push, SW2 SW_DIP_x02, U1 OSC-20MHz, U10 27WZ06, U11 74LVC125AS, U12 74LVC273, U13 74FCT2245, U14 AS7C1024B, U15 74FCT2245, U16 74FCT2245, U17 74FCT2245, U18 ATF1508AS, U19 74HCT166, U2 74FCT2245, U20 74FCT2244, U21 74HCT166, U22 ATF1504AS-44T, U23 74AHCT00, U24 74FCT2244, U25 ATF1504AS-44T, U26 ATF1504AS-44T, U27 ATF1504AS-44T, U28 ATF1504AS-44T, U3 24LC32, U4 MIC2775, U5 SST39SF010, U6 74LVC245, U7 74FCT2245, U8 74AHCT14, U9 Z80 C20MHz-PLCC

Commit message: PCB: All components placed V0.1
Parts:
- removed C3: 100uF, Capacitor_SMD:C_0603_1608Metric, symbol Device:C_Small
- removed JA1, JB1, JS6, JS7: SolderJumper_2_Open, Jumper:SolderJumper-2_P1.3mm_Open_TrianglePad1.0x1.5mm, symbol Jumper:SolderJumper_2_Open
- removed TP19, TP20, TP23, TP24, TP27, TP30, TP42, TP43, TP44, TP45: TestPoint, Connector_PinHeader_2.54mm:PinHeader_1x01_P2.54mm_Vertical, symbol Connector:TestPoint
- removed U15, U17: 74FCT2245, Package_SO:SSOP-20_3.9x8.7mm_P0.635mm, symbol AES_Library:74FCT2245-AES
- removed U19, U21: 74HCT166, Package_SO:SOIC-16_3.9x9.9mm_P1.27mm, symbol AES_Library:74166-AES
- added C3: 100UF TANT, Capacitor_Tantalum_SMD:CP_EIA-7343-31_Kemet-D_HandSolder, symbol Device:C_Polarized_US
- added OP4: AES-Option_A-B_2mm, Connector_PinHeader_2.00mm:PinHeader_1x03_P2.00mm_Vertical, symbol AES_Library:AES-Option_A-B_2mm
- added RN2: 20k, Resistor_THT:R_Array_SIP9, symbol Device:R_Network08_US
- added SPRU8F1: Conn_01x03_Pin, Connector_PinHeader_2.00mm:PinHeader_1x03_P2.00mm_Vertical, symbol Connector:Conn_01x03_Pin
- J1: Function I2C-RTC -> RTC (I2C); P3 SCL (RX) -> SCL(RX); P4 SDA (TX) -> SDA(TX)
- J11: P1 PWR -> 1CK; P2 GND -> 2-; P3 SCK -> 3MI; P4 MISO -> 4+; P5 MOSI -> 5CS; P6 CS -> 6MO
- J2: P4 MISO -> MI; P5 MOSI -> MO
- J5: now not fitted; now left out of the parts list
- J6: Function TGT DATA -> TDATA DEBUG; now not fitted; now left out of the parts list
- J7: Function SBC OUT -> Out 0-3
- J8: Function EXP PWR -> EPWR
- J9: Function SBC IN -> In 0-2; POS4 (none) -> MINT
- OP2: OP-A WAIT -> P-WAIT; OP-B NO WAIT -> NO
- OP3: OP-A HIGH-T -> T+; OP-B LOW-T -> T-
- SW2: S2 OPT-1 -> SBC-In3
- TP1: footprint Connector_PinHeader_2.54mm:PinHeader_1x01_P2.54mm_Vertical -> Connector_PinHeader_2.00mm:PinHeader_1x01_P2.00mm_Vertical; Function IO2 -> SBC-CLK; now not fitted; now left out of the parts list
- TP10, TP11, TP12, TP13, TP17, TP18, TP2, TP21, TP22, TP25, TP26, TP28, TP29, TP3, TP31, TP32, TP33, TP34, TP4, TP5, TP6, TP7, TP8, TP9: footprint Connector_PinHeader_2.54mm:PinHeader_1x01_P2.54mm_Vertical -> TestPoint:TestPoint_THTPad_D1.0mm_Drill0.5mm; now not fitted; now left out of the parts list
- TP15: Function SYNC -> EBRK
- TP16: value TestPoint -> GND-CONN; symbol Connector:TestPoint -> Connector:TestPoint_Alt
- U1: footprint AES_Library:OSC-8_14-AES -> AES_Library:OSC-8_14-CO-AES; symbol AES_Library:OSC-8_14CAN-AES -> AES_Library:OSC-8_14CAN-CO-AES
- U10: footprint (none) -> Package_TO_SOT_SMD:SOT-363_SC-70-6
- U14: footprint Package_SO:SOJ-32_10.16x20.955mm_P1.27mm -> AES_Library:SOJ-32_WN-AES; Function SRAM -> 128Kx8 SRAM
- U20: symbol AES_Library:74FCT244-AES -> AES_Library:74FCT2244-AES
- U24: symbol AES_Library:74244-AB-AES -> AES_Library:74FCT2244-AB-AES
- U25: Function BRK1&2n Addr Cmp -> BRK1&2 PCL-H; ISP_CN ISP#2 -> ISP#3
- U26: Function BRK3&4 Addr Cmp -> BRK3&4 PCL-L; ISP_CN ISP#3 -> ISP#4
- U27: Function BRK5&6 Addr Cmp -> BRK5&6; ISP_CN ISP#4 -> ISP#5
- U28: Function BRK7&8 Addr Cmp -> BRK7&8; ISP_CN ISP#5 -> ISP#6
- U5: Function FLASH -> 128Kx8 FLASH
- renumbered C50 to C47, C49 to C48, C48 to C49, C47 to C50
Connections:
- net GPI_A- is gone; now on net PCRD_DIN: U26.33 (DMC57/IO)
- net GPO_A- is gone; now on net BRKN_AEQ-: U26.34 (DMC62/IO)
- net IO10A is gone; now on net ZA9: U25.10 (BMC25/IO)
- net IO10B is gone; now on net ZA13: U26.10 (BMC25/IO)
- net IO8A is gone; now on net ENBL_DOA: U25.8 (BMC30/IO)
- net IO8B is gone; now on net ENBL_DOB: U26.8 (BMC30/IO)
- net +5V: now also U1.11 (PWRs), U1.4 (ENs), C3.1, RN2.1 (common)
- net ADDR_DOA: now also U25.42 (AMC16/IO), U26.31 (DMC53/IO); no longer U25.3 (AMC4/IO), U26.6 (AMC1/IO)
- net ADDR_DOB: now also U26.42 (AMC16/IO); no longer U26.3 (AMC4/IO)
- net BA_CLK: now also U25.35 (D41/IO/GCK3), U26.35 (D41/IO/GCK3); no longer U25.37 (IN/GCK1), U26.37 (IN/GCK1)
- net BA_CLR-: now also U25.3 (AMC4/IO), U26.3 (AMC4/IO); no longer U25.35 (D41/IO/GCK3), U26.35 (D41/IO/GCK3)
- net BRK1_AEQ-: now also U25.25 (CMC46/IO), OP4.3 (B); no longer U25.43 (AMC14/IO)
- net BRKHWDET-: now also U25.6 (AMC1/IO), U26.6 (AMC1/IO); no longer U25.44 (AMC11/IO), U26.44 (AMC11/IO)
- net BRKN_AEQ-: now also U26.25 (CMC46/IO), OP4.1 (A); no longer U25.42 (AMC16/IO), U26.42 (AMC16/IO), U26.43 (AMC14/IO)
- net BRKPC_RD-: now also U25.37 (IN/GCK1), U26.37 (IN/GCK1)
- net ENBL_DOA: no longer U25.2 (AMC5/IO)
- net ENBL_DOB: no longer U26.2 (AMC5/IO)
- net GND: now also U25.31 (DMC53/IO), C3.2, SPRU8F1.1 (Pin_1); no longer U1.4 (G)
- net PC_LATCH-: now also U25.19 (C35/IO/PD2), U26.12 (BMC21/IO)
- net ZA0: now also RN1.9 (R8), U25.12 (BMC21/IO), U26.2 (AMC5/IO), U27.11 (BMC24/IO), U28.11 (BMC24/IO)
- net ZA1: now also RN1.8 (R7), U25.28 (DMC51/IO), U26.27 (DMC49/IO), U27.12 (BMC21/IO), U28.12 (BMC21/IO)
- net ZA10: now also U25.2 (AMC5/IO), U26.43 (AMC14/IO), U27.23 (CMC41/IO), U28.23 (CMC41/IO), RN2.9 (R8); no longer RN1.4 (R3)
- net ZA11: now also U25.13 (BMC20/IO), U26.20 (CMC36/IO), U27.25 (CMC46/IO), U28.25 (CMC46/IO), RN2.8 (R7); no longer RN1.3 (R2)
- net ZA12: now also U25.44 (AMC11/IO), U26.11 (BMC24/IO), U27.27 (DMC49/IO), U28.27 (DMC49/IO), RN2.4 (R3); no longer RN1.2 (R1)
- net ZA13: now also U25.43 (AMC14/IO), U27.28 (DMC51/IO), U28.28 (DMC51/IO), RN2.5 (R4); no longer RN1.6 (R5)
- net ZA14: now also U25.15 (BMC17/IO), U26.18 (CMC33/IO), U27.30 (DMC52/IO), U28.30 (DMC52/IO), RN2.3 (R2); no longer RN1.8 (R7)
- net ZA15: now also U25.14 (BMC19/IO), U26.19 (C35/IO/PD2), U27.31 (DMC53/IO), U28.31 (DMC53/IO), RN2.2 (R1); no longer RN1.9 (R8)
- net ZA2: now also RN1.7 (R6), U25.27 (DMC49/IO), U26.23 (CMC41/IO), U27.13 (BMC20/IO), U28.13 (BMC20/IO)
- net ZA3: now also RN1.6 (R5), U25.23 (CMC41/IO), U26.28 (DMC51/IO), U27.14 (BMC19/IO), U28.14 (BMC19/IO)
- net ZA4: now also RN1.5 (R4), U25.22 (CMC40/IO), U26.13 (BMC20/IO), U27.15 (BMC17/IO), U28.15 (BMC17/IO)
- net ZA5: now also RN1.4 (R3), U25.21 (CMC37/IO), U26.14 (BMC19/IO), U27.18 (CMC33/IO), U28.18 (CMC33/IO)
- net ZA6: now also RN1.3 (R2), U25.20 (CMC36/IO), U26.15 (BMC17/IO), U27.19 (C35/IO/PD2), U28.19 (C35/IO/PD2)
- net ZA7: now also RN1.2 (R1), U25.11 (BMC24/IO), U26.44 (AMC11/IO), U27.20 (CMC36/IO), U28.20 (CMC36/IO)
- net ZA8: now also U25.18 (CMC33/IO), U26.22 (CMC40/IO), U27.21 (CMC37/IO), U28.21 (CMC37/IO), RN2.6 (R5); no longer RN1.7 (R6)
- net ZA9: now also U26.21 (CMC37/IO), U27.22 (CMC40/IO), U28.22 (CMC40/IO), RN2.7 (R6); no longer RN1.5 (R4)
- net ZD7: now also U25.30 (DMC52/IO); no longer U25.6 (AMC1/IO)
- net ZRST-: now also U8.11; no longer U2.19 (~{OE}), U7.19 (~{OE})
- net _CLK: no longer U1.11 (O)
- net at U8.13: now also SPRU8F1.2 (Pin_2)
- net at U8.12: now also SPRU8F1.3 (Pin_3)
- net ZRST: now reaches U8.10
- net ZRST: now also U2.19 (~{OE}), U7.19 (~{OE})
- net SD_OUTIN: now reaches U25.33 (DMC57/IO)
- net SD_OUTIN: now also U26.30 (DMC52/IO)
- net at U25.34 (DMC62/IO): now also OP4.2 (C)
- net GPI_B- renamed GPI_C-
- net GPI_C-: no longer TP32.1, U28.33 (DMC57/IO)
- net GPO_B- renamed GPO_C-
- net GPO_C-: no longer TP29.1, U28.34 (DMC62/IO)
- removed net LA0: U25.11 (BMC24/IO), U26.11 (BMC24/IO), U27.11 (BMC24/IO), U28.11 (BMC24/IO)
- removed net LA1: U25.12 (BMC21/IO), U26.12 (BMC21/IO), U27.12 (BMC21/IO), U28.12 (BMC21/IO)
- removed net LA10: U25.23 (CMC41/IO), U26.23 (CMC41/IO), U27.23 (CMC41/IO), U28.23 (CMC41/IO)
- removed net LA11: U25.25 (CMC46/IO), U26.25 (CMC46/IO), U27.25 (CMC46/IO), U28.25 (CMC46/IO)
- removed net LA12: U25.27 (DMC49/IO), U26.27 (DMC49/IO), U27.27 (DMC49/IO), U28.27 (DMC49/IO)
- removed net LA13: U25.28 (DMC51/IO), U26.28 (DMC51/IO), U27.28 (DMC51/IO), U28.28 (DMC51/IO)
- removed net LA14: U25.30 (DMC52/IO), U26.30 (DMC52/IO), U27.30 (DMC52/IO), U28.30 (DMC52/IO)
- removed net LA15: U25.31 (DMC53/IO), U26.31 (DMC53/IO), U27.31 (DMC53/IO), U28.31 (DMC53/IO)
- removed net LA2: U25.13 (BMC20/IO), U26.13 (BMC20/IO), U27.13 (BMC20/IO), U28.13 (BMC20/IO)
- removed net LA3: U25.14 (BMC19/IO), U26.14 (BMC19/IO), U27.14 (BMC19/IO), U28.14 (BMC19/IO)
- removed net LA4: U25.15 (BMC17/IO), U26.15 (BMC17/IO), U27.15 (BMC17/IO), U28.15 (BMC17/IO)
- removed net LA5: U25.18 (CMC33/IO), U26.18 (CMC33/IO), U27.18 (CMC33/IO), U28.18 (CMC33/IO)
- removed net LA6: U25.19 (C35/IO/PD2), U26.19 (C35/IO/PD2), U27.19 (C35/IO/PD2), U28.19 (C35/IO/PD2)
- removed net LA7: U25.20 (CMC36/IO), U26.20 (CMC36/IO), U27.20 (CMC36/IO), U28.20 (CMC36/IO)
- removed net LA8: U25.21 (CMC37/IO), U26.21 (CMC37/IO), U27.21 (CMC37/IO), U28.21 (CMC37/IO)
- removed net LA9: U25.22 (CMC40/IO), U26.22 (CMC40/IO), U27.22 (CMC40/IO), U28.22 (CMC40/IO)
- new net GPI_D-: TP32.1, U28.33 (DMC57/IO)
- new net GPO_D-: TP29.1, U28.34 (DMC62/IO)
Other:
- moved on the sheet: C47, C48, C49, C50, D2, D3, D4, H1, H2, H3, H4, J14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
