File: hw/ZID_MAIN/zid_main_logic.kicad_sch (KiCad schematic)
At the start: 82 parts, among them J1 Conn_01x02_Pin_2.54mm, J2 Conn_02x05_2.54mm, J3 Conn_02x05_2.54mm, J4 Conn_02x05_PINHDR_2.54mm, J5 HDR 1x04 Socket, J6 Conn_02x03_Odd_Even, J7 Conn_01x03, M1 WS-RP2040-Zero, SW1 SW_Push, SW2 SW_DIP_x02, U1 74HCT161, U10 74FCT2245, U11 SST39SF010, U12 AS7C1024B-10J, U13 74FCT541C, U14 74AHCT244, U15 74FCT257T, U16 74HCT166, U17 74HCT166, U18 74LVC245, U19 74LVC125AS, U2 74FCT541C, U20 24LC32, U21 ATF1504AS-44T, U22 74AHCT1G125, U23 74LVC273, U25 74LVC3G04, U3 74FCT541C, U4 MIC2775, U5 OSC-20MHz, U6 Z80 C20MHz-PLCC, U7 ATF1508AS, U8 74FCT2245, U9 74FCT2245

Commit message: PCB layout 2
Parts:
- removed U25: 74LVC3G04, Package_SO:SSOP-8_2.95x2.8mm_P0.65mm, symbol AES_Library:74LVC3G04-AES
- added U25: 74LVC2G04, Package_TO_SOT_SMD:SOT-23-6, symbol AES_Library:74LVC2G04-AES
- added U26: 74AHCT1G14, Package_TO_SOT_SMD:SOT-23-5, symbol 74xGxx:74AHCT1G14
- renumbered D7 to LED5, D5 to LED6, D8 to LED7, D6 to LED8, D9 to LED9
Connections:
- net +3.3V: now also U25.5 (VCC)
- net +5V: now also U26.5 (VCC)
- net BUSACK: now also U26.4
- net GND: now also U25.2 (GND), U26.3 (GND)
- net MINT-: now also U25.6
- net SPICS2-: now also U25.4
- net ZA11: now also RN1.3 (R2); no longer RN1.5 (R4)
- net ZA12: now also RN1.2 (R1); no longer RN1.6 (R5)
- net ZA13: now also RN1.6 (R5); no longer RN1.7 (R6)
- net ZA8: now also RN1.7 (R6); no longer RN1.2 (R1)
- net ZA9: now also RN1.5 (R4); no longer RN1.3 (R2)
- net ZBACK-: now also U26.2
- net at U23.5 (Q1): now also U25.1
- net at U23.6 (Q2): now also U25.3
Other:
- moved on the sheet: OP1, R13, U15, U19E

Commit message: PCB-Main layout 3
Parts:
- SBC1, SBC2, SBC3: OP1-2 NOR -> TGT
Changed lines of the file:
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@@
 	(title_block
 		(title "ZID Main Logic")
-		(date "2026-04-09")
+		(date "2026-04-10")
 		(rev "PR-1.0")
 		(company "SilkyDESIGN / CMOS1")
@@
 			)
 		)
-		(property "OP1-2" "NOR"
+		(property "OP1-2" "TGT"
 			(at 85.09 134.62 0)
 			(effects
@@
 			)
 		)
-		(property "OP1-2" "NOR"
+		(property "OP1-2" "TGT"
 			(at 80.01 16.51 0)
 			(effects
@@
 			)
 		)
-		(property "OP1-2" "NOR"
+		(property "OP1-2" "TGT"
 			(at 80.01 40.64 0)
 			(effects

Commit message: PCB Main: layout 20250411a
Parts:
- LED5, LED6, LED7, LED8, LED9: footprint LED_SMD:LED_0805_2012Metric_Pad1.15x1.40mm_HandSolder -> LED_THT:LED_D3.0mm
Connections:
- net GND: now also J1.1 (Pin_1); no longer J1.2 (Pin_2)
- net at SW1.2, U4.4 (~{MR}): now also J1.2 (Pin_2); no longer J1.1 (Pin_1)
Other:
- moved on the sheet: J1
Changed lines of the file:
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@@
 	(title_block
 		(title "ZID Main Logic")
-		(date "2026-04-10")
+		(date "2026-04-11")
 		(rev "PR-1.0")
 		(company "SilkyDESIGN / CMOS1")
@@
 	(symbol
 		(lib_id "Connector_Generic:Conn_01x02")
-		(at 31.75 52.07 90)
+		(at 34.29 52.07 270)
+		(mirror x)
 		(unit 1)
 		(exclude_from_sim no)
@@
 		(dnp no)
 		(property "Reference" "J1"
-			(at 36.322 52.07 90)
+			(at 29.718 52.07 90)
 			(effects
 				(font
@@
 		)
 		(property "Value" "Conn_01x02_Pin_2.54mm"
-			(at 36.83 53.3399 90)
+			(at 29.21 53.3399 90)
 			(effects
 				(font
@@
 		)
 		(property "Footprint" "Connector_PinHeader_2.54mm:PinHeader_1x02_P2.54mm_Vertical"
-			(at 31.75 52.07 0)
+			(at 34.29 52.07 0)
 			(effects
 				(font
@@
 		)
 		(property "Datasheet" "~"
-			(at 31.75 52.07 0)
+			(at 34.29 52.07 0)
 			(effects
 				(font
@@
 		)
 		(property "Description" "Generic connector, single row, 01x02, script generated (kicad-library-utils/schlib/autogen/connector/)"
-			(at 31.75 52.07 0)
+			(at 34.29 52.07 0)
 			(effects
 				(font
@@
 		)
 		(property "Function" "RST PB"
-			(at 32.766 49.53 90)
+			(at 33.274 49.53 90)
 			(effects
 				(font
@@
 		)
 		(instances
-			(project ""
+			(project "ZID_MAIN"
 				(path "/2be47242-6db6-4d8d-b590-8c682dee013e/f092485f-e7d4-42be-add8-9bafec004ccb"
 					(reference "J1")
@@
 			)
 		)
-		(property "Footprint" "LED_SMD:LED_0805_2012Metric_Pad1.15x1.40mm_HandSolder"
+		(property "Footprint" "LED_THT:LED_D3.0mm"
 			(at 381 107.95 0)
 			(effects
@@
 			)
 		)
-		(property "Footprint" "LED_SMD:LED_0805_2012Metric_Pad1.15x1.40mm_HandSolder"
+		(property "Footprint" "LED_THT:LED_D3.0mm"
 			(at 386.08 114.3 0)
 			(effects
@@
 			)
 		)
-		(property "Footprint" "LED_SMD:LED_0805_2012Metric_Pad1.15x1.40mm_HandSolder"
+		(property "Footprint" "LED_THT:LED_D3.0mm"
 			(at 386.08 101.6 0)
 			(effects
@@
 			)
 		)
-		(property "Footprint" "LED_SMD:LED_0805_2012Metric_Pad1.15x1.40mm_HandSolder"
+		(property "Footprint" "LED_THT:LED_D3.0mm"
 			(at 386.08 127 0)
 			(effects
@@
 			)
 		)
-		(property "Footprint" "LED_SMD:LED_0805_2012Metric_Pad1.15x1.40mm_HandSolder"
+		(property "Footprint" "LED_THT:LED_D3.0mm"
 			(at 381 120.65 0)
 			(effects

Commit message: Exp-BP: Add display
Parts:
- added D1: BAT20J, Diode_SMD:D_SOD-323_HandSoldering, symbol AES_Library:AES-Schottky_Diode_PWR_Input
Connections:
- net +5V: now also D1.2 (A); no longer JP3.2 (B)
- new net: D1.1 (K), JP3.2 (B)
Other:
- moved on the sheet: C1, C2, JP4, R12
