File: hw/ZID_MAIN/ZID_MAIN.kicad_pcb (KiCad board)
At the start: 2 copper layers, 165.1 x 101.6 mm, 151 parts, among them J1 Conn_01x02_Pin_2.54mm, J10 USB-C PWR ONLY, J11 Conn_01x08, J2 Conn_02x05_2.54mm, J3 Conn_02x05_2.54mm, J4 Conn_02x05_PINHDR_2.54mm, J5 HDR 1x04 Socket, J6 Conn_02x03_Odd_Even, J7 Conn_01x03, J8 BRK-EXP-UNIT, J9 Z80-TARGET, M1 WS-RP2040-Zero, SW1 SW_Push, SW2 SW_DIP_x02, U1 74HCT161, U10 74FCT2245, U11 SST39SF010, U12 AS7C1024B-10J, U13 74FCT541C, U14 74AHCT244, U15 74FCT257T, U16 74HCT166, U17 74HCT166, U18 74LVC245, U19 74LVC125AS, U2 74FCT541C, U20 24LC32, U21 ATF1504AS-44T, U22 74AHCT1G125, U23 74LVC273, U24 74AHCT00, U25 74LVC2G04, U26 74AHCT1G14, U3 74FCT541C, U4 MIC2775, U5 OSC-20MHz, U6 Z80 C20MHz-PLCC, U7 ATF1508AS, U8 74FCT2245, U9 74FCT2245

Commit message: BP-EXP: 1 board only. PLCC-DIP: Adapter form.
Parts:
- removed TP2: TestPoint, Connector_PinHeader_2.54mm:PinHeader_1x01_P2.54mm_Vertical
- moved C16 6.30 mm to (67.4, 51.8)
- moved C20 6.30 mm to (67.2, 41.8)
- moved C18 6.30 mm to (67.4, 56.8)
- moved C22 6.30 mm to (67.2, 46.8)
- moved C30 4.89 mm to (247.9, 48.1)
- moved C27 4.89 mm to (247.9, 40.5)
- moved C28 4.89 mm to (247.9, 43.0)
- moved C29 4.89 mm to (247.9, 45.6)
- moved C31 4.89 mm to (247.9, 50.6)
- moved C32 4.89 mm to (247.9, 53.1)
- moved C33 4.89 mm to (247.9, 55.6)
- moved C15 4.89 mm to (239.9, 50.6)
- moved C17 4.89 mm to (239.9, 55.6)
- moved C19 4.89 mm to (243.9, 40.5)
- moved C21 4.89 mm to (243.9, 45.6)
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Connections:
- J4 pad 1: /Main Logic/JTCK -> JTCK
- J4 pad 3: /Main Logic/JTDO_CI -> JTDO_CI
- J4 pad 5: /Main Logic/JTMS -> JTMS
- J8 pad 1: LA1 -> GND
- J8 pad 10: LA8 -> LA2
- J8 pad 11: LA11 -> LA5
- J8 pad 12: LA10 -> LA4
- J8 pad 13: LA13 -> LA7
- J8 pad 14: LA12 -> LA6
- J8 pad 15: LA15 -> LA9
- J8 pad 16: LA14 -> LA8
- J8 pad 17: BA_CLK -> LA11
- J8 pad 18: D7_B -> LA10
- J8 pad 19: BA_CLR- -> LA13
- J8 pad 2: LA0 -> +5V
- J8 pad 20: unconnected-(J8-ADDO1-Pad20) -> LA12
- J8 pad 21: AEN_CLK -> LA15
- J8 pad 22: unconnected-(J8-ADDI2-Pad22) -> LA14
- J8 pad 23: AEN_CLR- -> BA_CLK
- J8 pad 24: unconnected-(J8-ADDO2-Pad24) -> D7_B
- J8 pad 25: BRKHW_DET- -> BA_CLR-
- J8 pad 26: unconnected-(J8-ADDI3-Pad26) -> D7_B
- J8 pad 27: BRK2N_AEQ- -> AEN_CLK
- J8 pad 28: D7_B -> BRKHW_DET-
- J8 pad 29: TM1- -> AEN_CLR-
- J8 pad 3: LA3 -> GND
- J8 pad 30: unconnected-(J8-AEDO1-Pad30) -> BRK2N_AEQ-
- J8 pad 31: TMREQ- -> TM1-
- J8 pad 32: unconnected-(J8-AEDI2-Pad32) -> ZRFSH-
- J8 pad 33: TIORQ- -> TMREQ-
- J8 pad 34: unconnected-(J8-AEDO2-Pad34) -> TRD-
- J8 pad 35: TWR- -> TIORQ-
- J8 pad 36: unconnected-(J8-AEDI3-Pad36) -> TWR-
- J8 pad 37: TRD- -> JTCK
- J8 pad 38: GND -> JTMS
- J8 pad 39: GND -> JTD2O3I
- J8 pad 4: LA2 -> +5V
- J8 pad 40: +5V -> JTDO_CI
- J8 pad 5: LA5 -> GND
- J8 pad 6: LA4 -> +5V
- J8 pad 7: LA7 -> LA1
- J8 pad 8: LA6 -> LA0
- J8 pad 9: LA9 -> LA3
- R10 pad 2: /Main Logic/JTDO_CI -> JTDO_CI
- R8 pad 2: /Main Logic/JTMS -> JTMS
- R9 pad 2: /Main Logic/JTCK -> JTCK
- U21 pad 26: /Main Logic/JTCK -> JTCK
- U21 pad 32: /Main Logic/JTDO_CI -> JTD2O3I
- U21 pad 7: /Main Logic/JTMS -> JTMS
- U23 pad 1: /Main Logic/RST- -> LRST-
- U24 pad 10: TRST- -> LRST-
- U24 pad 13: TRST- -> LRST-
- U24 pad 2: TRST- -> LRST-
- U24 pad 5: TRST- -> LRST-
- U7 pad 15: /Main Logic/JTMS -> JTMS
- U7 pad 50: /Main Logic/IO50 -> LRST-
- U7 pad 62: /Main Logic/JTCK -> JTCK

Commit message: ZID Main: TVS from SMC5.0 to SMA6.0
Parts:
- D12: value SMCJ5.0A -> SMAJ6.0A; footprint Diode_SMD:D_SOD-523 -> Diode_SMD:D_SMA
- J9: value Z80-TARGET -> FFC/FPC-40 Socket
- moved C1 3.53 mm to (103.1, 29.2)
- moved D12 1.21 mm to (95.8, 27.9)

Commit message: HW: Ready to lay out.
Parts:
- removed D10, D11: PESD5V0L2U, Package_TO_SOT_SMD:SOT-323_SC-70
- removed D12: SMAJ6.0A, Diode_SMD:D_SMA
- added C35: 0.1uF, Capacitor_SMD:C_0603_1608Metric, F.Cu at (362.3, 80.6)
- added C36: 0.1uF, Capacitor_SMD:C_0603_1608Metric, F.Cu at (362.3, 83.1)
- added C37: 0.1uF, Capacitor_SMD:C_0603_1608Metric, F.Cu at (362.3, 85.6)
- added C38: 0.1uF, Capacitor_SMD:C_0603_1608Metric, F.Cu at (362.3, 88.1)
- added C39: 0.1uF, Capacitor_SMD:C_0603_1608Metric, F.Cu at (362.3, 90.7)
- added C40: 0.1uF, Capacitor_SMD:C_0603_1608Metric, F.Cu at (366.4, 70.6)
- added C41: 0.1uF, Capacitor_SMD:C_0603_1608Metric, F.Cu at (366.4, 73.1)
- added C42: 0.1uF, Capacitor_SMD:C_0603_1608Metric, F.Cu at (366.4, 75.6)
- added C43: 0.1uF, Capacitor_SMD:C_0603_1608Metric, F.Cu at (366.4, 78.1)
- added C44: 0.1uF, Capacitor_SMD:C_0603_1608Metric, F.Cu at (366.4, 80.6)
- added C45: 0.1uF, Capacitor_SMD:C_0603_1608Metric, F.Cu at (366.4, 83.1)
- added C46: 0.1uF, Capacitor_SMD:C_0603_1608Metric, F.Cu at (366.4, 85.6)
- added D2: SMAJ6.0A, Diode_SMD:D_SMA, F.Cu at (299.3, 92.4)
- added D3: PESD5V0L2U, Package_TO_SOT_SMD:SOT-323_SC-70, F.Cu at (297.6, 96.6)
- added D4: PESD5V0L2U, Package_TO_SOT_SMD:SOT-323_SC-70, F.Cu at (297.6, 100.3)
- added J12: USB-C PWR ONLY, AES_Library:AES-USB_C-Molex-BdTopMnt-2171790001, F.Cu at (301.1, 69.2)
- added JA1: SolderJumper_2_Open, Jumper:SolderJumper-2_P1.3mm_Open_TrianglePad1.0x1.5mm, F.Cu at (345.1, 83.9)
- added JB1: SolderJumper_2_Open, Jumper:SolderJumper-2_P1.3mm_Open_TrianglePad1.0x1.5mm, F.Cu at (345.1, 87.4)
- added JC1: SolderJumper_2_Open, Jumper:SolderJumper-2_P1.3mm_Open_TrianglePad1.0x1.5mm, F.Cu at (345.1, 91.0)
- added JD1: SolderJumper_2_Open, Jumper:SolderJumper-2_P1.3mm_Open_TrianglePad1.0x1.5mm, F.Cu at (345.1, 94.5)
- added JP6: Jumper_2_Small_Open, Connector_PinHeader_2.00mm:PinHeader_1x02_P2.00mm_Vertical, F.Cu at (339.1, 106.0)
- added JS1: SolderJumper_2_Open, Jumper:SolderJumper-2_P1.3mm_Open_TrianglePad1.0x1.5mm, F.Cu at (345.1, 101.6)
- added OP2: AES-Option_A-B_2mm, Connector_PinHeader_2.00mm:PinHeader_1x03_P2.00mm_Vertical, F.Cu at (392.8, 8.54)
- added OP3: AES-Option_A-B, Connector_PinHeader_2.54mm:PinHeader_1x03_P2.54mm_Vertical, F.Cu at (302.1, 76.2)
- added R38: 10k, Resistor_SMD:R_0805_2012Metric, F.Cu at (372.6, 42.7)
- added R39: 1.2k, Resistor_SMD:R_0805_2012Metric, F.Cu at (372.6, 45.7)
- added R40: 10k, Resistor_SMD:R_0805_2012Metric, F.Cu at (372.6, 48.6)
- added R41: 22, Resistor_SMD:R_0805_2012Metric, F.Cu at (372.6, 51.6)
- added R42: 4.7k, Resistor_SMD:R_0805_2012Metric, F.Cu at (372.6, 54.5)
- added R43: 4.7k, Resistor_SMD:R_0805_2012Metric, F.Cu at (372.6, 57.5)
- added R44: 0, Resistor_SMD:R_0805_2012Metric_Pad1.20x1.40mm_HandSolder, F.Cu at (306.1, 88.0)
- added TP10: TestPoint, Connector_PinHeader_2.54mm:PinHeader_1x01_P2.54mm_Vertical, F.Cu at (335.8, 61.4)
- added TP11: TestPoint, Connector_PinHeader_2.54mm:PinHeader_1x01_P2.54mm_Vertical, F.Cu at (335.8, 66.0)
- added TP12: TestPoint, Connector_PinHeader_2.54mm:PinHeader_1x01_P2.54mm_Vertical, F.Cu at (335.8, 70.6)
- added TP13: TestPoint, Connector_PinHeader_2.54mm:PinHeader_1x01_P2.54mm_Vertical, F.Cu at (335.8, 75.2)
- added TP14: TestPoint, Connector_PinHeader_2.54mm:PinHeader_1x01_P2.54mm_Vertical, F.Cu at (335.8, 79.8)
- added TP15: TestPoint, Connector_PinHeader_2.54mm:PinHeader_1x01_P2.54mm_Vertical, F.Cu at (340.4, 52.3)
- added TP16: TestPoint, Connector_PinHeader_2.54mm:PinHeader_1x01_P2.54mm_Vertical, F.Cu at (340.4, 56.8)
- added TP17: TestPoint, Connector_PinHeader_2.54mm:PinHeader_1x01_P2.54mm_Vertical, F.Cu at (340.4, 61.4)
- added TP18: TestPoint, Connector_PinHeader_2.54mm:PinHeader_1x01_P2.54mm_Vertical, F.Cu at (340.4, 66.0)
- added TP19: TestPoint, Connector_PinHeader_2.54mm:PinHeader_1x01_P2.54mm_Vertical, F.Cu at (340.4, 70.6)
- added TP2: TestPoint, Connector_PinHeader_2.54mm:PinHeader_1x01_P2.54mm_Vertical, F.Cu at (331.2, 56.8)
- added TP20: TestPoint, Connector_PinHeader_2.54mm:PinHeader_1x01_P2.54mm_Vertical, F.Cu at (340.4, 75.2)
- added TP21: TestPoint, Connector_PinHeader_2.54mm:PinHeader_1x01_P2.54mm_Vertical, F.Cu at (340.4, 79.8)
- added TP22: TestPoint, Connector_PinHeader_2.54mm:PinHeader_1x01_P2.54mm_Vertical, F.Cu at (345.0, 52.3)
- added TP23: TestPoint, Connector_PinHeader_2.54mm:PinHeader_1x01_P2.54mm_Vertical, F.Cu at (345.0, 56.8)
- added TP24: TestPoint, Connector_PinHeader_2.54mm:PinHeader_1x01_P2.54mm_Vertical, F.Cu at (345.0, 61.4)
- added TP25: TestPoint, Connector_PinHeader_2.54mm:PinHeader_1x01_P2.54mm_Vertical, F.Cu at (345.0, 66.0)
- added TP26: TestPoint, Connector_PinHeader_2.54mm:PinHeader_1x01_P2.54mm_Vertical, F.Cu at (345.0, 70.6)
- added TP27: TestPoint, Connector_PinHeader_2.54mm:PinHeader_1x01_P2.54mm_Vertical, F.Cu at (345.0, 75.2)
- added U27: ATF1504AS-44T, Package_QFP:TQFP-44_10x10mm_P0.8mm, F.Cu at (314.1, -35.7)
- added U28: ATF1504AS-44T, Package_QFP:TQFP-44_10x10mm_P0.8mm, F.Cu at (314.1, -21.4)
- C3: value 0.1uF -> 100uF; footprint Capacitor_SMD:C_0603_1608Metric -> Capacitor_SMD:C_1210_3225Metric_Pad1.33x2.70mm_HandSolder
- C34: value 100uF -> 0.1uF; footprint Capacitor_SMD:C_1210_3225Metric_Pad1.33x2.70mm_HandSolder -> Capacitor_SMD:C_0603_1608Metric
- J1: value Conn_01x02_Pin_2.54mm -> HDR 1x04 Socket; footprint Connector_PinHeader_2.54mm:PinHeader_1x02_P2.54mm_Vertical -> Connector_PinSocket_2.54mm:PinSocket_1x04_P2.54mm_Vertical
- J10: value USB-C PWR ONLY -> FFC/FPC-40 Socket; footprint AES_Library:AES-USB_C-Molex-BdTopMnt-2171790001 -> AES_Library:CviLux_CF25401D0-05-NH_FFC-FPC-AES
- J11: value Conn_01x08 -> Conn_02x05_PINHDR_2.54mm; footprint Connector_PinHeader_2.54mm:PinHeader_1x08_P2.54mm_Vertical -> Connector_IDC:IDC-Header_2x05_P2.54mm_Vertical
- J2: value Conn_02x05_2.54mm -> Conn_02x03_Odd_Even; footprint AES_Library:PinHeader_2x05_AB-AES -> Connector_IDC:IDC-Header_2x03_P2.54mm_Vertical
- J3: value Conn_02x05_2.54mm -> Conn_01x02_Pin_2.54mm; footprint AES_Library:PinHeader_2x05_AB-AES -> Connector_PinHeader_2.54mm:PinHeader_1x02_P2.54mm_Vertical
- J4: value Conn_02x05_PINHDR_2.54mm -> Conn_01x03; footprint Connector_IDC:IDC-Header_2x05_P2.54mm_Vertical -> Connector_PinHeader_2.54mm:PinHeader_1x03_P2.54mm_Vertical
- J5: value HDR 1x04 Socket -> Conn_01x08; footprint Connector_PinSocket_2.54mm:PinSocket_1x04_P2.54mm_Vertical -> Connector_PinHeader_2.54mm:PinHeader_1x08_P2.54mm_Vertical
- J6: value Conn_02x03_Odd_Even -> Conn_01x08; footprint Connector_IDC:IDC-Header_2x03_P2.54mm_Vertical -> Connector_PinHeader_2.54mm:PinHeader_1x08_P2.54mm_Vertical
- J7: value Conn_01x03 -> Conn_02x04_2.54mm; footprint Connector_PinHeader_2.54mm:PinHeader_1x03_P2.54mm_Vertical -> Connector_PinHeader_2.54mm:PinHeader_2x04_P2.54mm_Vertical
- J8: value BRK-EXP-UNIT -> Conn_02x02_2.54mm; footprint Connector_PinHeader_2.54mm:PinHeader_2x20_P2.54mm_Vertical -> Connector_PinHeader_2.54mm:PinHeader_2x02_P2.54mm_Vertical
- J9: value FFC/FPC-40 Socket -> Conn_02x04_2.54mm; footprint AES_Library:CviLux_CF25401D0-05-NH_FFC-FPC-AES -> Connector_PinHeader_2.54mm:PinHeader_2x04_P2.54mm_Vertical
- JP2: value Jumper_2_Small_Open_wsto-AES -> SolderJumper_2_Open; footprint Connector_PinHeader_2.00mm:PinHeader_1x03_P2.00mm_Vertical -> Jumper:SolderJumper-2_P1.3mm_Open_RoundedPad1.0x1.5mm
- JP3: value Jumper_2_Small_Bridged -> Jumper_2_Small_Open_wsto-AES; footprint Connector_PinHeader_2.00mm:PinHeader_1x02_P2.00mm_Vertical -> Connector_PinHeader_2.00mm:PinHeader_1x03_P2.00mm_Vertical
- JP4: value SolderJumper_2_Open -> Jumper_2_Small_Bridged; footprint Jumper:SolderJumper-2_P1.3mm_Open_RoundedPad1.0x1.5mm -> Connector_PinHeader_2.00mm:PinHeader_1x02_P2.00mm_Vertical
- JP5: value Jumper_2_Small_Open -> Jumper_2_Small_Bridged
- LED1: value LED BLUE -> LED GREEN; footprint LED_THT:LED_D3.0mm -> LED_SMD:LED_0805_2012Metric
- LED10: value LED ORANGE -> LED BLUE; footprint LED_THT:LED_D3.0mm -> LED_SMD:LED_0805_2012Metric
- LED2: value LED YELLOW -> LED GREEN; footprint LED_THT:LED_D3.0mm -> LED_SMD:LED_0805_2012Metric
- LED3, LED9: value LED RED -> LED YELLOW; footprint LED_THT:LED_D3.0mm -> LED_SMD:LED_0805_2012Metric
- LED4: value LED ORANGE -> LED YELLOW; footprint LED_THT:LED_D3.0mm -> LED_SMD:LED_0805_2012Metric
- LED5: value LED GREEN -> LED RED; footprint LED_THT:LED_D3.0mm -> LED_SMD:LED_0805_2012Metric
- LED6: footprint LED_THT:LED_D3.0mm -> LED_SMD:LED_0805_2012Metric
- LED7: value LED YELLOW -> LED ORANGE; footprint LED_THT:LED_D3.0mm -> LED_SMD:LED_0805_2012Metric
- LED8: value LED YELLOW -> LED RED; footprint LED_THT:LED_D3.0mm -> LED_SMD:LED_0805_2012Metric
- R1: value 10k -> 18k
- R10: value 10k -> 0; footprint Resistor_SMD:R_0805_2012Metric -> Resistor_SMD:R_0805_2012Metric_Pad1.20x1.40mm_HandSolder
- R11, R13: value 10k -> 820
- R12: value 18k -> 10k
- R14, R16, R8, R9: value 4.7k -> 10k
- R15, R18: value 4.7k -> 820
- R17: value 22 -> 820
- R19, R20: value 4.7k -> 20k
- R2, R3: value 10k -> 6.8k
- R23, R24, R25: value 20k -> 10k
- R26: value 20k -> 4.7k
- R27, R28: value 1.2k -> 4.7k
- R30: value 1.2k -> 20k
- R31: value 0 -> 10k; footprint Resistor_SMD:R_0805_2012Metric_Pad1.20x1.40mm_HandSolder -> Resistor_SMD:R_0805_2012Metric
- R32, R35, R36: value 820 -> 1.2k
- R33: value 820 -> 10k
- R34: value 820 -> 20k
- R37: value 1.2k -> 22
- R4: value 10k -> 4.7k
- R6, R7: value 6.8k -> 4.7k
- TP1: value SYNC-CONN -> TestPoint
- TP7: value TestPoint -> SYNC-CONN
- TP9: value TestPoint -> EXT-BRK
- U1: value 74HCT161 -> OSC-20MHz; footprint Package_SO:SOIC-16_3.9x9.9mm_P1.27mm -> AES_Library:OSC-8_14-AES
- U10: value 74FCT2245 -> 74LVC2G04; footprint Package_SO:SOIC-20W_7.5x12.8mm_P1.27mm -> Package_TO_SOT_SMD:SOT-23-6
- U11: value SST39SF010 -> 74LVC125AS; footprint Package_DIP:DIP-32_W15.24mm_Socket_LongPads -> Package_SO:SOIC-14_3.9x8.7mm_P1.27mm
- U12: value AS7C1024B-10J -> 74LVC273; footprint Package_SO:SOJ-32_10.16x20.955mm_P1.27mm -> Package_SO:SOIC-20W_7.5x12.8mm_P1.27mm
- U13, U2: value 74FCT541C -> 74FCT2245
- U14: value 74AHCT244 -> AS7C1024B; footprint Package_SO:SOIC-20W_7.5x12.8mm_P1.27mm -> Package_SO:SOJ-32_10.16x20.955mm_P1.27mm
- U15: value 74FCT257T -> 74FCT2245; footprint Package_SO:SOIC-16W_7.5x10.3mm_P1.27mm -> Package_SO:SOIC-20W_7.5x12.8mm_P1.27mm
- U16, U17: value 74HCT166 -> 74FCT2245; footprint Package_SO:SOIC-16_3.9x9.9mm_P1.27mm -> Package_SO:SOIC-20W_7.5x12.8mm_P1.27mm
- U18: value 74LVC245 -> ATF1508AS; footprint Package_SO:SOIC-20W_7.5x12.8mm_P1.27mm -> Package_QFP:TQFP-100_14x14mm_P0.5mm
- U19: value 74LVC125AS -> 74HCT166; footprint Package_SO:SOIC-14_3.9x8.7mm_P1.27mm -> Package_SO:SOIC-16_3.9x9.9mm_P1.27mm
- U20: value 24LC32 -> 74FCT257T; footprint Package_SO:SOIC-8_3.9x4.9mm_P1.27mm -> Package_SO:SOIC-16W_7.5x10.3mm_P1.27mm
- U21: value ATF1504AS-44T -> 74HCT161; footprint Package_QFP:TQFP-44_10x10mm_P0.8mm -> Package_SO:SOIC-16_3.9x9.9mm_P1.27mm
- U22: value 74AHCT1G125 -> 74AHCT244; footprint Package_TO_SOT_SMD:SOT-23-5 -> Package_SO:SOIC-20W_7.5x12.8mm_P1.27mm
- U23: value 74LVC273 -> 74HCT166; footprint Package_SO:SOIC-20W_7.5x12.8mm_P1.27mm -> Package_SO:SOIC-16_3.9x9.9mm_P1.27mm
- U25: value 74LVC2G04 -> ATF1504AS-44T; footprint Package_TO_SOT_SMD:SOT-23-6 -> Package_QFP:TQFP-44_10x10mm_P0.8mm
- U26: value 74AHCT1G14 -> ATF1504AS-44T; footprint Package_TO_SOT_SMD:SOT-23-5 -> Package_QFP:TQFP-44_10x10mm_P0.8mm
- U3: value 74FCT541C -> 24LC32; footprint Package_SO:SOIC-20W_7.5x12.8mm_P1.27mm -> Package_SO:SOIC-8_3.9x4.9mm_P1.27mm
- U5: value OSC-20MHz -> SST39SF010; footprint AES_Library:OSC-8_14-AES -> Package_DIP:DIP-32_W15.24mm_Socket_LongPads
- U6: value Z80 C20MHz-PLCC -> 74LVC245; footprint Package_LCC:PLCC-44_THT-Socket -> Package_SO:SOIC-20W_7.5x12.8mm_P1.27mm
- U7: value ATF1508AS -> 74FCT2245; footprint Package_QFP:TQFP-100_14x14mm_P0.5mm -> Package_SO:SOIC-20W_7.5x12.8mm_P1.27mm
- U8: value 74FCT2245 -> 74HCT14; footprint Package_SO:SOIC-20W_7.5x12.8mm_P1.27mm -> Package_SO:SOIC-14_3.9x8.7mm_P1.27mm
- U9: value 74FCT2245 -> Z80 C20MHz-PLCC; footprint Package_SO:SOIC-20W_7.5x12.8mm_P1.27mm -> Package_LCC:PLCC-44
- moved LED9 334.7 mm to (408.3, 102.4), turned to 0 degrees
- moved LED8 334.6 mm to (408.3, 99.3), turned to 0 degrees
- moved LED7 334.5 mm to (408.3, 96.3), turned to 0 degrees
- moved LED6 334.5 mm to (408.3, 93.2), turned to 0 degrees
- moved LED5 330.0 mm to (403.9, 105.4), turned to 0 degrees
- moved SW2 329.4 mm to (401.2, 62.2)
- moved J10 317.2 mm to (392.2, 18.1), turned to 0 degrees
- moved JP3 313.9 mm to (384.7, 8.54), turned to 0 degrees
- moved U23 305.2 mm to (395.9, 44.2), turned to 0 degrees
- moved J6 303.6 mm to (400.8, 71.6), turned to 0 degrees
- moved U20 294.7 mm to (399.4, 29.2), turned to 0 degrees
- moved R33 294.1 mm to (368.2, 48.6)
- moved R31 293.2 mm to (368.2, 42.7)
- moved R36 292.9 mm to (368.2, 57.5)
- moved R32 292.7 mm to (368.2, 45.7)
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Connections:
- C1 pad 1: GND -> +3.3V
- C1 pad 2: +3.3V -> GND
- C16 pad 2: +3.3V -> +5V
- C18 pad 2: +3.3V -> +5V
- C2 pad 1: +3.3V -> GND
- C2 pad 2: GND -> +3.3V
- C20 pad 2: +3.3V -> +5V
- C22 pad 2: +3.3V -> +5V
- C3 pad 1: GND -> +5V
- C3 pad 2: +5V -> GND
- C34 pad 1: +5V -> GND
- C34 pad 2: GND -> +5V
- C4 pad 2: +5V -> +3.3V
- C5 pad 2: +5V -> +3.3V
- C6 pad 2: +5V -> +3.3V
- C7 pad 2: +5V -> +3.3V
- J1 pad 1: GND -> +3.3V
- J1 pad 2: Net-(J1-Pin_2) -> GND
- J11 pad 1: TD0 -> /JTCK
- J11 pad 2: TD1 -> GND
- J11 pad 3: TD2 -> /JTDO_CI
- J11 pad 4: TD3 -> +5V
- J11 pad 5: TD4 -> /JTMS
- J11 pad 6: TD5 -> unconnected-(J11-Pin_6-Pad6)
- J11 pad 7: TD6 -> unconnected-(J11-Pin_7-Pad7)
- J11 pad 8: TD7 -> unconnected-(J11-Pin_8-Pad8)
- J4 pad 1: JTCK -> GND
- J4 pad 2: GND -> /SPICS-
- J4 pad 3: JTDO_CI -> /SPIMI
- J5 pad 1: +3.3V -> GND
- J5 pad 2: GND -> /ZRFSH-
- J5 pad 3: /Main Logic/SCK_RX -> /ZM1-
- J5 pad 4: /Main Logic/SDA_TX -> /ZMREQ-
- J6 pad 1: /Main Logic/SPIMI -> /TD0
- J6 pad 2: +3.3V -> /TD1
- J6 pad 3: /Main Logic/SPICK -> /TD2
- J6 pad 4: /Main Logic/SPIMO -> /TD3
- J6 pad 5: /Main Logic/SPICS2- -> /TD4
- J6 pad 6: GND -> /TD5
- J7 pad 1: GND -> (no net)
- J7 pad 2: /Main Logic/SPICS- -> (no net)
- J7 pad 3: /Main Logic/SPIMI -> (no net)
- J8 pad 1: GND -> (no net)
- J8 pad 2: +5V -> (no net)
- J8 pad 3: GND -> (no net)
- J8 pad 4: +5V -> (no net)
- J9 pad 1: TA11 -> (no net)
- J9 pad 2: TA12 -> (no net)
- J9 pad 3: TA13 -> (no net)
- J9 pad 4: TA14 -> (no net)
- J9 pad 5: TA15 -> (no net)
- J9 pad 6: CLK -> (no net)
- J9 pad 7: TD4 -> (no net)
- J9 pad 8: TD3 -> (no net)
- JP1 pad 2: /Main Logic/_RST- -> /_CLK
- JP1 pad 3: TRST- -> /TCLK
- JP2 pad 1: unconnected-(JP2-A-Pad1) -> GND
- JP2 pad 2: /Main Logic/_CLK -> Net-(JP2-B)
- JP3 pad 1: Net-(JP3-A) -> unconnected-(JP3-A-Pad1)
- JP3 pad 2: Net-(D1-K) -> /RST-
- JP4 pad 1: GND -> Net-(JP4-A)
- JP4 pad 2: Net-(JP4-B) -> Net-(D1-K)
- JP5 pad 1: MODINT- -> /ZRST-
- JP5 pad 2: TINT- -> Net-(JP5-B)
- M1 pad 1: /Main Logic/SDA_TX -> /SDA_TX
- M1 pad 10: /Main Logic/V3D7 -> /V3D7
- M1 pad 11: /Main Logic/MA0 -> /MA0
- M1 pad 12: /Main Logic/MRD- -> /MRD-
- M1 pad 13: /Main Logic/MWR- -> /MSEL-
- M1 pad 14: /Main Logic/MSEL- -> /MWTRQ-
- M1 pad 15: /Main Logic/MWTRQ- -> /MRST-
- M1 pad 16: /Main Logic/IOECLK -> /IOECLK
- M1 pad 17: /Main Logic/SPICK -> /SPICK
- M1 pad 18: /Main Logic/SPIMO -> /SPIMO
- M1 pad 19: /Main Logic/SPIMI -> /SPIMI
- M1 pad 2: /Main Logic/SCK_RX -> /SCK_RX
- M1 pad 20: /Main Logic/SPICS- -> /SPICS-
- M1 pad 23: Net-(JP3-A) -> Net-(JP4-A)
- M1 pad 3: /Main Logic/V3D0 -> /V3D0
- M1 pad 4: /Main Logic/V3D1 -> /V3D1
- M1 pad 5: /Main Logic/V3D2 -> /V3D2
- M1 pad 6: /Main Logic/V3D3 -> /V3D3
- M1 pad 7: /Main Logic/V3D4 -> /V3D4
- M1 pad 8: /Main Logic/V3D5 -> /V3D5
- M1 pad 9: /Main Logic/V3D6 -> /V3D6
- OP1 pad 1: /Main Logic/PU -> unconnected-(OP1-A-Pad1)
- OP1 pad 3: /Main Logic/RFMR- -> /RFMR-
- R1 pad 1: +5V -> +3.3V
- R1 pad 2: Net-(U1-CET) -> Net-(JP2-B)
- R10 pad 1: +5V -> GND
- R10 pad 2: JTDO_CI -> Net-(SD1-SHLD)
- R11 pad 1: +5V -> Net-(LED1-K)
- R11 pad 2: /Main Logic/PU -> GND
- R12 pad 2: Net-(JP4-B) -> /MWTRQ-
- R13 pad 1: +3.3V -> Net-(LED2-K)
- R13 pad 2: /Main Logic/MWTRQ- -> GND
- R14 pad 1: /Main Logic/SPICS- -> +5V
- R14 pad 2: +3.3V -> Net-(JP5-B)
- R15 pad 1: /Main Logic/SPIMO -> Net-(LED3-K)
- R15 pad 2: +3.3V -> GND
- R16 pad 1: /Main Logic/SPIMI -> /SBCMODE-
- R16 pad 2: +3.3V -> +5V
- R17 pad 1: Net-(R17-Pad1) -> Net-(LED4-K)
- R17 pad 2: Net-(R17-Pad2) -> GND
- R18 pad 1: /Main Logic/SPICK -> Net-(LED5-A)
- R19 pad 2: BRKHW_DET- -> /TINT-
- R2 pad 1: +5V -> /SCK_RX
- R2 pad 2: /Main Logic/TGTONLY- -> +3.3V
- R20 pad 2: BRK2N_AEQ- -> /TNMI-
- R21 pad 2: TINT- -> /TWAIT-
- R22 pad 2: TNMI- -> /TBREQ-
- R23 pad 1: +5V -> Net-(OP1-C)
- R23 pad 2: TBREQ- -> +5V
- R24 pad 2: TWAIT- -> Net-(U21-CET)
- R25 pad 1: ZBACK- -> +5V
- R25 pad 2: +5V -> /JTDO_CI
- R26 pad 1: ZHALT- -> +5V
- R26 pad 2: +5V -> /JTCK
- R27 pad 1: Net-(LED1-K) -> +5V
- R27 pad 2: GND -> /JTMS
- R28 pad 1: Net-(LED2-K) -> +5V
- R28 pad 2: GND -> /JTDI_CO
- R29 pad 1: Net-(LED3-K) -> Net-(LED6-K)
- R3 pad 1: +5V -> /SDA_TX
- R3 pad 2: /Main Logic/SBC_GPI3 -> +3.3V
- R30 pad 1: Net-(LED4-K) -> /ZBACK-
- R30 pad 2: GND -> +5V
- R31 pad 1: Net-(J10-SHIELD-PadSH1) -> /PU
- R31 pad 2: GND -> +5V
- R32 pad 1: Net-(LED6-K) -> Net-(LED7-K)
- R32 pad 2: +3.3V -> GND
- R33 pad 1: Net-(LED8-K) -> /TWAITRQ-
- R33 pad 2: +3.3V -> +5V
- R34 pad 1: Net-(LED5-K) -> /ZHALT-
- R34 pad 2: +3.3V -> +5V
- R35 pad 1: Net-(LED7-K) -> Net-(LED8-K)
- R35 pad 2: +3.3V -> GND
- R36 pad 1: Net-(LED9-A) -> Net-(LED9-K)
- R36 pad 2: +3.3V -> GND
- R37 pad 1: Net-(LED10-K) -> Net-(R37-Pad1)
- R37 pad 2: GND -> Net-(R37-Pad2)
- R4 pad 1: /Main Logic/SBCMODE- -> /SPIMO
- R4 pad 2: +5V -> +3.3V
- R5 pad 1: +5V -> /SPICK
- R5 pad 2: /Main Logic/JTDI_CO -> +3.3V
- R6 pad 1: /Main Logic/SCK_RX -> /SPICS-
- R7 pad 1: /Main Logic/SDA_TX -> /SPIMI
- R8 pad 2: JTMS -> /TGTONLY-
- R9 pad 2: JTCK -> /SBC_GPI3
- RN1 pad 2: /Main Logic/ZA12 -> /ZA12
- RN1 pad 3: /Main Logic/ZA11 -> /ZA11
- RN1 pad 4: /Main Logic/ZA10 -> /ZA10
- RN1 pad 5: /Main Logic/ZA9 -> /ZA9
- RN1 pad 6: /Main Logic/ZA13 -> /ZA13
- RN1 pad 7: /Main Logic/ZA8 -> /ZA8
- RN1 pad 8: /Main Logic/ZA14 -> /ZA14
- RN1 pad 9: /Main Logic/ZA15 -> /ZA15
- SBC1 pad 1: TRST- -> /TCLK
- SBC1 pad 2: /Main Logic/RST- -> /CLK
- SBC1 pad 3: /Main Logic/_RST- -> /_CLK
- SBC2 pad 1: /Main Logic/TCLK -> /TRST-
- SBC2 pad 2: CLK -> /BRD_RST-
- SBC2 pad 3: /Main Logic/_CLK -> /RST-
- SBC3 pad 2: /Main Logic/SBCMODE- -> /SBCMODE-
- SD1 pad 10: GND -> Net-(SD1-SHLD)
- SD1 pad 2: /Main Logic/SPICS- -> /SPICS-
- SD1 pad 3: /Main Logic/SPIMO -> /SPIMO
- SD1 pad 5: /Main Logic/SPICK -> /SPICK
- SD1 pad 7: /Main Logic/SPIMI -> /SPIMI
- SW1 pad 2: Net-(J1-Pin_2) -> Net-(J3-Pin_2)
- SW2 pad 3: /Main Logic/SBC_GPI3 -> /SBC_GPI3
- SW2 pad 4: /Main Logic/TGTONLY- -> /TGTONLY-
- TP1 pad 1: Net-(R17-Pad1) -> /_CLK
- TP3 pad 1: /Main Logic/IO65 -> /IO78
- TP4 pad 1: /Main Logic/IO63 -> /IO77
- TP5 pad 1: /Main Logic/IO8 -> /LCL_IO
- TP6 pad 1: /Main Logic/IO10 -> /IO83
- TP7 pad 1: /Main Logic/IO2 -> Net-(R37-Pad1)
- TP8 pad 1: /Main Logic/IO1 -> GND
- TP9 pad 1: GND -> Net-(R40-Pad2)
- U1 pad 1: TGTMODE- -> +5V
- U1 pad 10: Net-(U1-CET) -> unconnected-(U1-NC10-Pad10)
- U1 pad 11: unconnected-(U1-Q3-Pad11) -> /_CLK
- U1 pad 12: /Main Logic/SOPNOW -> unconnected-(U1-NC12-Pad12)
- U1 pad 14: unconnected-(U1-Q0-Pad14) -> +5V
- U1 pad 2: /Main Logic/MEMOP -> unconnected-(U1-NC2-Pad2)
- U1 pad 3: Net-(U1-CET) -> unconnected-(U1-NC3-Pad3)
- U1 pad 4: Net-(U1-CET) -> GND
- U1 pad 5: Net-(U1-CET) -> unconnected-(U1-NC5-Pad5)
- U1 pad 6: Net-(U1-CET) -> unconnected-(U1-NC6-Pad6)
- U1 pad 7: /Main Logic/TGTGO -> GND
- U1 pad 8: GND -> /_CLK
- U1 pad 9: Net-(U1-CET) -> unconnected-(U1-NC9-Pad9)
- U10 pad 1: /Main Logic/TDBUSIN- -> Net-(U12-Q1)
- U10 pad 2: /Main Logic/ZD0 -> GND
- U10 pad 3: /Main Logic/ZD1 -> Net-(U12-Q2)
- U10 pad 4: /Main Logic/ZD2 -> /SPICS2-
- U10 pad 5: /Main Logic/ZD3 -> +3.3V
- U10 pad 6: /Main Logic/ZD4 -> /MINT-
- U11 pad 10: /Main Logic/ZA2 -> GND
- U11 pad 11: /Main Logic/ZA1 -> /MRST-
- U11 pad 12: /Main Logic/ZA0 -> /LRST-
- U11 pad 13: /Main Logic/ZD0 -> GND
- U11 pad 14: /Main Logic/ZD1 -> +3.3V
- U11 pad 2: /Main Logic/RRA2 -> /MOD_SEL-
- U11 pad 3: /Main Logic/RRA1 -> /MSEL-
- U11 pad 4: /Main Logic/ZA12 -> GND
- U11 pad 5: /Main Logic/ZA7 -> /ZA0
- U11 pad 6: /Main Logic/ZA6 -> /MA0
- U11 pad 7: /Main Logic/ZA5 -> GND
- U11 pad 8: /Main Logic/ZA4 -> /MRD-
- U11 pad 9: /Main Logic/ZA3 -> /ZRD-
- U12 pad 1: unconnected-(U12-NC-Pad1) -> /MRST-
- U12 pad 10: /Main Logic/ZA2 -> GND
- U12 pad 11: /Main Logic/ZA1 -> /IOECLK
- U12 pad 12: /Main Logic/ZA0 -> Net-(LED2-A)
- U12 pad 13: /Main Logic/ZD0 -> /V3D4
- U12 pad 14: /Main Logic/ZD1 -> /V3D5
- U12 pad 15: /Main Logic/ZD2 -> Net-(LED3-A)
- U12 pad 16: GND -> Net-(LED4-A)
- U12 pad 17: /Main Logic/ZD3 -> /V3D6
- U12 pad 18: /Main Logic/ZD4 -> /V3D7
- U12 pad 19: /Main Logic/ZD5 -> Net-(LED5-K)
- U12 pad 2: /Main Logic/RRA2 -> /ATTN
- U12 pad 20: /Main Logic/ZD6 -> +3.3V
- U12 pad 3: /Main Logic/RRA0 -> /V3D0
- U12 pad 4: /Main Logic/ZA12 -> /V3D1
- U12 pad 5: /Main Logic/ZA7 -> Net-(U12-Q1)
- U12 pad 6: /Main Logic/ZA6 -> Net-(U12-Q2)
- U12 pad 7: /Main Logic/ZA5 -> /V3D2
- U12 pad 8: /Main Logic/ZA4 -> /V3D3
- U12 pad 9: /Main Logic/ZA3 -> Net-(LED1-A)
- U13 pad 1: GND -> /TDBUSIN-
- U13 pad 11: TM1- -> /TD7
- U13 pad 12: /Main Logic/SBC_GPI2 -> /TD6
- U13 pad 13: /Main Logic/SBC_GPI1 -> /TD5
- U13 pad 14: /Main Logic/SBC_GPI0 -> /TD4
- U13 pad 15: /Main Logic/SBC_O3 -> /TD3
- U13 pad 16: /Main Logic/SBC_O2 -> /TD2
- U13 pad 17: /Main Logic/SBC_O1 -> /TD1
- U13 pad 18: /Main Logic/SBC_O0 -> /TD0
- U13 pad 19: GND -> /TDBUSEN-
- U13 pad 2: /Main Logic/SBC_GPO0 -> /ZD0
- U13 pad 3: /Main Logic/SBC_GPO1 -> /ZD1
- U13 pad 4: /Main Logic/SBC_GPO2 -> /ZD2
- U13 pad 5: /Main Logic/SBC_GPO3 -> /ZD3
- U13 pad 6: /Main Logic/SBC_I0 -> /ZD4
- U13 pad 7: /Main Logic/SBC_I1 -> /ZD5
- U13 pad 8: /Main Logic/SBC_I2 -> /ZD6
- U13 pad 9: ZM1- -> /ZD7
- U14 pad 1: ZBACK- -> unconnected-(U14-NC-Pad1)
- U14 pad 10: GND -> /ZA2
- U14 pad 11: TNMI- -> /ZA1
- U14 pad 12: ZMREQ- -> /ZA0
- U14 pad 13: TBREQ- -> /ZD0
- U14 pad 14: ZIORQ- -> /ZD1
- U14 pad 15: TINT- -> /ZD2
- U14 pad 16: ZRD- -> GND
- U14 pad 17: TWAIT- -> /ZD3
- U14 pad 18: ZWR- -> /ZD4
- U14 pad 19: GND -> /ZD5
- U14 pad 2: TWR- -> /RRA2
- U14 pad 20: +5V -> /ZD6
- U14 pad 3: /Main Logic/WAIT- -> /RRA0
- U14 pad 4: TRD- -> /ZA12
- U14 pad 5: /Main Logic/INT- -> /ZA7
- U14 pad 6: TIORQ- -> /ZA6
- U14 pad 7: /Main Logic/BUSREQ- -> /ZA5
- U14 pad 8: TMREQ- -> /ZA4
- U14 pad 9: /Main Logic/NMI- -> /ZA3
- U15 pad 1: /Main Logic/FIXED_SEL -> GND
- U15 pad 10: Net-(OP1-C) -> GND
- U15 pad 11: ZMREQ- -> /ZA7
- U15 pad 12: TIORQ- -> /ZA6
- U15 pad 13: /Main Logic/PU -> /ZA5
- U15 pad 14: ZIORQ- -> /ZA4
- U15 pad 15: /Main Logic/BUSACK -> /ZA3
- U15 pad 16: +5V -> /ZA2
- U15 pad 2: ZWR- -> /LA0
- U15 pad 3: /Main Logic/PU -> /LA1
- U15 pad 4: TWR- -> /LA2
- U15 pad 5: ZRD- -> /LA3
- U15 pad 6: /Main Logic/PU -> /LA4
- U15 pad 7: TRD- -> /LA5
- U15 pad 8: GND -> /LA6
- U15 pad 9: TMREQ- -> /LA7
- U16 pad 10: /Main Logic/ZA11 -> GND
- U16 pad 11: /Main Logic/ZA10 -> /ZM1-
- U16 pad 12: /Main Logic/ZA9 -> /SBC_I2
- U16 pad 13: Net-(U16-Qh) -> /SBC_I1
- U16 pad 14: /Main Logic/ZA8 -> /SBC_I0
- U16 pad 15: TGTMODE- -> /SBC_GPO3
- U16 pad 16: +5V -> /SBC_GPO2
- U16 pad 2: /Main Logic/ZA15 -> /SBC_O0
- U16 pad 3: /Main Logic/ZA14 -> /SBC_O1
- U16 pad 4: /Main Logic/ZA13 -> /SBC_O2
- U16 pad 5: /Main Logic/ZA12 -> /SBC_O3
- U16 pad 6: GND -> /SBC_GPI0
- U16 pad 7: /Main Logic/PCSAV_CLK -> /SBC_GPI1
- U16 pad 8: GND -> /SBC_GPI2
- U16 pad 9: /Main Logic/PU -> /TM1-
- U17 pad 1: Net-(U16-Qh) -> GND
- U17 pad 10: /Main Logic/ZA3 -> GND
- U17 pad 11: /Main Logic/ZA2 -> /ZA15
- U17 pad 12: /Main Logic/ZA1 -> /ZA14
- U17 pad 13: /Main Logic/PCRD_DIN -> /ZA13
- U17 pad 14: /Main Logic/ZA0 -> /ZA12
- U17 pad 15: TGTMODE- -> /ZA11
- U17 pad 16: +5V -> /ZA10
- U17 pad 2: /Main Logic/ZA7 -> /LA8
- U17 pad 3: /Main Logic/ZA6 -> /LA9
- U17 pad 4: /Main Logic/ZA5 -> /LA10
- U17 pad 5: /Main Logic/ZA4 -> /LA11
- U17 pad 6: GND -> /LA12
- U17 pad 7: /Main Logic/PCSAV_CLK -> /LA13
- U17 pad 8: GND -> /LA14
- U17 pad 9: /Main Logic/PU -> /LA15
- U18 pad 1: ZRD- -> /ZA1
- U18 pad 10: GND -> /ZA14
- U18 pad 11: /Main Logic/V3D7 -> GND
- U18 pad 12: /Main Logic/V3D6 -> /ZWR-
- U18 pad 13: /Main Logic/V3D5 -> /ZA4
- U18 pad 14: /Main Logic/V3D4 -> /ZA3
- U18 pad 15: /Main Logic/V3D3 -> /JTMS
- U18 pad 16: /Main Logic/V3D2 -> /SBC_GPO1
- U18 pad 17: /Main Logic/V3D1 -> /SBC_GPO0
- U18 pad 18: /Main Logic/V3D0 -> +5V
- U18 pad 19: /Main Logic/MOD_SEL- -> /ZA2
- U18 pad 2: /Main Logic/ZD0 -> /ZRD-
- U18 pad 20: +3.3V -> /SBC_GPI3
- U18 pad 3: /Main Logic/ZD1 -> +5V
- U18 pad 4: /Main Logic/ZD2 -> /JTDI_CO
- U18 pad 5: /Main Logic/ZD3 -> /ZD6
- U18 pad 6: /Main Logic/ZD4 -> /ZD0
- U18 pad 7: /Main Logic/ZD5 -> /ZD7
- U18 pad 8: /Main Logic/ZD6 -> /MWTRQ-
- U18 pad 9: /Main Logic/ZD7 -> /ZA15
- U19 pad 10: GND -> /ZA11
- U19 pad 11: /Main Logic/MWR- -> /ZA10
- U19 pad 12: ZWR- -> /ZA9
- U19 pad 13: GND -> Net-(U19-Qh)
- U19 pad 14: +3.3V -> /ZA8
- U19 pad 2: /Main Logic/MOD_SEL- -> /ZA15
- U19 pad 3: /Main Logic/MSEL- -> /ZA14
- U19 pad 4: GND -> /ZA13
- U19 pad 5: /Main Logic/ZA0 -> /ZA12
- U19 pad 6: /Main Logic/MA0 -> GND
- U19 pad 7: GND -> /BRKPC_RD-
- U19 pad 8: /Main Logic/MRD- -> GND
- U19 pad 9: ZRD- -> /PU
- U2 pad 1: GND -> /ZBACK-
- U2 pad 11: LA7 -> /TA0
- U2 pad 12: LA6 -> /TA1
- U2 pad 13: LA5 -> /TA2
- U2 pad 14: LA4 -> /TA3
- U2 pad 15: LA3 -> /TA4
- U2 pad 16: LA2 -> /TA5
- U2 pad 17: LA1 -> /TA6
- U2 pad 18: LA0 -> /TA7
- U2 pad 19: GND -> /ZRST-
- U2 pad 2: /Main Logic/ZA0 -> /ZA7
- U2 pad 3: /Main Logic/ZA1 -> /ZA6
- U2 pad 4: /Main Logic/ZA2 -> /ZA5
- U2 pad 5: /Main Logic/ZA3 -> /ZA4
- U2 pad 6: /Main Logic/ZA4 -> /ZA3
- U2 pad 7: /Main Logic/ZA5 -> /ZA2
- U2 pad 8: /Main Logic/ZA6 -> /ZA1
- U2 pad 9: /Main Logic/ZA7 -> /ZA0
- U20 pad 1: Net-(JP4-B) -> /FIXED_SEL
- U20 pad 2: GND -> /ZWR-
- U20 pad 3: GND -> /PU
- U20 pad 4: GND -> /TWR-
- U20 pad 5: /Main Logic/SDA_TX -> /ZRD-
- U20 pad 6: /Main Logic/SCK_RX -> /PU
- U20 pad 7: GND -> /TRD-
- U20 pad 8: +3.3V -> GND
- U21 pad 1: /Main Logic/JTD1O2I -> /TGTMODE-
- U21 pad 10: /Main Logic/IO10 -> Net-(U21-CET)
- U21 pad 11: LA0 -> unconnected-(U21-Q3-Pad11)
- U21 pad 12: LA1 -> unconnected-(U21-Q2-Pad12)
- U21 pad 13: LA2 -> unconnected-(U21-Q1-Pad13)
- U21 pad 14: LA3 -> unconnected-(U21-Q0-Pad14)
- U21 pad 15: LA4 -> /TGTNOW
- U21 pad 16: GND -> +5V
- U21 pad 2: /Main Logic/AE_DOUT -> /MEMOP-
- U21 pad 3: /Main Logic/BA_DOUT -> Net-(U21-CET)
- U21 pad 4: GND -> Net-(U21-CET)
- U21 pad 5: BRKHW_DET- -> Net-(U21-CET)
- U21 pad 6: D7_B -> Net-(U21-CET)
- U21 pad 7: JTMS -> /TGTGO
- U21 pad 8: /Main Logic/IO8 -> GND
- U21 pad 9: +5V -> Net-(U21-CET)
- U22 pad 1: GND -> /ZBACK-
- U22 pad 2: /Main Logic/SYNC -> /ZWR-
- U22 pad 3: GND -> /TWAITB-
- U22 pad 4: Net-(R17-Pad2) -> /ZRD-
- U22 pad 5: +5V -> /TINTB-
- U23 pad 1: LRST- -> Net-(U19-Qh)
- U23 pad 10: GND -> /ZA3
- U23 pad 11: /Main Logic/IOECLK -> /ZA2
- U23 pad 12: Net-(LED6-A) -> /ZA1
- U23 pad 13: /Main Logic/V3D4 -> /PCRD_DIN
- U23 pad 14: /Main Logic/V3D5 -> /ZA0
- U23 pad 15: Net-(LED7-A) -> /PC_LATCH-
- U23 pad 16: Net-(LED8-A) -> +5V
- U23 pad 2: /Main Logic/ATTN -> /ZA7
- U23 pad 3: /Main Logic/V3D0 -> /ZA6
- U23 pad 4: /Main Logic/V3D1 -> /ZA5
- U23 pad 5: Net-(U23-Q1) -> /ZA4
- U23 pad 6: Net-(U23-Q2) -> GND
- U23 pad 7: /Main Logic/V3D2 -> /BRKPC_RD-
- U23 pad 8: /Main Logic/V3D3 -> GND
- U23 pad 9: Net-(LED5-A) -> /PU
- U24 pad 1: TGTMODE- -> /TGTMODE-
- U24 pad 10: LRST- -> /LRST-
- U24 pad 11: Net-(LED4-A) -> Net-(LED9-A)
- U24 pad 12: TWAIT- -> /TWAIT-
- U24 pad 13: LRST- -> /LRST-
- U24 pad 2: LRST- -> /LRST-
- U24 pad 3: Net-(LED1-A) -> Net-(LED6-A)
- U24 pad 4: ZBACK- -> /ZBACK-
- U24 pad 5: LRST- -> /LRST-
- U24 pad 6: Net-(LED2-A) -> Net-(LED7-A)
- U24 pad 8: Net-(LED3-A) -> Net-(LED8-A)
- U24 pad 9: ZHALT- -> /ZHALT-
- U25 pad 1: Net-(U23-Q1) -> /JTD1O2I
- U25 pad 2: GND -> /ENBL_DOA
- U25 pad 3: Net-(U23-Q2) -> /ADDR_DOA
- U25 pad 4: /Main Logic/SPICS2- -> GND
- U25 pad 5: +3.3V -> /BRKHW_DET-
- U25 pad 6: /Main Logic/MINT- -> /D7_B
- U26 pad 1: unconnected-(U26-NC-Pad1) -> /JTD2O3I
- U26 pad 2: ZBACK- -> /ENBL_DOB
- U26 pad 3: GND -> /ADDR_DOB
- U26 pad 4: /Main Logic/BUSACK -> GND
- U26 pad 5: +5V -> /BRKHW_DET-
- U3 pad 1: GND -> Net-(JP2-B)
- U3 pad 2: /Main Logic/ZA8 -> GND
- U3 pad 3: /Main Logic/ZA9 -> GND
- U3 pad 4: /Main Logic/ZA10 -> GND
- U3 pad 5: /Main Logic/ZA11 -> /SDA_TX
- U3 pad 6: /Main Logic/ZA12 -> /SCK_RX
- U3 pad 7: /Main Logic/ZA13 -> GND
- U3 pad 8: /Main Logic/ZA14 -> +3.3V
- U4 pad 1: /Main Logic/_RST- -> /RST-
- U4 pad 4: Net-(J1-Pin_2) -> Net-(J3-Pin_2)
- U5 pad 1: +5V -> GND
- U5 pad 10: unconnected-(U5-NC10-Pad10) -> /ZA2
- U5 pad 11: /Main Logic/_CLK -> /ZA1
- U5 pad 12: unconnected-(U5-NC12-Pad12) -> /ZA0
- U5 pad 13: unconnected-(U5-NC13-Pad13) -> /ZD0
- U5 pad 14: +5V -> /ZD1
- U5 pad 2: unconnected-(U5-NC2-Pad2) -> /RRA2
- U5 pad 3: unconnected-(U5-NC3-Pad3) -> /RRA1
- U5 pad 4: GND -> /ZA12
- U5 pad 5: unconnected-(U5-NC5-Pad5) -> /ZA7
- U5 pad 6: unconnected-(U5-NC6-Pad6) -> /ZA6
- U5 pad 7: GND -> /ZA5
- U5 pad 8: /Main Logic/_CLK -> /ZA4
- U5 pad 9: unconnected-(U5-NC9-Pad9) -> /ZA3
- U6 pad 1: /Main Logic/ZA11 -> /ZRD-
- U6 pad 10: /Main Logic/ZD5 -> GND
- U6 pad 11: /Main Logic/ZD6 -> /V3D7
- U6 pad 12: unconnected-(U6-NC-Pad12) -> /V3D6
- U6 pad 13: +5V -> /V3D5
- U6 pad 14: /Main Logic/ZD2 -> /V3D4
- U6 pad 15: /Main Logic/ZD7 -> /V3D3
- U6 pad 16: /Main Logic/ZD0 -> /V3D2
- U6 pad 17: /Main Logic/ZD1 -> /V3D1
- U6 pad 18: ZINT- -> /V3D0
- U6 pad 19: ZNMI- -> /MOD_SEL-
- U6 pad 2: /Main Logic/ZA12 -> /ZD0
- U6 pad 20: ZHALT- -> +3.3V
- U6 pad 3: /Main Logic/ZA13 -> /ZD1
- U6 pad 4: /Main Logic/ZA14 -> /ZD2
- U6 pad 5: /Main Logic/ZA15 -> /ZD3
- U6 pad 6: unconnected-(U6-NC-Pad6) -> /ZD4
- U6 pad 7: CLK -> /ZD5
- U6 pad 8: /Main Logic/ZD4 -> /ZD6
- U6 pad 9: /Main Logic/ZD3 -> /ZD7
- U7 pad 1: /Main Logic/IO1 -> /ZBACK-
- U7 pad 10: /Main Logic/TGTGO -> GND
- U7 pad 11: GND -> /TA8
- U7 pad 12: /Main Logic/RRA0 -> /TA9
- U7 pad 13: /Main Logic/RRA1 -> /TA10
- U7 pad 14: /Main Logic/RRA2 -> /TA11
- U7 pad 15: JTMS -> /TA12
- U7 pad 16: /Main Logic/ZD0 -> /TA13
- U7 pad 17: /Main Logic/ZD1 -> /TA14
- U7 pad 18: +5V -> /TA15
- U7 pad 19: /Main Logic/ZD2 -> /ZRST-
- U7 pad 2: /Main Logic/IO2 -> /ZA15
- U7 pad 20: /Main Logic/ZD3 -> +5V
- U7 pad 3: +5V -> /ZA14
- U7 pad 4: /Main Logic/JTDI_CO -> /ZA13
- U7 pad 5: BRK2N_AEQ- -> /ZA12
- U7 pad 6: /Main Logic/INT- -> /ZA11
- U7 pad 7: /Main Logic/PCRD_DIN -> /ZA10
- U7 pad 8: BRKHW_DET- -> /ZA9
- U7 pad 9: TGTMODE- -> /ZA8
- U8 pad 1: ZBACK- -> /ROM_SEL
- U8 pad 10: GND -> /ZBACK
- U8 pad 11: TA0 -> /ZBACK-
- U8 pad 12: TA1 -> Net-(TP27-Pad1)
- U8 pad 13: TA2 -> Net-(JS1-B)
- U8 pad 14: TA3 -> +5V
- U8 pad 2: /Main Logic/ZA7 -> /ROM_SEL-
- U8 pad 3: /Main Logic/ZA6 -> /SYNC
- U8 pad 4: /Main Logic/ZA5 -> Net-(R37-Pad2)
- U8 pad 5: /Main Logic/ZA4 -> Net-(R41-Pad2)
- U8 pad 6: /Main Logic/ZA3 -> Net-(OP3-A)
- U8 pad 7: /Main Logic/ZA2 -> GND
- U8 pad 8: /Main Logic/ZA1 -> Net-(OP3-B)
- U8 pad 9: /Main Logic/ZA0 -> Net-(OP3-A)
- U9 pad 1: ZBACK- -> /ZA11
- U9 pad 10: GND -> /ZD5
- U9 pad 11: TA8 -> /ZD6
- U9 pad 12: TA9 -> unconnected-(U9-NC-Pad12)
- U9 pad 13: TA10 -> +5V
- U9 pad 14: TA11 -> /ZD2
- U9 pad 15: TA12 -> /ZD7
- U9 pad 16: TA13 -> /ZD0
- U9 pad 17: TA14 -> /ZD1
- U9 pad 18: TA15 -> /ZINT-
- U9 pad 19: ZRST- -> /ZNMI-
- U9 pad 2: /Main Logic/ZA15 -> /ZA12
- U9 pad 20: +5V -> /ZHALT-
- U9 pad 3: /Main Logic/ZA14 -> /ZA13
- U9 pad 4: /Main Logic/ZA13 -> /ZA14
- U9 pad 5: /Main Logic/ZA12 -> /ZA15
- U9 pad 6: /Main Logic/ZA11 -> unconnected-(U9-NC-Pad6)
- U9 pad 7: /Main Logic/ZA10 -> /CLK
- U9 pad 8: /Main Logic/ZA9 -> /ZD4
- U9 pad 9: /Main Logic/ZA8 -> /ZD3
Other:
- board outline removed
