File: hw/ZID_MAIN/ZID_MAIN.kicad_pcb (KiCad board)
At the start: 2 copper layers, 199 parts, among them J1 HDR 1x04 Socket, J10 FFC/FPC-40 Socket, J11 Conn_02x05_PINHDR_2.54mm, J12 USB-C PWR ONLY, J2 Conn_02x03_Odd_Even, J3 Conn_01x02_Pin_2.54mm, J4 Conn_01x03, J5 Conn_01x08, J6 Conn_01x08, J7 Conn_02x04_2.54mm, J8 Conn_02x02_2.54mm, J9 Conn_02x04_2.54mm, M1 WS-RP2040-Zero, SW1 SW_Push, SW2 SW_DIP_x02, U1 OSC-20MHz, U10 74LVC2G04, U11 74LVC125AS, U12 74LVC273, U13 74FCT2245, U14 AS7C1024B, U15 74FCT2245, U16 74FCT2245, U17 74FCT2245, U18 ATF1508AS, U19 74HCT166, U2 74FCT2245, U20 74FCT257T, U21 74HCT161, U22 74AHCT244, U23 74HCT166, U24 74AHCT00, U25 ATF1504AS-44T, U26 ATF1504AS-44T, U27 ATF1504AS-44T, U28 ATF1504AS-44T, U3 24LC32, U4 MIC2775, U5 SST39SF010, U6 74LVC245, U7 74FCT2245, U8 74HCT14, U9 Z80 C20MHz-PLCC

Commit message: PLD/SCHM: Update pins.
Parts:
- removed J12: USB-C PWR ONLY, AES_Library:AES-USB_C-Molex-BdTopMnt-2171790001
- removed R44: 0, Resistor_SMD:R_0805_2012Metric_Pad1.20x1.40mm_HandSolder
- added C47: 0.1uF, Capacitor_SMD:C_0603_1608Metric, F.Cu at (390.3, 90.8)
- added C48: 0.1uF, Capacitor_SMD:C_0603_1608Metric, F.Cu at (390.3, 93.3)
- added C49: 0.1uF, Capacitor_SMD:C_0603_1608Metric, F.Cu at (390.3, 95.8)
- added C50: 0.1uF, Capacitor_SMD:C_0603_1608Metric, F.Cu at (390.3, 98.3)
- added J14: USB-C PWR ONLY, AES_Library:AES-USB_C-Molex-BdTopMnt-2171790001, F.Cu at (173.3, 59.7)
- J11: value Conn_02x05_PINHDR_2.54mm -> JST-PH-K B6B; footprint Connector_IDC:IDC-Header_2x05_P2.54mm_Vertical -> Connector_JST:JST_PH_B6B-PH-K_1x06_P2.00mm_Vertical
- J2: value Conn_02x03_Odd_Even -> JST-PH-K B6B; footprint Connector_IDC:IDC-Header_2x03_P2.54mm_Vertical -> Connector_JST:JST_PH_B6B-PH-K_1x06_P2.00mm_Vertical
- OP2: value AES-Option_A-B_2mm -> pin header 1x03 0.1"; footprint Connector_PinHeader_2.00mm:PinHeader_1x03_P2.00mm_Vertical -> Connector_PinHeader_2.54mm:PinHeader_1x03_P2.54mm_Vertical
- OP3: value AES-Option_A-B -> pin header 1x03 0.1"
- R30: value 20k -> 10k
- R31, R33: value 10k -> 20k
- R34: value 20k -> 1.2k
- R35, R39: value 1.2k -> 22
- R37: value 22 -> 10k
- R40: value 10k -> 1.2k
- R41: value 22 -> 4.7k
- R43: value 4.7k -> 0; footprint Resistor_SMD:R_0805_2012Metric -> Resistor_SMD:R_0805_2012Metric_Pad1.20x1.40mm_HandSolder
- SW1: footprint AES_Library:AES-SW_PUSH_SMD_1P1T_NO_6x6mm -> AES_Library:AES-SW_PUSH_SMD_1P1T_NO_45x45mm-CK
- TP8: value TestPoint -> EXT-BRK
- TP9: value EXT-BRK -> TestPoint
- U20: footprint Package_SO:SOIC-16W_7.5x10.3mm_P1.27mm -> Package_SO:SOIC-16_3.9x9.9mm_P1.27mm
- U21: value 74HCT161 -> 74AHCT244; footprint Package_SO:SOIC-16_3.9x9.9mm_P1.27mm -> Package_SO:SOIC-20W_7.5x12.8mm_P1.27mm
- U22: value 74AHCT244 -> 74HCT166; footprint Package_SO:SOIC-20W_7.5x12.8mm_P1.27mm -> Package_SO:SOIC-16_3.9x9.9mm_P1.27mm
- U23: value 74HCT166 -> ATF1504AS-44T; footprint Package_SO:SOIC-16_3.9x9.9mm_P1.27mm -> Package_QFP:TQFP-44_10x10mm_P0.8mm
- U9: footprint Package_LCC:PLCC-44 -> Package_LCC:PLCC-44_THT-Socket
- moved SW2 376.6 mm to (26.0, 93.3), turned to -90 degrees
- moved LED5 318.4 mm to (87.7, 142.8), turned to -90 degrees
- moved LED4 315.7 mm to (90.7, 142.8), turned to -90 degrees
- moved LED3 313.1 mm to (93.8, 142.8), turned to -90 degrees
- moved LED2 310.6 mm to (96.8, 142.8), turned to -90 degrees
- moved LED1 308.0 mm to (99.9, 142.8), turned to -90 degrees
- moved J9 300.1 mm to (89.7, 57.7), turned to -90 degrees
- moved OP2 287.4 mm to (111.6, 67.6), turned to 90 degrees
- moved SD1 283.4 mm to (76.0, 140.5)
- moved J7 277.8 mm to (105.0, 57.7), turned to -90 degrees
- moved J10 273.3 mm to (122.2, 60.4), turned to 180 degrees
- moved TP7 264.3 mm to (67.9, 57.4)
- moved TP8 262.9 mm to (73.0, 57.4)
- moved LED7 246.8 mm to (165.9, 142.7), turned to -90 degrees
- moved LED8 243.8 mm to (168.5, 142.7), turned to -90 degrees
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Connections:
- C4 pad 2: +3.3V -> +5V
- C5 pad 2: +3.3V -> +5V
- C6 pad 2: +3.3V -> +5V
- C7 pad 2: +3.3V -> +5V
- J11 pad 6: unconnected-(J11-Pin_6-Pad6) -> /JTDI_CO
- J2 pad 1: /SPIMI -> +3.3V
- J2 pad 2: +3.3V -> GND
- J2 pad 4: /SPIMO -> /SPIMI
- J2 pad 5: /SPICS2- -> /SPIMO
- J2 pad 6: GND -> /SPICS2-
- JA1 pad 1: /JTD1O2I -> /JTD2O3I
- JB1 pad 1: /JTD2O3I -> /JTD3O4I
- JC1 pad 1: /JTD3O4I -> /JTD4O5I
- JD1 pad 1: /JTD4O5I -> /JTD5O6I
- R24 pad 1: +5V -> /PU
- R24 pad 2: Net-(U21-CET) -> +5V
- R30 pad 1: /ZBACK- -> /TWAITRQ-
- R31 pad 1: /PU -> /ZBACK-
- R33 pad 1: /TWAITRQ- -> /ZHALT-
- R34 pad 1: /ZHALT- -> Net-(LED8-K)
- R34 pad 2: +5V -> GND
- R35 pad 1: Net-(LED8-K) -> Net-(R35-Pad1)
- R35 pad 2: GND -> Net-(R35-Pad2)
- R37 pad 1: Net-(R37-Pad1) -> /EXTBRKRQ-
- R37 pad 2: Net-(R37-Pad2) -> +5V
- R38 pad 1: /EXTBRKRQ- -> +5V
- R38 pad 2: +5V -> Net-(R38-Pad2)
- R39 pad 1: Net-(LED10-K) -> Net-(R38-Pad2)
- R39 pad 2: GND -> Net-(R39-Pad2)
- R40 pad 1: +5V -> Net-(LED10-K)
- R40 pad 2: Net-(R40-Pad2) -> GND
- R41 pad 1: Net-(R40-Pad2) -> +5V
- R41 pad 2: Net-(R41-Pad2) -> /BRKHW_DET-
- R42 pad 2: /BRKHW_DET- -> /BRK2N_AEQ-
- R43 pad 1: +5V -> Net-(J14-SHIELD-PadSH1)
- R43 pad 2: /BRK2N_AEQ- -> GND
- TP5 pad 1: /LCL_IO -> /IO83
- TP6 pad 1: /IO83 -> /IOBD24
- TP7 pad 1: Net-(R37-Pad1) -> Net-(R35-Pad1)
- TP8 pad 1: GND -> Net-(R38-Pad2)
- TP9 pad 1: Net-(R40-Pad2) -> GND
- U18 pad 33: /LCL_IO -> /SBC_IO
- U18 pad 48: /TGTGO -> /TGT_GO
- U18 pad 54: /TGTNOW -> /TGT_NOW
- U18 pad 60: /MEMOP- -> /MEM_OP-
- U21 pad 1: /TGTMODE- -> /ZBACK-
- U21 pad 10: Net-(U21-CET) -> GND
- U21 pad 11: unconnected-(U21-Q3-Pad11) -> /TNMI-
- U21 pad 12: unconnected-(U21-Q2-Pad12) -> /TMREQ-
- U21 pad 13: unconnected-(U21-Q1-Pad13) -> /TBREQ-
- U21 pad 14: unconnected-(U21-Q0-Pad14) -> /TIORQ-
- U21 pad 15: /TGTNOW -> /TINT-
- U21 pad 16: +5V -> /TRD-
- U21 pad 2: /MEMOP- -> /ZWR-
- U21 pad 3: Net-(U21-CET) -> /TWAITB-
- U21 pad 4: Net-(U21-CET) -> /ZRD-
- U21 pad 5: Net-(U21-CET) -> /TINTB-
- U21 pad 6: Net-(U21-CET) -> /ZIORQ-
- U21 pad 7: /TGTGO -> /TBREQB-
- U21 pad 8: GND -> /ZMREQ-
- U21 pad 9: Net-(U21-CET) -> /TNMIB-
- U22 pad 1: /ZBACK- -> Net-(U19-Qh)
- U22 pad 10: GND -> /ZA3
- U22 pad 11: /TNMI- -> /ZA2
- U22 pad 12: /TMREQ- -> /ZA1
- U22 pad 13: /TBREQ- -> /PCRD_DIN
- U22 pad 14: /TIORQ- -> /ZA0
- U22 pad 15: /TINT- -> /PC_LATCH-
- U22 pad 16: /TRD- -> +5V
- U22 pad 2: /ZWR- -> /ZA7
- U22 pad 3: /TWAITB- -> /ZA6
- U22 pad 4: /ZRD- -> /ZA5
- U22 pad 5: /TINTB- -> /ZA4
- U22 pad 6: /ZIORQ- -> GND
- U22 pad 7: /TBREQB- -> /BRKPC_RD-
- U22 pad 8: /ZMREQ- -> GND
- U22 pad 9: /TNMIB- -> /PU
- U23 pad 1: Net-(U19-Qh) -> /JTD1O2I
- U23 pad 10: /ZA3 -> /ZWR-
- U23 pad 11: /ZA2 -> /IOBD24
- U23 pad 12: /ZA1 -> /ZA4
- U23 pad 13: /PCRD_DIN -> /ZA3
- U23 pad 14: /ZA0 -> /ZA2
- U23 pad 15: /PC_LATCH- -> /ZA1
- U23 pad 16: +5V -> GND
- U23 pad 2: /ZA7 -> /SBC_GPO3
- U23 pad 3: /ZA6 -> /ZD6
- U23 pad 4: /ZA5 -> GND
- U23 pad 5: /ZA4 -> /ZD7
- U23 pad 6: GND -> /ZD5
- U23 pad 7: /BRKPC_RD- -> /JTMS
- U23 pad 8: GND -> /BRK_DEQ
- U23 pad 9: /PU -> +5V
- U25 pad 1: /JTD1O2I -> /JTD2O3I
- U25 pad 32: /JTD2O3I -> /JTD3O4I
- U26 pad 1: /JTD2O3I -> /JTD3O4I
- U26 pad 32: /JTD3O4I -> /JTD4O5I
- U27 pad 1: /JTD3O4I -> /JTD4O5I
- U27 pad 32: /JTD4O5I -> /JTD5O6I
- U28 pad 1: /JTD4O5I -> /JTD5O6I
- U8 pad 4: Net-(R37-Pad2) -> Net-(R35-Pad2)
- U8 pad 5: Net-(R41-Pad2) -> Net-(R39-Pad2)

Commit message: PLD: Update pins. SCHM: PLD pins, TCTRL correction.
Parts:
- removed JS1: SolderJumper_2_Open, Jumper:SolderJumper-2_P1.3mm_Open_TrianglePad1.0x1.5mm
- removed R32, R34: 1.2k, Resistor_SMD:R_0805_2012Metric
- added JS6: SolderJumper_2_Open, Jumper:SolderJumper-2_P1.3mm_Open_TrianglePad1.0x1.5mm, F.Cu at (221.8, 87.8)
- added JS7: SolderJumper_2_Open, Jumper:SolderJumper-2_P1.3mm_Open_TrianglePad1.0x1.5mm, F.Cu at (221.8, 91.3)
- added R44: 0, Resistor_SMD:R_0805_2012Metric_Pad1.20x1.40mm_HandSolder, F.Cu at (233.5, 85.5)
- added TP28: TestPoint, Connector_PinHeader_2.54mm:PinHeader_1x01_P2.54mm_Vertical, F.Cu at (208.1, 74.1)
- added TP29: TestPoint, Connector_PinHeader_2.54mm:PinHeader_1x01_P2.54mm_Vertical, F.Cu at (208.1, 78.7)
- added TP30: TestPoint, Connector_PinHeader_2.54mm:PinHeader_1x01_P2.54mm_Vertical, F.Cu at (208.1, 83.3)
- added TP31: TestPoint, Connector_PinHeader_2.54mm:PinHeader_1x01_P2.54mm_Vertical, F.Cu at (208.1, 87.9)
- added TP32: TestPoint, Connector_PinHeader_2.54mm:PinHeader_1x01_P2.54mm_Vertical, F.Cu at (208.1, 92.5)
- added TP33: TestPoint, Connector_PinHeader_2.54mm:PinHeader_1x01_P2.54mm_Vertical, F.Cu at (69.5, 31.7)
- added TP34: TestPoint, Connector_PinHeader_2.54mm:PinHeader_1x01_P2.54mm_Vertical, F.Cu at (69.5, 36.3)
- added TP42: TestPoint, Connector_PinHeader_2.54mm:PinHeader_1x01_P2.54mm_Vertical, F.Cu at (217.3, 83.3)
- added TP43: TestPoint, Connector_PinHeader_2.54mm:PinHeader_1x01_P2.54mm_Vertical, F.Cu at (217.3, 87.9)
- added TP44: TestPoint, Connector_PinHeader_2.54mm:PinHeader_1x01_P2.54mm_Vertical, F.Cu at (217.3, 92.5)
- added TP45: TestPoint, Connector_PinHeader_2.54mm:PinHeader_1x01_P2.54mm_Vertical, F.Cu at (217.3, 97.1)
- C1, C2: value 0.1u -> 0.1uf; footprint Capacitor_SMD:C_0603_1608Metric_Pad1.08x0.95mm_HandSolder -> Capacitor_SMD:C_0603_1608Metric
- C3: footprint Capacitor_SMD:C_1210_3225Metric_Pad1.33x2.70mm_HandSolder -> Capacitor_SMD:C_0603_1608Metric
- J1: value HDR 1x04 Socket -> Conn 1x04 0.1" Socket
- J3: value Conn_01x02_Pin_2.54mm -> Conn 1x02 0.1" pin
- J4: value Conn_01x03 -> Conn 1x03 0.1" pin
- J5, J6: value Conn_01x08 -> Conn 1x08 0.1" pin
- J7, J9: value Conn_02x04_2.54mm -> Conn 2x04 0.1" pin
- J8: value Conn_02x02_2.54mm -> Conn 2x02 0.1" pin
- R26: value 4.7k -> 10k
- R29: value 1.2k -> 4.7k
- R30, R37: value 10k -> 1.2k
- R31: value 20k -> 10k
- R33: value 20k -> 1.2k
- R35: value 22 -> 1.2k
- R36, R40: value 1.2k -> 22
- R39: value 22 -> 10k
- R41: value 4.7k -> 1.2k
- R43: value 0 -> 4.7k; footprint Resistor_SMD:R_0805_2012Metric_Pad1.20x1.40mm_HandSolder -> Resistor_SMD:R_0805_2012Metric
- SPARE1: footprint AES_Library:SPARE-and-SOIC-16-AES -> AES_Library:SPARE-16-SOT-5_6-AES
- TP14: value TestPoint -> SYNC-CONN
- TP15: value TestPoint -> EXT-BRK
- TP7: value SYNC-CONN -> TestPoint
- TP8: value EXT-BRK -> TestPoint
- U12: footprint Package_SO:SOIC-20W_7.5x12.8mm_P1.27mm -> Package_SO:SO-20_12.8x7.5mm_P1.27mm
- U13, U15, U16, U17, U2, U7: footprint Package_SO:SOIC-20W_7.5x12.8mm_P1.27mm -> Package_SO:SSOP-20_3.9x8.7mm_P0.635mm
- U20: value 74FCT257T -> 74FCT2244; footprint Package_SO:SOIC-16_3.9x9.9mm_P1.27mm -> Package_SO:SSOP-20_3.9x8.7mm_P0.635mm
- U21: value 74AHCT244 -> 74HCT166; footprint Package_SO:SOIC-20W_7.5x12.8mm_P1.27mm -> Package_SO:SOIC-16_3.9x9.9mm_P1.27mm
- U22: value 74HCT166 -> ATF1504AS-44T; footprint Package_SO:SOIC-16_3.9x9.9mm_P1.27mm -> Package_QFP:TQFP-44_10x10mm_P0.8mm
- U23: value ATF1504AS-44T -> 74AHCT00; footprint Package_QFP:TQFP-44_10x10mm_P0.8mm -> Package_SO:SO-14_3.9x8.65mm_P1.27mm
- U24: value 74AHCT00 -> 74FCT2244; footprint Package_SO:SOIC-14_3.9x8.7mm_P1.27mm -> Package_SO:SSOP-20_3.9x8.7mm_P0.635mm
- U6: footprint Package_SO:SOIC-20W_7.5x12.8mm_P1.27mm -> Package_SO:SO-20_5.3x12.6mm_P1.27mm
- U8: value 74HCT14 -> 74AHCT14; footprint Package_SO:SOIC-14_3.9x8.7mm_P1.27mm -> Package_SO:SO-14_3.9x8.65mm_P1.27mm
- moved U22 310.8 mm to (81.9, 33.9)
- moved U14 303.1 mm to (96.5, 108.6)
- moved TP14 299.6 mm to (68.9, 57.4)
- moved U5 294.4 mm to (62.8, 96.8)
- moved TP15 293.7 mm to (73.0, 57.4)
- moved J5 291.7 mm to (107.0, 72.1), turned to 90 degrees
- moved J6 283.1 mm to (119.7, 66.5), turned to 90 degrees
- moved U25 278.9 mm to (89.2, 157.0), turned to 135 degrees
- moved U15 275.1 mm to (70.2, 154.3)
- moved U9 269.4 mm to (119.7, 101.6)
- moved U17 262.9 mm to (70.0, 168.1)
- moved U20 261.5 mm to (121.0, 88.5), turned to 90 degrees
- moved J1 255.9 mm to (142.0, 133.6), turned to 90 degrees
- moved U26 253.6 mm to (110.6, 157.0), turned to 135 degrees
- moved U3 248.8 mm to (150.2, 124.0), turned to 90 degrees
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Connections:
- net /I88 renamed /IOE1
- J7 pad 1: (no net) -> GND
- J7 pad 2: (no net) -> /SBC_O0
- J7 pad 3: (no net) -> GND
- J7 pad 4: (no net) -> /SBC_O1
- J7 pad 5: (no net) -> GND
- J7 pad 6: (no net) -> /SBC_O2
- J7 pad 7: (no net) -> GND
- J7 pad 8: (no net) -> /SBC_O3
- J8 pad 1: (no net) -> +5V
- J8 pad 2: (no net) -> +5V
- J8 pad 3: (no net) -> +5V
- J8 pad 4: (no net) -> +5V
- J9 pad 1: (no net) -> GND
- J9 pad 2: (no net) -> /SBC_I0
- J9 pad 3: (no net) -> GND
- J9 pad 4: (no net) -> /SBC_I1
- J9 pad 5: (no net) -> GND
- J9 pad 6: (no net) -> /SBC_I2
- J9 pad 7: (no net) -> +5V
- J9 pad 8: (no net) -> /MODINT-
- R23 pad 1: Net-(OP1-C) -> +5V
- R23 pad 2: +5V -> Net-(U20-Ib1)
- R24 pad 1: /PU -> Net-(OP1-C)
- R25 pad 1: +5V -> /PU
- R25 pad 2: /JTDO_CI -> +5V
- R26 pad 2: /JTCK -> /JTDO_CI
- R27 pad 2: /JTMS -> /JTCK
- R28 pad 2: /JTDI_CO -> /JTMS
- R29 pad 1: Net-(LED6-K) -> +5V
- R29 pad 2: GND -> /JTDI_CO
- R30 pad 1: /TWAITRQ- -> Net-(LED6-K)
- R30 pad 2: +5V -> GND
- R31 pad 1: /ZBACK- -> /TWAITRQ-
- R33 pad 1: /ZHALT- -> Net-(LED7-K)
- R33 pad 2: +5V -> GND
- R35 pad 1: Net-(R35-Pad1) -> Net-(LED8-K)
- R35 pad 2: Net-(R35-Pad2) -> GND
- R36 pad 1: Net-(LED9-K) -> Net-(R36-Pad1)
- R36 pad 2: GND -> Net-(R36-Pad2)
- R37 pad 1: /EXTBRKRQ- -> Net-(LED9-K)
- R37 pad 2: +5V -> GND
- R38 pad 1: +5V -> /EXTBRKRQ-
- R38 pad 2: Net-(R38-Pad2) -> +5V
- R39 pad 1: Net-(R38-Pad2) -> +5V
- R40 pad 1: Net-(LED10-K) -> Net-(R39-Pad2)
- R40 pad 2: GND -> Net-(R40-Pad2)
- R41 pad 1: +5V -> Net-(LED10-K)
- R41 pad 2: /BRKHW_DET- -> GND
- R42 pad 2: /BRK2N_AEQ- -> /BRKHWDET-
- R43 pad 1: Net-(J14-SHIELD-PadSH1) -> +5V
- R43 pad 2: GND -> /BRKN_AEQ-
- TP10 pad 1: /ENBL_DOD -> /IO85
- TP11 pad 1: /ADDR_DOD -> /IO83
- TP12 pad 1: /IO8A -> /IO81
- TP13 pad 1: /IO8B -> /IOBD24
- TP14 pad 1: /IO8C -> Net-(R36-Pad1)
- TP15 pad 1: /IO8D -> Net-(R39-Pad2)
- TP16 pad 1: /IO10A -> GND
- TP17 pad 1: /IO10B -> /ENBL_DOD
- TP18 pad 1: /IO10C -> /ADDR_DOD
- TP19 pad 1: /IO10D -> /IO8A
- TP20 pad 1: /GPO_A- -> /IO8B
- TP21 pad 1: /GPO_B- -> /IO8C
- TP22 pad 1: /GPO_B- -> /IO8D
- TP23 pad 1: /GPI_A- -> /IO10A
- TP24 pad 1: /GPI_B- -> /IO10B
- TP25 pad 1: /GPI_B- -> /IO10C
- TP26 pad 1: Net-(JS1-B) -> /IO10D
- TP27 pad 1: Net-(TP27-Pad1) -> /GPO_A-
- TP3 pad 1: /IO78 -> /IO123
- TP4 pad 1: /IO77 -> /IO121
- TP5 pad 1: /IO83 -> /IO120
- TP6 pad 1: /IOBD24 -> /IO64
- TP7 pad 1: Net-(R35-Pad1) -> /IO62
- TP8 pad 1: Net-(R38-Pad2) -> /IO61
- TP9 pad 1: GND -> /IO59
- U15 pad 11: /ZA7 -> /LA7
- U15 pad 12: /ZA6 -> /LA6
- U15 pad 13: /ZA5 -> /LA5
- U15 pad 14: /ZA4 -> /LA4
- U15 pad 15: /ZA3 -> /LA3
- U15 pad 16: /ZA2 -> /LA2
- U15 pad 17: /ZA1 -> /LA1
- U15 pad 18: /ZA0 -> /LA0
- U15 pad 2: /LA0 -> /ZA0
- U15 pad 3: /LA1 -> /ZA1
- U15 pad 4: /LA2 -> /ZA2
- U15 pad 5: /LA3 -> /ZA3
- U15 pad 6: /LA4 -> /ZA4
- U15 pad 7: /LA5 -> /ZA5
- U15 pad 8: /LA6 -> /ZA6
- U15 pad 9: /LA7 -> /ZA7
- U17 pad 11: /ZA15 -> /LA15
- U17 pad 12: /ZA14 -> /LA14
- U17 pad 13: /ZA13 -> /LA13
- U17 pad 14: /ZA12 -> /LA12
- U17 pad 15: /ZA11 -> /LA11
- U17 pad 16: /ZA10 -> /LA10
- U17 pad 17: /ZA9 -> /LA9
- U17 pad 18: /ZA8 -> /LA8
- U17 pad 2: /LA8 -> /ZA8
- U17 pad 3: /LA9 -> /ZA9
- U17 pad 4: /LA10 -> /ZA10
- U17 pad 5: /LA11 -> /ZA11
- U17 pad 6: /LA12 -> /ZA12
- U17 pad 7: /LA13 -> /ZA13
- U17 pad 8: /LA14 -> /ZA14
- U17 pad 9: /LA15 -> /ZA15
- U18 pad 1: /ZA1 -> /ZA2
- U18 pad 10: /ZA14 -> /TGT_NOW
- U18 pad 100: /ZD2 -> /ZA3
- U18 pad 12: /ZWR- -> /BRKN_AEQ-
- U18 pad 13: /ZA4 -> /BRK1_AEQ-
- U18 pad 14: /ZA3 -> /BRK_DEQ
- U18 pad 16: /SBC_GPO1 -> /MEM_OP-
- U18 pad 17: /SBC_GPO0 -> /TDBUSIN-
- U18 pad 19: /ZA2 -> /MOD_SEL-
- U18 pad 2: /ZRD- -> /ZA1
- U18 pad 20: /SBC_GPI3 -> /PC_LATCH-
- U18 pad 21: /PCRD_DIN -> /RFMR-
- U18 pad 22: /SBC_GPI2 -> /SBCMODE-
- U18 pad 23: /BRKHW_DET- -> /ZMREQ-
- U18 pad 24: /SBCMODE- -> /MWTRQ-
- U18 pad 25: /ZRFSH- -> /ZWR-
- U18 pad 27: /ROM_SEL -> /IO64
- U18 pad 28: /RRA1 -> /IO62
- U18 pad 29: /RRA0 -> /IO61
- U18 pad 30: /RRA2 -> /IO59
- U18 pad 31: /ZWAIT- -> /TGTONLY-
- U18 pad 32: /RAM_SEL- -> /TINTB-
- U18 pad 33: /SBC_IO -> /TBREQB-
- U18 pad 35: /RFMR- -> /TNMIB-
- U18 pad 36: /TGTMODE- -> /BRD_RST-
- U18 pad 37: /SYNC -> /TWAITRQ-
- U18 pad 40: /BRK2N_AEQ- -> /ZBACK-
- U18 pad 41: /TWAITRQ- -> /TDBUSEN-
- U18 pad 42: /ZIORQ- -> /TCBUSEN-
- U18 pad 44: /ZA5 -> /TCBUSFEN-
- U18 pad 45: /ZA6 -> /SBC_IO
- U18 pad 46: /SBC_GPO2 -> /RRA1
- U18 pad 47: /SBC_GPO3 -> /RRA0
- U18 pad 48: /TGT_GO -> /RRA2
- U18 pad 49: /ZD5 -> /ROM_SEL
- U18 pad 5: /ZD6 -> /ZD0
- U18 pad 50: /ZD4 -> /RAM_SEL-
- U18 pad 52: /ZA7 -> /IO81
- U18 pad 54: /TGT_NOW -> /IO85
- U18 pad 55: /SBC_GPI0 -> /BA_CLK
- U18 pad 56: /SBC_GPI1 -> /AEN_CLR-
- U18 pad 57: /ZBACK- -> /AEN_CLK
- U18 pad 58: /ZNMI- -> /BA_CLR-
- U18 pad 6: /ZD0 -> /ZRD-
- U18 pad 60: /MEM_OP- -> /BRKPC_RD-
- U18 pad 61: /TDBUSIN- -> /TGT_GO
- U18 pad 63: /TNMIB- -> /ZIORQ-
- U18 pad 64: /BRK1_AEQ- -> /ZA5
- U18 pad 65: /TBREQB- -> /ZA6
- U18 pad 67: /BRD_RST- -> /SYNC
- U18 pad 68: /EXTBRKRQ- -> /ZINT-
- U18 pad 69: /PC_LATCH- -> /ZBREQ-
- U18 pad 7: /ZD7 -> /ZD6
- U18 pad 70: /ZBREQ- -> /ZNMI-
- U18 pad 72: /ZRST- -> /ZWAIT-
- U18 pad 75: /TINTB- -> /ZA7
- U18 pad 76: /TGTONLY- -> /BRKHWDET-
- U18 pad 77: /IO77 -> /PCRD_DIN
- U18 pad 78: /IO78 -> /EXTBRKRQ-
- U18 pad 79: /BRKPC_RD- -> /IO120
- U18 pad 8: /MWTRQ- -> /ZD4
- U18 pad 80: /ZINT- -> /IO121
- U18 pad 81: /TDBUSEN- -> /IO123
- U18 pad 83: /FIXED_SEL -> /ZRST-
- U18 pad 84: /D7_B -> /TGTMODE-
- U18 pad 89: /ZMREQ- -> /ZRFSH-
- U18 pad 9: /ZA15 -> /ZD5
- U18 pad 92: /AEN_CLK -> /ZD1
- U18 pad 93: /ZD1 -> /ZD2
- U18 pad 94: /AEN_CLR- -> /ZA15
- U18 pad 96: /MOD_SEL- -> /ZD3
- U18 pad 97: /BA_CLK -> /ZD7
- U18 pad 98: /BA_CLR- -> /ZA14
- U18 pad 99: /ZD3 -> /ZA4
- U20 pad 1: /FIXED_SEL -> /TCBUSEN-
- U20 pad 10: Net-(OP1-C) -> GND
- U20 pad 11: /ZMREQ- -> Net-(U20-Ib1)
- U20 pad 12: /TIORQ- -> /TWR-
- U20 pad 13: /PU -> Net-(U20-Ib1)
- U20 pad 14: /ZIORQ- -> /TRD-
- U20 pad 15: /ZBACK -> Net-(U20-Ib1)
- U20 pad 16: +5V -> /TIORQ-
- U20 pad 2: /ZWR- -> /ZMREQ-
- U20 pad 3: /PU -> /TMREQ-
- U20 pad 4: /TWR- -> /ZIORQ-
- U20 pad 5: /ZRD- -> /TIORQ-
- U20 pad 6: /PU -> /ZRD-
- U20 pad 8: GND -> /ZWR-
- U20 pad 9: /TMREQ- -> /TWR-
- U21 pad 1: /ZBACK- -> Net-(U19-Qh)
- U21 pad 10: GND -> /ZA3
- U21 pad 11: /TNMI- -> /ZA2
- U21 pad 12: /TMREQ- -> /ZA1
- U21 pad 13: /TBREQ- -> /PCRD_DIN
- U21 pad 14: /TIORQ- -> /ZA0
- U21 pad 15: /TINT- -> /PC_LATCH-
- U21 pad 16: /TRD- -> +5V
- U21 pad 2: /ZWR- -> /ZA7
- U21 pad 3: /TWAITB- -> /ZA6
- U21 pad 4: /ZRD- -> /ZA5
- U21 pad 5: /TINTB- -> /ZA4
- U21 pad 6: /ZIORQ- -> GND
- U21 pad 7: /TBREQB- -> /BRKPC_RD-
- U21 pad 8: /ZMREQ- -> GND
- U21 pad 9: /TNMIB- -> /PU
- U22 pad 1: Net-(U19-Qh) -> /JTD1O2I
- U22 pad 10: /ZA3 -> /IOBD25
- U22 pad 11: /ZA2 -> /IOBD24
- U22 pad 12: /ZA1 -> /ZA4
- U22 pad 13: /PCRD_DIN -> /ZA3
- U22 pad 14: /ZA0 -> /ZA2
- U22 pad 15: /PC_LATCH- -> /ZA1
- U22 pad 16: +5V -> GND
- U22 pad 2: /ZA7 -> /SBC_GPO3
- U22 pad 3: /ZA6 -> /ZD6
- U22 pad 4: /ZA5 -> GND
- U22 pad 5: /ZA4 -> /ZD7
- U22 pad 6: GND -> /ZD5
- U22 pad 7: /BRKPC_RD- -> /JTMS
- U22 pad 8: GND -> /BRK_DEQ
- U22 pad 9: /PU -> +5V
- U23 pad 1: /JTD1O2I -> /TGTMODE-
- U23 pad 10: /ZWR- -> /LRST-
- U23 pad 11: /IOBD24 -> Net-(LED9-A)
- U23 pad 12: /ZA4 -> /TWAIT-
- U23 pad 13: /ZA3 -> /LRST-
- U23 pad 14: /ZA2 -> +5V
- U23 pad 2: /SBC_GPO3 -> /LRST-
- U23 pad 3: /ZD6 -> Net-(LED6-A)
- U23 pad 4: GND -> /ZBACK-
- U23 pad 5: /ZD7 -> /LRST-
- U23 pad 6: /ZD5 -> Net-(LED7-A)
- U23 pad 7: /JTMS -> GND
- U23 pad 8: /BRK_DEQ -> Net-(LED8-A)
- U23 pad 9: +5V -> /ZHALT-
- U24 pad 1: /TGTMODE- -> /ZBACK-
- U24 pad 10: /LRST- -> GND
- U24 pad 11: Net-(LED9-A) -> /TNMI-
- U24 pad 12: /TWAIT- -> /ZWR-
- U24 pad 13: /LRST- -> /TBREQ-
- U24 pad 14: +5V -> /ZRD-
- U24 pad 2: /LRST- -> /TMREQ-
- U24 pad 3: Net-(LED6-A) -> /TWAITB-
- U24 pad 4: /ZBACK- -> /TIORQ-
- U24 pad 5: /LRST- -> /TINTB-
- U24 pad 6: Net-(LED7-A) -> /TRD-
- U24 pad 7: GND -> /TBREQB-
- U24 pad 8: Net-(LED8-A) -> /TWR-
- U24 pad 9: /ZHALT- -> /TNMIB-
- U25 pad 38: /D7_B -> /ZD7
- U25 pad 42: /BRK2N_AEQ- -> /BRKN_AEQ-
- U25 pad 44: /BRKHW_DET- -> /BRKHWDET-
- U25 pad 5: /BRKHW_DET- -> /BRKHWDET-
- U25 pad 6: /D7_B -> /ZD7
- U26 pad 42: /BRK2N_AEQ- -> /BRKN_AEQ-
- U26 pad 43: /BRK2N_AEQ- -> /BRKN_AEQ-
- U26 pad 44: /BRKHW_DET- -> /BRKHWDET-
- U26 pad 5: /BRKHW_DET- -> /BRKHWDET-
- U27 pad 42: /BRK2N_AEQ- -> /BRKN_AEQ-
- U27 pad 43: /BRK2N_AEQ- -> /BRKN_AEQ-
- U27 pad 44: /BRKHW_DET- -> /BRKHWDET-
- U27 pad 5: /BRKHW_DET- -> /BRKHWDET-
- U28 pad 42: /BRK2N_AEQ- -> /BRKN_AEQ-
- U28 pad 43: /BRK2N_AEQ- -> /BRKN_AEQ-
- U28 pad 44: /BRKHW_DET- -> /BRKHWDET-
- U28 pad 5: /BRKHW_DET- -> /BRKHWDET-
- U8 pad 10: /ZBACK -> Net-(TP43-Pad1)
- U8 pad 11: /ZBACK- -> Net-(JS6-B)
- U8 pad 12: Net-(TP27-Pad1) -> Net-(TP45-Pad1)
- U8 pad 13: Net-(JS1-B) -> Net-(JS7-B)
- U8 pad 4: Net-(R35-Pad2) -> Net-(R36-Pad2)
- U8 pad 5: Net-(R39-Pad2) -> Net-(R40-Pad2)
