File: hw/ZID_POD/Pod2/ZID_POD.kicad_sch (KiCad schematic)
At the start: 2 parts, among them J1 FFC/FPC-40 Socket

Commit message: PCB: Ready to order - ZID, POD1, POD2, POD3, POD4, ExpBP
Parts:
- J1: footprint (none) -> AES_Library:CviLux_CF25401D0-05-NH_FFC-FPC-AES
Changed lines of the file:
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@@
 	(title_block
 		(title "ZID POD (2)")
-		(date "2026-04-21")
+		(date "2026-08-16")
 		(rev "PR1.0")
 		(company "SilkyDESIGN")
@@
 		)
 		(instances
-			(project ""
+			(project "ZID_POD"
 				(path "/5064845c-49f8-454d-ae5f-d06818afd8fe"
 					(reference "Z80-SKT1")
@@
 			)
 		)
-		(property "Footprint" ""
+		(property "Footprint" "AES_Library:CviLux_CF25401D0-05-NH_FFC-FPC-AES"
 			(at 102.87 102.87 0)
 			(effects
