File: hw/ZID_EXP_BP/ZID_EXP_BP.kicad_sch (KiCad schematic)
At the start: 64 parts, among them J1 FFC/FPC-40 Socket, J15 JST-PH-K B6B, J2 Conn 2x04 0.1" pin, J3 Conn 2x02 0.1" pin, J4 Conn 2x04 0.1" pin, Q1 DMG2305UX, SW1 SW_DIP_x08, U1 ATF1502AS-44T

Commit message: PCB: Ready to order - ZID, POD1, POD2, POD3, POD4, ExpBP
Parts:
- SW1: SW4 (none) -> A3; SW5 (none) -> A4; SW6 (none) -> A5; SW7 (none) -> A6; SW8 (none) -> A7
Changed lines of the file:
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@@
+			)
+		)
+		(property "SW4" "A3"
+			(at 302.26 187.96 0)
+			(effects
+				(font
+					(size 1.27 1.27)
+				)
+				(hide yes)
+			)
+		)
+		(property "SW5" "A4"
+			(at 302.26 187.96 0)
+			(effects
+				(font
+					(size 1.27 1.27)
+				)
+				(hide yes)
+			)
+		)
+		(property "SW6" "A5"
+			(at 302.26 187.96 0)
+			(effects
+				(font
+					(size 1.27 1.27)
+				)
+				(hide yes)
+			)
+		)
+		(property "SW7" "A6"
+			(at 302.26 187.96 0)
+			(effects
+				(font
+					(size 1.27 1.27)
+				)
+				(hide yes)
+			)
+		)
+		(property "SW8" "A7"
+			(at 302.26 187.96 0)
+			(effects
+				(font
+					(size 1.27 1.27)
+				)
+				(hide yes)
 			)
 		)

Commit message: PCB: ExpBP, add power LED
Parts:
- added LED1: LED BLUE, LED_SMD:LED_0805_2012Metric, symbol Device:LED
- added R17: 1.2k, Resistor_SMD:R_0805_2012Metric, symbol Device:R_Small_US
Connections:
- net +5V: now also LED1.2 (A)
- net GND: now also R17.2
- new net: LED1.1 (K), R17.1
